File: matrix-switch/matrix-switch.kicad_pcb (KiCad board)
At the start: 4 copper layers, 53.3 x 71.1 mm, 347 parts, among them J1 Conn_01x02, J10 Conn_01x02, J11 Conn_01x02, J12 Conn_01x02, J13 Conn_01x02, J14 Conn_01x02, J15 Conn_01x02, J16 Conn_01x02, J17 Conn_01x02, J18 Conn_01x02, J19 Conn_01x02, J2 Conn_01x02, J20 Conn_01x02, J21 Conn_01x02, J22 Conn_01x02, J23 Conn_01x02, J24 Conn_01x02, J25 Conn_01x02, J26 Conn_01x02, J27 Conn_01x02, J28 Conn_01x02, J29 Conn_01x02, J3 Conn_01x02, J30 Conn_01x02, J31 Conn_01x02, J32 Conn_01x02, J33 Conn_01x02, J34 Conn_01x05, J35 Conn_01x05, J36 Conn_01x02, J37 Conn_01x02, J38 Conn_01x02, J39 Conn_01x02, J4 Conn_01x02, J40 Conn_01x02, J41 Conn_01x02, J42 Conn_01x02, J43 Conn_01x02, J5 Conn_01x02, J6 Conn_01x02, J7 Conn_01x02, J8 Conn_01x02, J9 Conn_01x02, U1 ASSR-1218, U10 ASSR-1218, U100 ASSR-1218, U101 ASSR-1218, U102 ASSR-1218, U103 ASSR-1218, U104 ASSR-1218, U105 ASSR-1218, U106 ASSR-1218, U107 ASSR-1218, U108 ASSR-1218, U109 ASSR-1218, U11 ASSR-1218, U110 ASSR-1218, U111 ASSR-1218, U112 ASSR-1218, U113 ASSR-1218, U114 ASSR-1218, U115 ASSR-1218, U116 ASSR-1218, U117 ASSR-1218, U118 ASSR-1218, U119 ASSR-1218, U12 ASSR-1218, U120 ASSR-1218, U121 ASSR-1218, U122 ASSR-1218, U123 ASSR-1218, U124 ASSR-1218, U125 ASSR-1218, U126 ASSR-1218, U127 ASSR-1218, U128 ASSR-1218, U129 STP16DPPS05, U13 ASSR-1218, U130 STP16DPPS05, U131 STP16DPPS05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

Commit message: wip on matrix switch card edge adapter board
Parts:
- removed TP100, TP101, TP102, TP103, TP104, TP105, TP106, TP107, TP108, TP109, TP110, TP111, TP112, TP113, TP114, TP115, TP116, TP117, TP118, TP119, TP120, TP121, TP122, TP123, TP124, TP125, TP126, TP127, TP128, TP65, TP66, TP67, TP68, TP69, TP70, TP71, TP72, TP73, TP74, TP75, TP76, TP77, TP78, TP79, TP80, TP81, TP82, TP83, TP84, TP85, TP86, TP87, TP88, TP89, TP90, TP91, TP92, TP93, TP94, TP95, TP96, TP97, TP98, TP99: TestPoint, Connector_Pin:Pin_D1.0mm_L10.0mm
- added H10: MountingHole_Pad, MountingHole:MountingHole_2.2mm_M2_Pad_Via, F.Cu at (-137.2, 289.6)
- added H11: MountingHole_Pad, MountingHole:MountingHole_2.2mm_M2_Pad_Via, F.Cu at (-88.9, 289.6)
- added H12: MountingHole_Pad, MountingHole:MountingHole_2.2mm_M2_Pad_Via, F.Cu at (-88.9, 355.6)
- added H9: MountingHole_Pad, MountingHole:MountingHole_2.2mm_M2_Pad_Via, F.Cu at (-137.2, 355.6)
- added J44: Conn_01x18, Connector_PinHeader_2.54mm:PinHeader_1x18_P2.54mm_Vertical, F.Cu at (367.6, 108.3)
- added J45: Conn_01x15, Connector_PinHeader_2.54mm:PinHeader_1x15_P2.54mm_Vertical, F.Cu at (404.8, 108.3)
- added J46: Conn_01x15, Connector_PinHeader_2.54mm:PinHeader_1x15_P2.54mm_Vertical, F.Cu at (400.1, 108.3)
- added J47: Conn_01x15, Connector_PinHeader_2.54mm:PinHeader_1x15_P2.54mm_Vertical, F.Cu at (395.5, 108.3)
- added J48: Conn_01x15, Connector_PinHeader_2.54mm:PinHeader_1x15_P2.54mm_Vertical, F.Cu at (390.8, 108.3)
- added J49: Conn_01x15, Connector_PinHeader_2.54mm:PinHeader_1x15_P2.54mm_Vertical, F.Cu at (386.2, 108.3)
- added J50: Conn_01x15, Connector_PinHeader_2.54mm:PinHeader_1x15_P2.54mm_Vertical, F.Cu at (381.5, 108.3)
- added J51: Conn_01x15, Connector_PinHeader_2.54mm:PinHeader_1x15_P2.54mm_Vertical, F.Cu at (376.9, 108.3)
- added J52: Conn_01x15, Connector_PinHeader_2.54mm:PinHeader_1x15_P2.54mm_Vertical, F.Cu at (372.2, 108.3)
- added J53: Conn_01x16, Connector_PinHeader_2.54mm:PinHeader_1x16_P2.54mm_Vertical, F.Cu at (-132.1, 355.6)
- added J54: Conn_02x30_Odd_Even, Connector_PCBEdge:Samtec_MECF-30-0_-L-DV_2x30_P1.27mm_Polarized_Edge, F.Cu at (-113.0, 361.9)
- added J55: Conn_01x23, Connector_PinHeader_2.54mm:PinHeader_1x23_P2.54mm_Vertical, F.Cu at (-91.4, 294.6)
- added J56: Conn_01x07, Connector_PinHeader_2.54mm:PinHeader_1x07_P2.54mm_Vertical, F.Cu at (409.4, 108.3)
- added J57: Conn_01x18, Connector_PinHeader_2.54mm:PinHeader_1x18_P2.54mm_Horizontal, B.Cu at (-119.4, 301.0)
- added J58: Conn_01x07, Connector_PinHeader_2.54mm:PinHeader_1x07_P2.54mm_Horizontal, B.Cu at (-97.8, 303.5)
- added JP13: Jumper_NC_Small, Jumper:SolderJumper-2_P1.3mm_Bridged_RoundedPad1.0x1.5mm, F.Cu at (413.9, 107.8)
- added R11: 0R, Resistor_SMD:R_0805_2012Metric, F.Cu at (367.5, 155.3)
Connections:
- H3 pad 1: GND -> VDD
- H4 pad 1: VDD -> GND
- U129 pad 5: SR1C1 -> Net-(JP13-Pad1)
Routing:
- net R7_FL: track 0.00 -> 7.58 mm, vias 0 -> 1
- net DATA_OUT: track 0.00 -> 7.58 mm, vias 0 -> 1
- net C_FL: track 0.00 -> 7.58 mm, vias 0 -> 1
- net CLOCK: track 0.00 -> 6.38 mm, vias 0 -> 1
- net R8_FL: track 0.00 -> 6.31 mm, vias 0 -> 1
- net R6_FL: track 0.00 -> 6.31 mm, vias 0 -> 1
- net C8_FH: track 24.0 -> 28.3 mm, vias 8 -> 9
- net C7_FH: track 24.0 -> 28.3 mm, vias 8 -> 9
- net R7_SL: track 0.00 -> 4.33 mm, vias 0 -> 1
- net R3_SL: track 0.00 -> 4.33 mm, vias 0 -> 1
- net DATA_IN: track 0.00 -> 4.33 mm, vias 0 -> 1
- net R5_SL: track 0.00 -> 4.33 mm, vias 0 -> 1
- net R1_SL: track 0.00 -> 4.33 mm, vias 0 -> 1
- net C_SL: track 0.00 -> 4.33 mm, vias 0 -> 1
- net LATCH: track 0.00 -> 3.06 mm, vias 0 -> 1
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- added copper zone on B.Cu, net GND
Other:
- board size 53.3 x 71.1 mm -> 251.5 x 325.1 mm

Commit message: matrix switch wip
Parts:
- moved J57 4.58 mm to (-116.8, 304.8)
- moved J58 1.80 mm to (-99.1, 304.8)
Routing:
- net R1_SH: track 11.7 -> 120.6 mm, vias 8 -> 10
- net R1_FH: track 18.0 -> 124.8 mm, vias 8 -> 11
- net R2_SH: track 11.7 -> 110.4 mm, vias 8 -> 10
- net VSS: track 0.00 -> 52.7 mm, vias 0 -> 4
- net C8_SH: track 27.1 -> 49.8 mm
- net C8_FH: track 28.3 -> 49.4 mm
- net C4_SH: track 24.0 -> 43.9 mm, vias 8 -> 10
- net C5_FH: track 24.0 -> 43.8 mm, vias 8 -> 9
- net C7_SH: track 27.1 -> 44.2 mm
- net C7_FH: track 28.3 -> 45.1 mm
- net C5_SH: track 24.0 -> 38.6 mm
- net C6_SH: track 27.1 -> 41.4 mm
- net C4_FH: track 24.0 -> 35.8 mm, vias 8 -> 9
- net C3_SH: track 24.0 -> 35.3 mm, vias 8 -> 9
- net C3_FH: track 24.0 -> 34.1 mm, vias 8 -> 9
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- added copper zone on F.Cu, net VSS
