File: four-by-four_crossbar/four-by-four_crossbar.kicad_pcb (KiCad board)
At the start: 6 copper layers, 150 x 35 mm, 6 parts, among them J1 Conn_02x12_USBC_pins, J2 Conn_02x12_USBC_pins, J3 Conn_02x12_USBC_pins, J4 Conn_02x12_USBC_pins, J5 Conn_02x12_USBC_pins_shielded, J6 Conn_02x12_USBC_pins_shielded

Commit message: take snapshot
Parts:
- added H1: MountingHole_Pad, MountingHole:MountingHole_2.2mm_M2_Pad, F.Cu at (-108.5, -10.5)
- added H2: MountingHole_Pad, MountingHole:MountingHole_2.2mm_M2_Pad, F.Cu at (108.5, -10.5)
- added H3: MountingHole_Pad, MountingHole:MountingHole_2.2mm_M2_Pad, F.Cu at (-108.5, -2.50)
- added H4: MountingHole_Pad, MountingHole:MountingHole_2.2mm_M2_Pad, F.Cu at (108.5, -2.50)
- added J10: Conn_01x12, my_footprints:SAMTEC-MMS-112-02-X-SH-BRIDGE-PAD, F.Cu at (60.0, -5.92)
- added J11: Conn_01x04, Connector_PinSocket_2.00mm:PinSocket_1x04_P2.00mm_Vertical_SMD_Pin1Left, F.Cu at (89.0, -4.00)
- added J12: Conn_01x04, Connector_PinSocket_2.00mm:PinSocket_1x04_P2.00mm_Vertical_SMD_Pin1Left, F.Cu at (97.0, -4.00)
- added J7: Conn_01x12, my_footprints:SAMTEC-MMS-112-02-X-SH-BRIDGE-PAD, F.Cu at (-60.0, -5.92)
- added J8: Conn_01x12, my_footprints:SAMTEC-MMS-112-02-X-SH-BRIDGE-PAD, F.Cu at (-20.0, -5.92)
- added J9: Conn_01x12, my_footprints:SAMTEC-MMS-112-02-X-SH-BRIDGE-PAD, F.Cu at (20.0, -5.92)
- J1, J2, J3, J4: value Conn_02x12_USBC_pins -> Conn_02x04_Odd_Even; footprint my_footprints:PinSocket_2x12_P2.00mm_Vertical_EDGE_USBC_pins -> Connector_PinSocket_2.00mm:PinSocket_2x04_P2.00mm_Vertical_SMD; moved to B.Cu
- J5, J6: value Conn_02x12_USBC_pins_shielded -> Conn_01x04; footprint Connector_USB:USB_C_Receptacle_Amphenol_12401548E4-2A -> Connector_PinSocket_2.00mm:PinSocket_1x04_P2.00mm_Vertical_SMD_Pin1Left
- moved J5 264.2 mm to (-97.0, -4.00)
- moved J6 258.7 mm to (-89.0, -4.00)
- moved J2 156.0 mm to (-89.0, -5.00), turned to 270 degrees
- moved J1 134.3 mm to (-97.0, -5.00), turned to 270 degrees
- moved J4 37.5 mm to (97.0, -5.00), turned to 270 degrees
- moved J3 25.7 mm to (89.0, -5.00), turned to 270 degrees
Routing:
- net /C2B8: track 149.3 -> 0.00 mm, vias 2 -> 0
- net /C2B5: track 149.3 -> 0.00 mm, vias 2 -> 0
- net /C1B8: track 149.3 -> 0.00 mm, vias 2 -> 0
- net /C1B5: track 148.8 -> 0.00 mm, vias 1 -> 0
- net /C2B2: track 143.2 -> 0.00 mm, vias 1 -> 0
- net /C2B11: track 143.2 -> 0.00 mm, vias 1 -> 0
- net /C1B2: track 143.2 -> 0.00 mm, vias 1 -> 0
- net /C1B11: track 143.2 -> 0.00 mm, vias 1 -> 0
- net /C2B3: track 142.9 -> 0.00 mm, vias 1 -> 0
- net /C2B10: track 142.9 -> 0.00 mm, vias 1 -> 0
- net /C1B3: track 142.9 -> 0.00 mm, vias 1 -> 0
- net /C1B10: track 142.9 -> 0.00 mm, vias 1 -> 0
- net /C2B12: track 142.8 -> 0.00 mm, vias 1 -> 0
- net /C2B1: track 142.8 -> 0.00 mm, vias 1 -> 0
- net /C1B12: track 142.8 -> 0.00 mm, vias 1 -> 0
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- added copper zone on In1.Cu, net /C1A1
- added copper zone on In1.Cu, net /C1A10
- added copper zone on In1.Cu, net /C1A11
- added copper zone on In1.Cu, net /C1A12
- added copper zone on In1.Cu, net /C1A2
- added copper zone on In1.Cu, net /C1A3
- added copper zone on In1.Cu, net /C1A4
- added copper zone on In1.Cu, net /C1A5
- added copper zone on In1.Cu, net /C1A6
- added copper zone on In1.Cu, net /C1A7
- added copper zone on In1.Cu, net /C1A8
- added copper zone on In1.Cu, net /C1A9
Other:
- board size 150 x 35 mm -> 222 x 13.2 mm
- copper layers 6 -> 4
