File: adapter_spacer/adapter_spacer.kicad_pcb (KiCad board)
At the start: 2 copper layers, 184 x 48 mm, 32 parts

Commit message: update silk
Other:
- board text added: "98e55eb"
- board text removed: "COMMIT_HASH"
Changed lines of the file:
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@@
   (gr_arc (start 46 -14) (end 46 -16) (angle -90) (layer "Edge.Cuts") (width 0.05))
   (gr_arc (start -34 14) (end -36 14) (angle -90) (layer "Edge.Cuts") (width 0.05))
-  (gr_text "COMMIT_HASH" (at -80 -19 90) (layer "B.SilkS")
+  (gr_text "98e55eb" (at -80 -17 270) (layer "B.SilkS")
     (effects (font (size 1 1) (thickness 0.15)) (justify mirror))
   )
-  (gr_text "COMMIT_HASH" (at -80 -19 90) (layer "F.SilkS")
+  (gr_text "98e55eb" (at -80 -17 90) (layer "F.SilkS")
     (effects (font (size 1 1) (thickness 0.15)))
   )
