File: top/top.kicad_pcb (KiCad board)
At the start: 4 copper layers, 184 x 29.6 mm, 57 parts, among them J1 Conn_01x01, J10 Conn_01x01, J11 Conn_01x01, J12 Conn_01x01, J13 Conn_01x02, J14 Conn_01x02, J15 Conn_01x02, J16 Conn_01x02, J17 Conn_01x02, J18 Conn_01x02, J19 Conn_01x02, J2 Conn_01x01, J20 Conn_01x02, J29 Conn_01x01, J3 Conn_01x01, J30 Conn_01x01, J31 Conn_01x01, J32 Conn_01x01, J33 Conn_01x01, J34 Conn_01x01, J35 Conn_01x01, J36 Conn_01x01, J37 Conn_01x01, J38 Conn_01x01, J39 Conn_01x01, J4 Conn_01x01, J40 Conn_01x01, J5 Conn_01x01, J6 Conn_01x01, J7 Conn_01x01, J8 Conn_01x01, J9 Conn_01x01

Commit message: update silk
Other:
- board text added: "0dbcc89"
- board text removed: "98e55eb"
Changed lines of the file:
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@@
   (gr_line (start -92 14.799999) (end -92 -14.8) (layer "Edge.Cuts") (width 0.05))
   (gr_line (start 92 -14.799999) (end 92 14.8) (layer "Edge.Cuts") (width 0.05))
-  (gr_text "98e55eb" (at -89.5 6 270) (layer "B.SilkS")
+  (gr_text "0dbcc89" (at -89.5 6 270) (layer "B.SilkS")
     (effects (font (size 1 1) (thickness 0.15)) (justify mirror))
   )
-  (gr_text "98e55eb" (at -89.5 6 90) (layer "F.SilkS")
+  (gr_text "0dbcc89" (at -89.5 6 90) (layer "F.SilkS")
     (effects (font (size 1 1) (thickness 0.15)))
   )
