File: badger/badger.kicad_sch (KiCad schematic)
At the start: 93 parts, among them J1 Conn_01x01, J10 Conn_01x01, J11 Conn_01x01, J12 Conn_01x01, J13 Conn_01x01, J14 Conn_01x01, J15 Conn_01x01, J16 Conn_01x01, J17 Conn_01x01, J18 Conn_01x01, J19 Conn_01x01, J2 Conn_01x01, J20 Conn_01x01, J21 Conn_01x01, J22 Conn_01x01, J23 Conn_01x01, J24 Conn_01x01, J25 Conn_01x01, J26 Conn_01x01, J27 Conn_01x01, J28 Conn_01x01, J29 Conn_01x01, J3 Conn_01x01, J30 Conn_01x01, J31 Conn_01x01, J32 Conn_01x01, J33 Conn_01x01, J34 Conn_01x01, J35 Conn_01x01, J36 Conn_01x01, J37 Conn_01x01, J38 Conn_01x01, J39 Conn_01x01, J4 Conn_01x01, J40 Conn_01x01, J41 Conn_01x01, J42 Conn_01x01, J43 Conn_01x01, J44 Conn_01x01, J45 Conn_01x01, J46 Conn_01x01, J47 Conn_01x01, J48 Conn_01x01, J49 Conn_02x40_Odd_Even, J5 Conn_01x01, J50 Conn_01x01, J51 Conn_01x01, J52 Conn_01x01, J53 Conn_01x01, J54 Conn_01x01, J55 Conn_01x01, J56 Conn_01x01, J57 Conn_01x01, J58 Conn_01x01, J59 Conn_01x01, J6 Conn_01x01, J60 Conn_01x01, J61 Conn_01x01, J62 Conn_01x01, J63 Conn_01x01, J64 Conn_01x01, J65 Conn_01x01, J66 Conn_01x01, J67 Conn_01x01, J68 Conn_01x01, J69 Conn_01x01, J7 Conn_01x01, J70 Conn_01x01, J71 Conn_01x01, J72 Conn_01x01, J73 Conn_01x01, J74 Conn_01x01, J75 Conn_01x01, J76 Conn_01x01, J77 Conn_01x01, J78 Conn_01x01, J79 Conn_01x01, J8 Conn_01x01, J80 Conn_01x01, J81 Conn_01x01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

Commit message: badger upgrades
Parts:
- removed H12: MountingHole, MountingHole:MountingHole_6mm, symbol Mechanical:MountingHole
- removed J49: Conn_02x40_Odd_Even, Connector_PinHeader_2.54mm:PinHeader_2x40_P2.54mm_Vertical, symbol Connector_Generic:Conn_02x40_Odd_Even
- added J1, J2: Conn_02x20_Odd_Even, Connector_IDC:IDC-Header_2x20_P2.54mm_Horizontal, symbol Connector_Generic:Conn_02x20_Odd_Even
- renumbered J8 to J10, J9 to J11, J10 to J12, J11 to J13, J12 to J14, J13 to J15, J14 to J16, J15 to J17, J16 to J18, J17 to J19, J18 to J20, J19 to J21, J20 to J22, J21 to J23, J22 to J24, J23 to J25, J24 to J26, J25 to J27, J26 to J28, J27 to J29, J1 to J3, J28 to J30, J29 to J31, J30 to J32, J31 to J33, J32 to J34, J33 to J35, J34 to J36, J35 to J37, J36 to J38, J37 to J39, J2 to J4, J38 to J40, J39 to J41, J40 to J42, J41 to J43, J42 to J44, J43 to J45, J44 to J46, J45 to J47, J46 to J48, J47 to J49, J3 to J5, J48 to J50, J50 to J51, J51 to J52, J52 to J53, J53 to J54, J54 to J55, J55 to J56, J56 to J57, J57 to J58, J58 to J59, J4 to J6, J59 to J60, J60 to J61, J61 to J62, J62 to J63, J63 to J64, J64 to J65, J65 to J66, J66 to J67, J67 to J68, J68 to J69, J5 to J7, J69 to J70, J70 to J71, J71 to J72, J72 to J73, J73 to J74, J74 to J75, J75 to J76, J76 to J77, J77 to J78, J78 to J79, J6 to J8, J79 to J80, J80 to J81, J81 to J82, J7 to J9
Connections:
- net A_1: now also J1.1 (Pin_1)
- net A_10: now also J1.19 (Pin_19)
- net A_11: now also J1.21 (Pin_21)
- net A_12: now also J1.23 (Pin_23)
- net A_13: now also J1.25 (Pin_25)
- net A_14: now also J1.27 (Pin_27)
- net A_15: now also J1.29 (Pin_29)
- net A_16: now also J1.31 (Pin_31)
- net A_17: now also J1.33 (Pin_33)
- net A_18: now also J1.35 (Pin_35)
- net A_19: now also J1.37 (Pin_37)
- net A_2: now also J1.3 (Pin_3)
- net A_20: now also J1.39 (Pin_39)
- net A_3: now also J1.5 (Pin_5)
- net A_4: now also J1.7 (Pin_7)
- net A_5: now also J1.9 (Pin_9)
- net A_6: now also J1.11 (Pin_11)
- net A_7: now also J1.13 (Pin_13)
- net A_8: now also J1.15 (Pin_15)
- net A_9: now also J1.17 (Pin_17)
- net B_1: now also J2.1 (Pin_1)
- net B_10: now also J2.19 (Pin_19)
- net B_11: now also J2.21 (Pin_21)
- net B_12: now also J2.23 (Pin_23)
- net B_13: now also J2.25 (Pin_25)
- net B_14: now also J2.27 (Pin_27)
- net B_15: now also J2.29 (Pin_29)
- net B_16: now also J2.31 (Pin_31)
- net B_17: now also J2.33 (Pin_33)
- net B_18: now also J2.35 (Pin_35)
- net B_19: now also J2.37 (Pin_37)
- net B_2: now also J2.3 (Pin_3)
- net B_20: now also J2.39 (Pin_39)
- net B_3: now also J2.5 (Pin_5)
- net B_4: now also J2.7 (Pin_7)
- net B_5: now also J2.9 (Pin_9)
- net B_6: now also J2.11 (Pin_11)
- net B_7: now also J2.13 (Pin_13)
- net B_8: now also J2.15 (Pin_15)
- net B_9: now also J2.17 (Pin_17)
- net C_1: now also J1.2 (Pin_2)
- net C_10: now also J1.20 (Pin_20)
- net C_11: now also J1.22 (Pin_22)
- net C_12: now also J1.24 (Pin_24)
- net C_13: now also J1.26 (Pin_26)
- net C_14: now also J1.28 (Pin_28)
- net C_15: now also J1.30 (Pin_30)
- net C_16: now also J1.32 (Pin_32)
- net C_17: now also J1.34 (Pin_34)
- net C_18: now also J1.36 (Pin_36)
- net C_19: now also J1.38 (Pin_38)
- net C_2: now also J1.4 (Pin_4)
- net C_20: now also J1.40 (Pin_40)
- net C_3: now also J1.6 (Pin_6)
- net C_4: now also J1.8 (Pin_8)
- net C_5: now also J1.10 (Pin_10)
- net C_6: now also J1.12 (Pin_12)
- net C_7: now also J1.14 (Pin_14)
- net C_8: now also J1.16 (Pin_16)
- net C_9: now also J1.18 (Pin_18)
- net D_1: now also J2.2 (Pin_2)
- net D_10: now also J2.20 (Pin_20)
- net D_11: now also J2.22 (Pin_22)
- net D_12: now also J2.24 (Pin_24)
- net D_13: now also J2.26 (Pin_26)
- net D_14: now also J2.28 (Pin_28)
- net D_15: now also J2.30 (Pin_30)
- net D_16: now also J2.32 (Pin_32)
- net D_17: now also J2.34 (Pin_34)
- net D_18: now also J2.36 (Pin_36)
- net D_19: now also J2.38 (Pin_38)
- net D_2: now also J2.4 (Pin_4)
- net D_20: now also J2.40 (Pin_40)
- net D_3: now also J2.6 (Pin_6)
- net D_4: now also J2.8 (Pin_8)
- net D_5: now also J2.10 (Pin_10)
- net D_6: now also J2.12 (Pin_12)
- net D_7: now also J2.14 (Pin_14)
- net D_8: now also J2.16 (Pin_16)
- net D_9: now also J2.18 (Pin_18)

Commit message: crossbar redesign to get linear trace highway
Parts:
- removed H1, H10, H11, H2, H3, H4, H5, H6, H7, H8, H9: MountingHole, MountingHole:MountingHole_6mm, symbol Mechanical:MountingHole
Changed lines of the file:
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@@
     (effects (font (size 1.27 1.27)) (justify left bottom))
-  )
-  (symbol (lib_id "Mechanical:MountingHole") (at 25.4 38.1 0) (unit 1)
-    (in_bom yes) (on_board yes)
-    (property "Reference" "H1" (id 0) (at 29.21 36.83 0)
-      (effects (font (size 1.27 1.27)) (justify left))
-    )
-    (property "Value" "MountingHole" (id 1) (at 29.21 39.37 0)
-      (effects (font (size 1.27 1.27)) (justify left))
-    )
-    (property "Footprint" "MountingHole:MountingHole_6mm" (id 2) (at 25.4 38.1 0)
-      (effects (font (size 1.27 1.27)) hide)
-    )
-    (property "Datasheet" "~" (id 3) (at 25.4 38.1 0)
-      (effects (font (size 1.27 1.27)) hide)
-    )
-  )
-  (symbol (lib_id "Mechanical:MountingHole") (at 25.4 50.8 0) (unit 1)
-    (in_bom yes) (on_board yes)
-    (property "Reference" "H2" (id 0) (at 29.21 49.53 0)
-      (effects (font (size 1.27 1.27)) (justify left))
-    )
-    (property "Value" "MountingHole" (id 1) (at 29.21 52.07 0)
-      (effects (font (size 1.27 1.27)) (justify left))
-    )
-    (property "Footprint" "MountingHole:MountingHole_6mm" (id 2) (at 25.4 50.8 0)
-      (effects (font (size 1.27 1.27)) hide)
-    )
-    (property "Datasheet" "~" (id 3) (at 25.4 50.8 0)
-      (effects (font (size 1.27 1.27)) hide)
-    )
-  )
-  (symbol (lib_id "Mechanical:MountingHole") (at 25.4 63.5 0) (unit 1)
-    (in_bom yes) (on_board yes)
-    (property "Reference" "H3" (id 0) (at 29.21 62.23 0)
-      (effects (font (size 1.27 1.27)) (justify left))
-    )
-    (property "Value" "MountingHole" (id 1) (at 29.21 64.77 0)
-      (effects (font (size 1.27 1.27)) (justify left))
-    )
-    (property "Footprint" "MountingHole:MountingHole_6mm" (id 2) (at 25.4 63.5 0)
-      (effects (font (size 1.27 1.27)) hide)
-    )
-    (property "Datasheet" "~" (id 3) (at 25.4 63.5 0)
-      (effects (font (size 1.27 1.27)) hide)
-    )
-  )
-  (symbol (lib_id "Mechanical:MountingHole") (at 25.4 76.2 0) (unit 1)
-    (in_bom yes) (on_board yes)
-    (property "Reference" "H4" (id 0) (at 29.21 74.93 0)
-      (effects (font (size 1.27 1.27)) (justify left))
-    )
-    (property "Value" "MountingHole" (id 1) (at 29.21 77.47 0)
-      (effects (font (size 1.27 1.27)) (justify left))
-    )
-    (property "Footprint" "MountingHole:MountingHole_6mm" (id 2) (at 25.4 76.2 0)
-      (effects (font (size 1.27 1.27)) hide)
-    )
-    (property "Datasheet" "~" (id 3) (at 25.4 76.2 0)
-      (effects (font (size 1.27 1.27)) hide)
-    )
-  )
-  (symbol (lib_id "Mechanical:MountingHole") (at 25.4 88.9 0) (unit 1)
-    (in_bom yes) (on_board yes)
-    (property "Reference" "H5" (id 0) (at 29.21 87.63 0)
-      (effects (font (size 1.27 1.27)) (justify left))
-    )
-    (property "Value" "MountingHole" (id 1) (at 29.21 90.17 0)
-      (effects (font (size 1.27 1.27)) (justify left))
-    )
-    (property "Footprint" "MountingHole:MountingHole_6mm" (id 2) (at 25.4 88.9 0)
-      (effects (font (size 1.27 1.27)) hide)
-    )
-    (property "Datasheet" "~" (id 3) (at 25.4 88.9 0)
-      (effects (font (size 1.27 1.27)) hide)
-    )
-  )
-  (symbol (lib_id "Mechanical:MountingHole") (at 25.4 101.6 0) (unit 1)
-    (in_bom yes) (on_board yes)
-    (property "Reference" "H6" (id 0) (at 29.21 100.33 0)
-      (effects (font (size 1.27 1.27)) (justify left))
-    )
-    (property "Value" "MountingHole" (id 1) (at 29.21 102.87 0)
-      (effects (font (size 1.27 1.27)) (justify left))
-    )
-    (property "Footprint" "MountingHole:MountingHole_6mm" (id 2) (at 25.4 101.6 0)
-      (effects (font (size 1.27 1.27)) hide)
-    )
-    (property "Datasheet" "~" (id 3) (at 25.4 101.6 0)
-      (effects (font (size 1.27 1.27)) hide)
-    )
-  )
-  (symbol (lib_id "Mechanical:MountingHole") (at 25.4 114.3 0) (unit 1)
-    (in_bom yes) (on_board yes)
-    (property "Reference" "H7" (id 0) (at 29.21 113.03 0)
-      (effects (font (size 1.27 1.27)) (justify left))
-    )
-    (property "Value" "MountingHole" (id 1) (at 29.21 115.57 0)
-      (effects (font (size 1.27 1.27)) (justify left))
-    )
-    (property "Footprint" "MountingHole:MountingHole_6mm" (id 2) (at 25.4 114.3 0)
-      (effects (font (size 1.27 1.27)) hide)
-    )
-    (property "Datasheet" "~" (id 3) (at 25.4 114.3 0)
-      (effects (font (size 1.27 1.27)) hide)
-    )
-  )
-  (symbol (lib_id "Mechanical:MountingHole") (at 25.4 127 0) (unit 1)
-    (in_bom yes) (on_board yes)
-    (property "Reference" "H8" (id 0) (at 29.21 125.73 0)
-      (effects (font (size 1.27 1.27)) (justify left))
-    )
-    (property "Value" "MountingHole" (id 1) (at 29.21 128.27 0)
-      (effects (font (size 1.27 1.27)) (justify left))
-    )
-    (property "Footprint" "MountingHole:MountingHole_6mm" (id 2) (at 25.4 127 0)
-      (effects (font (size 1.27 1.27)) hide)
-    )
-    (property "Datasheet" "~" (id 3) (at 25.4 127 0)
-      (effects (font (size 1.27 1.27)) hide)
-    )
-  )
-  (symbol (lib_id "Mechanical:MountingHole") (at 25.4 139.7 0) (unit 1)
-    (in_bom yes) (on_board yes)
-    (property "Reference" "H9" (id 0) (at 29.21 138.43 0)
-      (effects (font (size 1.27 1.27)) (justify left))
-    )
-    (property "Value" "MountingHole" (id 1) (at 29.21 140.97 0)
-      (effects (font (size 1.27 1.27)) (justify left))
-    )
-    (property "Footprint" "MountingHole:MountingHole_6mm" (id 2) (at 25.4 139.7 0)
-      (effects (font (size 1.27 1.27)) hide)
-    )
-    (property "Datasheet" "~" (id 3) (at 25.4 139.7 0)
-      (effects (font (size 1.27 1.27)) hide)
-    )
-  )
-  (symbol (lib_id "Mechanical:MountingHole") (at 25.4 152.4 0) (unit 1)
-    (in_bom yes) (on_board yes)
-    (property "Reference" "H10" (id 0) (at 29.21 151.13 0)
-      (effects (font (size 1.27 1.27)) (justify left))
-    )
-    (property "Value" "MountingHole" (id 1) (at 29.21 153.67 0)
-      (effects (font (size 1.27 1.27)) (justify left))
-    )
-    (property "Footprint" "MountingHole:MountingHole_6mm" (id 2) (at 25.4 152.4 0)
-      (effects (font (size 1.27 1.27)) hide)
-    )
-    (property "Datasheet" "~" (id 3) (at 25.4 152.4 0)
-      (effects (font (size 1.27 1.27)) hide)
-    )
-  )
-  (symbol (lib_id "Mechanical:MountingHole") (at 25.4 165.1 0) (unit 1)
-    (in_bom yes) (on_board yes)
-    (property "Reference" "H11" (id 0) (at 29.21 163.83 0)
-      (effects (font (size 1.27 1.27)) (justify left))
-    )
-    (property "Value" "MountingHole" (id 1) (at 29.21 166.37 0)
-      (effects (font (size 1.27 1.27)) (justify left))
-    )
-    (property "Footprint" "MountingHole:MountingHole_6mm" (id 2) (at 25.4 165.1 0)
-      (effects (font (size 1.27 1.27)) hide)
-    )
-    (property "Datasheet" "~" (id 3) (at 25.4 165.1 0)
-      (effects (font (size 1.27 1.27)) hide)
-    )
   )
   (symbol (lib_id "Connector_Generic:Conn_01x01") (at 166.37 34.29 270) (unit 1)
@@
   )
   (symbol_instances
-    (path "/30d0d661-b0df-4f3b-9ea4-d4cf2dbd99b9"
-      (reference "H1") (unit 1) (value "MountingHole") (footprint "MountingHole:MountingHole_6mm")
-    )
-    (path "/3b9718ce-75c4-4c2c-a511-11906b2070a5"
-      (reference "H2") (unit 1) (value "MountingHole") (footprint "MountingHole:MountingHole_6mm")
-    )
-    (path "/2fffdaae-3384-45aa-a2da-d20be2d3ae43"
-      (reference "H3") (unit 1) (value "MountingHole") (footprint "MountingHole:MountingHole_6mm")
-    )
-    (path "/95847b94-2731-418a-9170-cff84cfc20df"
-      (reference "H4") (unit 1) (value "MountingHole") (footprint "MountingHole:MountingHole_6mm")
-    )
-    (path "/40763a08-81e0-4f6c-9bbb-51f516b989b8"
-      (reference "H5") (unit 1) (value "MountingHole") (footprint "MountingHole:MountingHole_6mm")
-    )
-    (path "/3f87c5a0-bbe3-452b-948d-84f683ea3444"
-      (reference "H6") (unit 1) (value "MountingHole") (footprint "MountingHole:MountingHole_6mm")
-    )
-    (path "/a80b7f6f-c725-49a5-99ff-3c03c3fd9cca"
-      (reference "H7") (unit 1) (value "MountingHole") (footprint "MountingHole:MountingHole_6mm")
-    )
-    (path "/65415b96-c801-4012-8fe7-a59a744a9f73"
-      (reference "H8") (unit 1) (value "MountingHole") (footprint "MountingHole:MountingHole_6mm")
-    )
-    (path "/8d91f80d-e7b5-4fff-8e91-b555993ee8dc"
-      (reference "H9") (unit 1) (value "MountingHole") (footprint "MountingHole:MountingHole_6mm")
-    )
-    (path "/29be1cfb-8bd5-4fba-9791-2441f45370df"
-      (reference "H10") (unit 1) (value "MountingHole") (footprint "MountingHole:MountingHole_6mm")
-    )
-    (path "/ea40bb38-cddf-4832-ba48-780be24421c0"
-      (reference "H11") (unit 1) (value "MountingHole") (footprint "MountingHole:MountingHole_6mm")
-    )
     (path "/1ee9073d-68d1-4212-927d-832096d21277"
       (reference "J1") (unit 1) (value "Conn_02x20_Odd_Even") (footprint "Connector_IDC:IDC-Header_2x20_P2.54mm_Horizontal")

Commit message: wip on 4x1 crossbar
Parts:
- J1, J2: footprint Connector_IDC:IDC-Header_2x20_P2.54mm_Horizontal -> MINE:HTSS-120-04-G-D-RA
- J10, J11, J12, J13, J14, J15, J16, J17, J18, J19, J20, J21, J22, J23, J24, J25, J26, J27, J28, J29, J3, J30, J31, J32, J33, J34, J35, J36, J37, J38, J39, J4, J40, J41, J42, J43, J44, J45, J46, J47, J48, J49, J5, J50, J51, J52, J53, J54, J55, J56, J57, J58, J59, J6, J60, J61, J62, J63, J64, J65, J66, J67, J68, J69, J7, J70, J71, J72, J73, J74, J75, J76, J77, J78, J79, J8, J80, J81, J82, J9: footprint MINE:low_profile_spring_pin -> MINE:0921

Commit message: new otter and badger boards done
Parts:
- added H1, H2: MountingHole, MINE:MountingHole_7.1mm, symbol Mechanical:MountingHole
- added LOGO1, LOGO2: Logo_Open_Hardware_Small, MINE:site_small, symbol Graphic:Logo_Open_Hardware_Small
Connections:
- net A_1: now also J1.39 (Pin_39), J15.1 (Pin_1); no longer J1.1 (Pin_1), J3.1 (Pin_1)
- net A_10: now also J1.21 (Pin_21), J43.1 (Pin_1); no longer J1.19 (Pin_19), J39.1 (Pin_1)
- net A_11: now also J1.19 (Pin_19), J39.1 (Pin_1); no longer J1.21 (Pin_21), J43.1 (Pin_1)
- net A_12: now also J1.17 (Pin_17), J35.1 (Pin_1); no longer J1.23 (Pin_23), J47.1 (Pin_1)
- net A_13: now also J1.15 (Pin_15), J63.1 (Pin_1); no longer J1.25 (Pin_25), J51.1 (Pin_1)
- net A_14: now also J1.13 (Pin_13), J59.1 (Pin_1); no longer J1.27 (Pin_27), J55.1 (Pin_1)
- net A_15: now also J1.11 (Pin_11), J55.1 (Pin_1); no longer J1.29 (Pin_29), J59.1 (Pin_1)
- net A_16: now also J1.9 (Pin_9), J51.1 (Pin_1); no longer J1.31 (Pin_31), J63.1 (Pin_1)
- net A_17: now also J1.7 (Pin_7), J79.1 (Pin_1); no longer J1.33 (Pin_33), J67.1 (Pin_1)
- net A_18: now also J1.5 (Pin_5), J75.1 (Pin_1); no longer J1.35 (Pin_35), J71.1 (Pin_1)
- net A_19: now also J1.3 (Pin_3), J71.1 (Pin_1); no longer J1.37 (Pin_37), J75.1 (Pin_1)
- net A_2: now also J1.37 (Pin_37), J11.1 (Pin_1); no longer J1.3 (Pin_3), J7.1 (Pin_1)
- net A_20: now also J1.1 (Pin_1), J67.1 (Pin_1); no longer J1.39 (Pin_39), J79.1 (Pin_1)
- net A_3: now also J1.35 (Pin_35), J7.1 (Pin_1); no longer J1.5 (Pin_5), J11.1 (Pin_1)
- net A_4: now also J1.33 (Pin_33), J3.1 (Pin_1); no longer J1.7 (Pin_7), J15.1 (Pin_1)
- net A_5: now also J1.31 (Pin_31), J31.1 (Pin_1); no longer J1.9 (Pin_9), J19.1 (Pin_1)
- net A_6: now also J1.29 (Pin_29), J27.1 (Pin_1); no longer J1.11 (Pin_11), J23.1 (Pin_1)
- net A_7: now also J1.27 (Pin_27), J23.1 (Pin_1); no longer J1.13 (Pin_13), J27.1 (Pin_1)
- net A_8: now also J1.25 (Pin_25), J19.1 (Pin_1); no longer J1.15 (Pin_15), J31.1 (Pin_1)
- net A_9: now also J1.23 (Pin_23), J47.1 (Pin_1); no longer J1.17 (Pin_17), J35.1 (Pin_1)
- net B_1: now also J16.1 (Pin_1), J2.39 (Pin_39); no longer J2.1 (Pin_1), J4.1 (Pin_1)
- net B_10: now also J2.21 (Pin_21), J44.1 (Pin_1); no longer J2.19 (Pin_19), J40.1 (Pin_1)
- net B_11: now also J2.19 (Pin_19), J40.1 (Pin_1); no longer J2.21 (Pin_21), J44.1 (Pin_1)
- net B_12: now also J2.17 (Pin_17), J36.1 (Pin_1); no longer J2.23 (Pin_23), J48.1 (Pin_1)
- net B_13: now also J2.15 (Pin_15), J64.1 (Pin_1); no longer J2.25 (Pin_25), J52.1 (Pin_1)
- net B_14: now also J2.13 (Pin_13), J60.1 (Pin_1); no longer J2.27 (Pin_27), J56.1 (Pin_1)
- net B_15: now also J2.11 (Pin_11), J56.1 (Pin_1); no longer J2.29 (Pin_29), J60.1 (Pin_1)
- net B_16: now also J2.9 (Pin_9), J52.1 (Pin_1); no longer J2.31 (Pin_31), J64.1 (Pin_1)
- net B_17: now also J2.7 (Pin_7), J80.1 (Pin_1); no longer J2.33 (Pin_33), J68.1 (Pin_1)
- net B_18: now also J2.5 (Pin_5), J76.1 (Pin_1); no longer J2.35 (Pin_35), J72.1 (Pin_1)
- net B_19: now also J2.3 (Pin_3), J72.1 (Pin_1); no longer J2.37 (Pin_37), J76.1 (Pin_1)
- net B_2: now also J12.1 (Pin_1), J2.37 (Pin_37); no longer J2.3 (Pin_3), J8.1 (Pin_1)
- net B_20: now also J2.1 (Pin_1), J68.1 (Pin_1); no longer J2.39 (Pin_39), J80.1 (Pin_1)
- net B_3: now also J2.35 (Pin_35), J8.1 (Pin_1); no longer J12.1 (Pin_1), J2.5 (Pin_5)
- net B_4: now also J2.33 (Pin_33), J4.1 (Pin_1); no longer J16.1 (Pin_1), J2.7 (Pin_7)
- net B_5: now also J2.31 (Pin_31), J32.1 (Pin_1); no longer J2.9 (Pin_9), J20.1 (Pin_1)
- net B_6: now also J2.29 (Pin_29), J28.1 (Pin_1); no longer J2.11 (Pin_11), J24.1 (Pin_1)
- net B_7: now also J2.27 (Pin_27), J24.1 (Pin_1); no longer J2.13 (Pin_13), J28.1 (Pin_1)
- net B_8: now also J2.25 (Pin_25), J20.1 (Pin_1); no longer J2.15 (Pin_15), J32.1 (Pin_1)
- net B_9: now also J2.23 (Pin_23), J48.1 (Pin_1); no longer J2.17 (Pin_17), J36.1 (Pin_1)
- net C_1: now also J1.40 (Pin_40), J17.1 (Pin_1); no longer J1.2 (Pin_2), J5.1 (Pin_1)
- net C_10: now also J1.22 (Pin_22), J45.1 (Pin_1); no longer J1.20 (Pin_20), J41.1 (Pin_1)
- net C_11: now also J1.20 (Pin_20), J41.1 (Pin_1); no longer J1.22 (Pin_22), J45.1 (Pin_1)
- net C_12: now also J1.18 (Pin_18), J37.1 (Pin_1); no longer J1.24 (Pin_24), J49.1 (Pin_1)
- net C_13: now also J1.16 (Pin_16), J65.1 (Pin_1); no longer J1.26 (Pin_26), J53.1 (Pin_1)
- net C_14: now also J1.14 (Pin_14), J61.1 (Pin_1); no longer J1.28 (Pin_28), J57.1 (Pin_1)
- net C_15: now also J1.12 (Pin_12), J57.1 (Pin_1); no longer J1.30 (Pin_30), J61.1 (Pin_1)
- net C_16: now also J1.10 (Pin_10), J53.1 (Pin_1); no longer J1.32 (Pin_32), J65.1 (Pin_1)
- net C_17: now also J1.8 (Pin_8), J81.1 (Pin_1); no longer J1.34 (Pin_34), J69.1 (Pin_1)
- net C_18: now also J1.6 (Pin_6), J77.1 (Pin_1); no longer J1.36 (Pin_36), J73.1 (Pin_1)
- net C_19: now also J1.4 (Pin_4), J73.1 (Pin_1); no longer J1.38 (Pin_38), J77.1 (Pin_1)
- net C_2: now also J1.38 (Pin_38), J13.1 (Pin_1); no longer J1.4 (Pin_4), J9.1 (Pin_1)
- net C_20: now also J1.2 (Pin_2), J69.1 (Pin_1); no longer J1.40 (Pin_40), J81.1 (Pin_1)
- net C_3: now also J1.36 (Pin_36), J9.1 (Pin_1); no longer J1.6 (Pin_6), J13.1 (Pin_1)
- net C_4: now also J1.34 (Pin_34), J5.1 (Pin_1); no longer J1.8 (Pin_8), J17.1 (Pin_1)
- net C_5: now also J1.32 (Pin_32), J33.1 (Pin_1); no longer J1.10 (Pin_10), J21.1 (Pin_1)
- net C_6: now also J1.30 (Pin_30), J29.1 (Pin_1); no longer J1.12 (Pin_12), J25.1 (Pin_1)
- net C_7: now also J1.28 (Pin_28), J25.1 (Pin_1); no longer J1.14 (Pin_14), J29.1 (Pin_1)
- net C_8: now also J1.26 (Pin_26), J21.1 (Pin_1); no longer J1.16 (Pin_16), J33.1 (Pin_1)
- net C_9: now also J1.24 (Pin_24), J49.1 (Pin_1); no longer J1.18 (Pin_18), J37.1 (Pin_1)
- net D_1: now also J18.1 (Pin_1), J2.40 (Pin_40); no longer J2.2 (Pin_2), J6.1 (Pin_1)
- net D_10: now also J2.22 (Pin_22), J46.1 (Pin_1); no longer J2.20 (Pin_20), J42.1 (Pin_1)
- net D_11: now also J2.20 (Pin_20), J42.1 (Pin_1); no longer J2.22 (Pin_22), J46.1 (Pin_1)
- net D_12: now also J2.18 (Pin_18), J38.1 (Pin_1); no longer J2.24 (Pin_24), J50.1 (Pin_1)
- net D_13: now also J2.16 (Pin_16), J66.1 (Pin_1); no longer J2.26 (Pin_26), J54.1 (Pin_1)
- net D_14: now also J2.14 (Pin_14), J62.1 (Pin_1); no longer J2.28 (Pin_28), J58.1 (Pin_1)
- net D_15: now also J2.12 (Pin_12), J58.1 (Pin_1); no longer J2.30 (Pin_30), J62.1 (Pin_1)
- net D_16: now also J2.10 (Pin_10), J54.1 (Pin_1); no longer J2.32 (Pin_32), J66.1 (Pin_1)
- net D_17: now also J2.8 (Pin_8), J82.1 (Pin_1); no longer J2.34 (Pin_34), J70.1 (Pin_1)
- net D_18: now also J2.6 (Pin_6), J78.1 (Pin_1); no longer J2.36 (Pin_36), J74.1 (Pin_1)
- net D_19: now also J2.4 (Pin_4), J74.1 (Pin_1); no longer J2.38 (Pin_38), J78.1 (Pin_1)
- net D_2: now also J14.1 (Pin_1), J2.38 (Pin_38); no longer J10.1 (Pin_1), J2.4 (Pin_4)
- net D_20: now also J2.2 (Pin_2), J70.1 (Pin_1); no longer J2.40 (Pin_40), J82.1 (Pin_1)
- net D_3: now also J10.1 (Pin_1), J2.36 (Pin_36); no longer J14.1 (Pin_1), J2.6 (Pin_6)
- net D_4: now also J2.34 (Pin_34), J6.1 (Pin_1); no longer J18.1 (Pin_1), J2.8 (Pin_8)
- net D_5: now also J2.32 (Pin_32), J34.1 (Pin_1); no longer J2.10 (Pin_10), J22.1 (Pin_1)
- net D_6: now also J2.30 (Pin_30), J30.1 (Pin_1); no longer J2.12 (Pin_12), J26.1 (Pin_1)
- net D_7: now also J2.28 (Pin_28), J26.1 (Pin_1); no longer J2.14 (Pin_14), J30.1 (Pin_1)
- net D_8: now also J2.26 (Pin_26), J22.1 (Pin_1); no longer J2.16 (Pin_16), J34.1 (Pin_1)
- net D_9: now also J2.24 (Pin_24), J50.1 (Pin_1); no longer J2.18 (Pin_18), J38.1 (Pin_1)
Other:
- moved on the sheet: J1, J10, J11, J12, J13, J14, J15, J16, J17, J18, J19, J2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
