File: badger/badger.kicad_pcb (KiCad board)
At the start: 2 copper layers, 200 x 200 mm, 93 parts, among them J1 Conn_01x01, J10 Conn_01x01, J11 Conn_01x01, J12 Conn_01x01, J13 Conn_01x01, J14 Conn_01x01, J15 Conn_01x01, J16 Conn_01x01, J17 Conn_01x01, J18 Conn_01x01, J19 Conn_01x01, J2 Conn_01x01, J20 Conn_01x01, J21 Conn_01x01, J22 Conn_01x01, J23 Conn_01x01, J24 Conn_01x01, J25 Conn_01x01, J26 Conn_01x01, J27 Conn_01x01, J28 Conn_01x01, J29 Conn_01x01, J3 Conn_01x01, J30 Conn_01x01, J31 Conn_01x01, J32 Conn_01x01, J33 Conn_01x01, J34 Conn_01x01, J35 Conn_01x01, J36 Conn_01x01, J37 Conn_01x01, J38 Conn_01x01, J39 Conn_01x01, J4 Conn_01x01, J40 Conn_01x01, J41 Conn_01x01, J42 Conn_01x01, J43 Conn_01x01, J44 Conn_01x01, J45 Conn_01x01, J46 Conn_01x01, J47 Conn_01x01, J48 Conn_01x01, J49 Conn_02x40_Odd_Even, J5 Conn_01x01, J50 Conn_01x01, J51 Conn_01x01, J52 Conn_01x01, J53 Conn_01x01, J54 Conn_01x01, J55 Conn_01x01, J56 Conn_01x01, J57 Conn_01x01, J58 Conn_01x01, J59 Conn_01x01, J6 Conn_01x01, J60 Conn_01x01, J61 Conn_01x01, J62 Conn_01x01, J63 Conn_01x01, J64 Conn_01x01, J65 Conn_01x01, J66 Conn_01x01, J67 Conn_01x01, J68 Conn_01x01, J69 Conn_01x01, J7 Conn_01x01, J70 Conn_01x01, J71 Conn_01x01, J72 Conn_01x01, J73 Conn_01x01, J74 Conn_01x01, J75 Conn_01x01, J76 Conn_01x01, J77 Conn_01x01, J78 Conn_01x01, J79 Conn_01x01, J8 Conn_01x01, J80 Conn_01x01, J81 Conn_01x01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

Commit message: badger upgrades
Parts:
- removed H12: MountingHole, MountingHole:MountingHole_6mm
- removed the J49 at (-83.3, -49.5)
- added J1: Conn_02x20_Odd_Even, Connector_IDC:IDC-Header_2x20_P2.54mm_Horizontal, F.Cu at (-66.8, -22.4)
- added J2: Conn_02x20_Odd_Even, Connector_IDC:IDC-Header_2x20_P2.54mm_Horizontal, F.Cu at (-66.8, 70.6)
- moved H11 31.7 mm to (-93.0, 0.00)
- moved J10 10.0 mm to (-6.00, -69.0)
- moved J11 10.0 mm to (29.0, -69.0)
- moved J12 10.0 mm to (19.5, -69.0)
- moved J13 10.0 mm to (26.0, -69.0)
- moved J14 10.0 mm to (51.5, 47.0)
- moved J15 10.0 mm to (29.0, 47.0)
- moved J16 10.0 mm to (54.5, 47.0)
- moved J17 10.0 mm to (16.5, -40.0)
- moved J18 10.0 mm to (29.0, 18.0)
- moved J19 10.0 mm to (29.0, -11.0)
- moved J20 10.0 mm to (-18.5, -40.0)
- moved J21 10.0 mm to (26.0, -40.0)
- moved J22 10.0 mm to (51.5, -11.0)
- moved J23 10.0 mm to (-41.0, -40.0)
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- renumbered J8 to J10, J9 to J11, J10 to J12, J11 to J13, J12 to J14, J13 to J15, J14 to J16, J15 to J17, J16 to J18, J17 to J19, J18 to J20, J19 to J21, J20 to J22, J21 to J23, J22 to J24, J23 to J25, J24 to J26, J25 to J27, J26 to J28, J27 to J29, J1 to J3, J28 to J30, J29 to J31, J30 to J32, J31 to J33, J32 to J34, J33 to J35, J34 to J36, J35 to J37, J36 to J38, J37 to J39, J2 to J4, J38 to J40, J39 to J41, J40 to J42, J41 to J43, J42 to J44, J43 to J45, J44 to J46, J45 to J47, J46 to J48, J47 to J49, J3 to J5, J48 to J50, J50 to J51, J51 to J52, J52 to J53, J53 to J54, J54 to J55, J55 to J56, J56 to J57, J57 to J58, J58 to J59, J4 to J6, J59 to J60, J60 to J61, J61 to J62, J62 to J63, J63 to J64, J64 to J65, J65 to J66, J66 to J67, J67 to J68, J68 to J69, J5 to J7, J69 to J70, J70 to J71, J71 to J72, J72 to J73, J73 to J74, J74 to J75, J75 to J76, J76 to J77, J77 to J78, J78 to J79, J6 to J8, J79 to J80, J80 to J81, J81 to J82, J7 to J9
Other:
- outline, holes or cut-outs redrawn

Commit message: crossbar redesign to get linear trace highway
Parts:
- removed H1, H10, H11, H2, H3, H4, H5, H6, H7, H8, H9: MountingHole, MountingHole:MountingHole_6mm
Other:
- board size 200 x 200 mm -> 172 x 172 mm

Commit message: wip on 4x1 crossbar
Parts:
- J1, J2: footprint Connector_IDC:IDC-Header_2x20_P2.54mm_Horizontal -> MINE:HTSS-120-04-G-D-RA
- J10, J11, J12, J13, J14, J15, J16, J17, J18, J19, J20, J21, J22, J23, J24, J25, J26, J27, J28, J29, J3, J30, J31, J32, J33, J34, J35, J36, J37, J38, J39, J4, J40, J41, J42, J43, J44, J45, J46, J47, J48, J49, J5, J50, J51, J52, J53, J54, J55, J56, J57, J58, J59, J6, J60, J61, J62, J63, J64, J65, J66, J67, J68, J69, J7, J70, J71, J72, J73, J74, J75, J76, J77, J78, J79, J8, J80, J81, J82, J9: footprint MINE:low_profile_spring_pin -> MINE:0921

Commit message: new otter and badger boards done
Parts:
- added H1: MountingHole, MINE:MountingHole_7.1mm, F.Cu at (0.00, -80.0)
- added H2: MountingHole, MINE:MountingHole_7.1mm, F.Cu at (20.0, 80.0)
- added LOGO1: Logo_Open_Hardware_Small, MINE:site_small, B.Cu at (-82.0, -56.7)
- added LOGO2: Logo_Open_Hardware_Small, MINE:site_small, F.Cu at (-82.0, -56.7)
- renumbered J25 to J11, J11 to J14, J55 to J15, J41 to J16, J78 to J17, J81 to J18, J61 to J19, J75 to J20, J46 to J21, J23 to J22, J20 to J23, J53 to J24, J59 to J25, J48 to J26, J17 to J27, J69 to J28, J21 to J29, J54 to J30, J35 to J31, J80 to J32, J29 to J33, J37 to J34, J51 to J35, J66 to J36, J43 to J37, J60 to J38, J30 to J40, J33 to J41, J77 to J42, J58 to J43, J74 to J44, J28 to J45, J19 to J46, J22 to J47, J65 to J48, J79 to J49, J49 to J50, J57 to J51, J36 to J52, J64 to J53, J31 to J54, J42 to J55, J27 to J56, J52 to J57, J44 to J58, J40 to J59, J63 to J60, J76 to J61, J18 to J62, J45 to J63, J82 to J64, J67 to J65, J34 to J66, J32 to J67, J62 to J68, J50 to J69, J47 to J70, J70 to J71, J68 to J74, J71 to J75, J26 to J76, J38 to J77, J15 to J78, J14 to J79, J16 to J80, J56 to J81, J24 to J82
Connections:
- J1 pad 1: /A_1 -> /A_20
- J1 pad 10: /C_5 -> /C_16
- J1 pad 11: /A_6 -> /A_15
- J1 pad 12: /C_6 -> /C_15
- J1 pad 13: /A_7 -> /A_14
- J1 pad 14: /C_7 -> /C_14
- J1 pad 15: /A_8 -> /A_13
- J1 pad 16: /C_8 -> /C_13
- J1 pad 17: /A_9 -> /A_12
- J1 pad 18: /C_9 -> /C_12
- J1 pad 19: /A_10 -> /A_11
- J1 pad 2: /C_1 -> /C_20
- J1 pad 20: /C_10 -> /C_11
- J1 pad 21: /A_11 -> /A_10
- J1 pad 22: /C_11 -> /C_10
- J1 pad 23: /A_12 -> /A_9
- J1 pad 24: /C_12 -> /C_9
- J1 pad 25: /A_13 -> /A_8
- J1 pad 26: /C_13 -> /C_8
- J1 pad 27: /A_14 -> /A_7
- J1 pad 28: /C_14 -> /C_7
- J1 pad 29: /A_15 -> /A_6
- J1 pad 3: /A_2 -> /A_19
- J1 pad 30: /C_15 -> /C_6
- J1 pad 31: /A_16 -> /A_5
- J1 pad 32: /C_16 -> /C_5
- J1 pad 33: /A_17 -> /A_4
- J1 pad 34: /C_17 -> /C_4
- J1 pad 35: /A_18 -> /A_3
- J1 pad 36: /C_18 -> /C_3
- J1 pad 37: /A_19 -> /A_2
- J1 pad 38: /C_19 -> /C_2
- J1 pad 39: /A_20 -> /A_1
- J1 pad 4: /C_2 -> /C_19
- J1 pad 40: /C_20 -> /C_1
- J1 pad 5: /A_3 -> /A_18
- J1 pad 6: /C_3 -> /C_18
- J1 pad 7: /A_4 -> /A_17
- J1 pad 8: /C_4 -> /C_17
- J1 pad 9: /A_5 -> /A_16
- J10 pad 1: /D_2 -> /D_3
- J11 pad 1: /C_6 -> /A_2
- J12 pad 1: /B_3 -> /B_2
- J13 pad 1: /C_3 -> /C_2
- J14 pad 1: /A_3 -> /D_2
- J15 pad 1: /A_14 -> /A_1
- J16 pad 1: /C_10 -> /B_1
- J17 pad 1: /D_19 -> /C_1
- J18 pad 1: /C_20 -> /D_1
- J19 pad 1: /C_15 -> /A_8
- J2 pad 1: /B_1 -> /B_20
- J2 pad 10: /D_5 -> /D_16
- J2 pad 11: /B_6 -> /B_15
- J2 pad 12: /D_6 -> /D_15
- J2 pad 13: /B_7 -> /B_14
- J2 pad 14: /D_7 -> /D_14
- J2 pad 15: /B_8 -> /B_13
- J2 pad 16: /D_8 -> /D_13
- J2 pad 17: /B_9 -> /B_12
- J2 pad 18: /D_9 -> /D_12
- J2 pad 19: /B_10 -> /B_11
- J2 pad 2: /D_1 -> /D_20
- J2 pad 20: /D_10 -> /D_11
- J2 pad 21: /B_11 -> /B_10
- J2 pad 22: /D_11 -> /D_10
- J2 pad 23: /B_12 -> /B_9
- J2 pad 24: /D_12 -> /D_9
- J2 pad 25: /B_13 -> /B_8
- J2 pad 26: /D_13 -> /D_8
- J2 pad 27: /B_14 -> /B_7
- J2 pad 28: /D_14 -> /D_7
- J2 pad 29: /B_15 -> /B_6
- J2 pad 3: /B_2 -> /B_19
- J2 pad 30: /D_15 -> /D_6
- J2 pad 31: /B_16 -> /B_5
- J2 pad 32: /D_16 -> /D_5
- J2 pad 33: /B_17 -> /B_4
- J2 pad 34: /D_17 -> /D_4
- J2 pad 35: /B_18 -> /B_3
- J2 pad 36: /D_18 -> /D_3
- J2 pad 37: /B_19 -> /B_2
- J2 pad 38: /D_19 -> /D_2
- J2 pad 39: /B_20 -> /B_1
- J2 pad 4: /D_2 -> /D_19
- J2 pad 40: /D_20 -> /D_1
- J2 pad 5: /B_3 -> /B_18
- J2 pad 6: /D_3 -> /D_18
- J2 pad 7: /B_4 -> /B_17
- J2 pad 8: /D_4 -> /D_17
- J2 pad 9: /B_5 -> /B_16
- J20 pad 1: /A_19 -> /B_8
- J21 pad 1: /D_11 -> /C_8
- J22 pad 1: /A_6 -> /D_8
- J23 pad 1: /B_5 -> /A_7
- J24 pad 1: /C_13 -> /B_7
- J25 pad 1: /A_15 -> /C_7
- J26 pad 1: /B_12 -> /D_7
- J27 pad 1: /C_4 -> /A_6
- J28 pad 1: /C_17 -> /B_6
- J29 pad 1: /C_5 -> /C_6
- J3 pad 1: /A_1 -> /A_4
- J30 pad 1: /D_13 -> /D_6
- J31 pad 1: /A_9 -> /A_5
- J32 pad 1: /B_20 -> /B_5
- J33 pad 1: /C_7 -> /C_5
- J34 pad 1: /C_9 -> /D_5
- J35 pad 1: /A_13 -> /A_12
- J36 pad 1: /D_16 -> /B_12
- J37 pad 1: /A_11 -> /C_12
- J38 pad 1: /B_15 -> /D_12
- J39 pad 1: /A_10 -> /A_11
- J4 pad 1: /B_1 -> /B_4
- J40 pad 1: /D_7 -> /B_11
- J41 pad 1: /C_8 -> /C_11
- J42 pad 1: /C_19 -> /D_11
- J43 pad 1: /D_14 -> /A_10
- J44 pad 1: /D_18 -> /B_10
- J45 pad 1: /B_7 -> /C_10
- J46 pad 1: /A_5 -> /D_10
- J47 pad 1: /D_5 -> /A_9
- J48 pad 1: /C_16 -> /B_9
- J49 pad 1: /A_20 -> /C_9
- J5 pad 1: /C_1 -> /C_4
- J50 pad 1: /C_12 -> /D_9
- J51 pad 1: /C_14 -> /A_16
- J52 pad 1: /B_9 -> /B_16
- J53 pad 1: /B_16 -> /C_16
- J54 pad 1: /A_8 -> /D_16
- J55 pad 1: /D_10 -> /A_15
- J56 pad 1: /A_7 -> /B_15
- J57 pad 1: /B_13 -> /C_15
- J58 pad 1: /B_11 -> /D_15
- J59 pad 1: /B_10 -> /A_14
- J6 pad 1: /D_1 -> /D_4
- J60 pad 1: /A_16 -> /B_14
- J61 pad 1: /B_19 -> /C_14
- J62 pad 1: /D_4 -> /D_14
- J63 pad 1: /C_11 -> /A_13
- J64 pad 1: /D_20 -> /B_13
- J65 pad 1: /A_17 -> /C_13
- J66 pad 1: /D_8 -> /D_13
- J67 pad 1: /B_8 -> /A_20
- J68 pad 1: /D_15 -> /B_20
- J69 pad 1: /D_12 -> /C_20
- J7 pad 1: /A_2 -> /A_3
- J70 pad 1: /A_12 -> /D_20
- J71 pad 1: /D_17 -> /A_19
- J72 pad 1: /B_18 -> /B_19
- J73 pad 1: /C_18 -> /C_19
- J74 pad 1: /B_17 -> /D_19
- J76 pad 1: /D_6 -> /B_18
- J77 pad 1: /D_9 -> /C_18
- J78 pad 1: /A_4 -> /D_18
- J79 pad 1: /D_3 -> /A_17
- J8 pad 1: /B_2 -> /B_3
- J80 pad 1: /B_4 -> /B_17
- J81 pad 1: /B_14 -> /C_17
- J82 pad 1: /B_6 -> /D_17
- J9 pad 1: /C_2 -> /C_3
Routing:
- net /D_1: track 0.00 -> 245.6 mm, vias 0 -> 1
- net /B_1: track 0.00 -> 237.6 mm, vias 0 -> 1
- net /D_5: track 0.00 -> 211.2 mm, vias 0 -> 1
- net /D_2: track 0.00 -> 209.3 mm, vias 0 -> 1
- net /C_17: track 0.00 -> 205.5 mm
- net /B_5: track 0.00 -> 204.1 mm, vias 0 -> 1
- net /B_2: track 0.00 -> 199.8 mm, vias 0 -> 1
- net /C_13: track 0.00 -> 188.9 mm
- net /A_17: track 0.00 -> 187.5 mm
- net /D_9: track 0.00 -> 187.4 mm
- net /D_6: track 0.00 -> 175.8 mm, vias 0 -> 1
- net /B_9: track 0.00 -> 174.9 mm
- net /A_13: track 0.00 -> 170.7 mm
- net /D_3: track 0.00 -> 169.3 mm, vias 0 -> 1
- net /D_13: track 0.00 -> 168.0 mm
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Other:
- outline, holes or cut-outs redrawn
- copper layers 2 -> 4
- board text added: "01"
- board text added: "02"
- board text added: "03"
- board text added: "04"
- board text added: "05"
- board text added: "06"
- board text added: "1000mA MAX"
- board text added: "19"
- board text added: "20"
- board text added: "300mA MAX"
- board text added: "COMMIT_HASH"
- board text added: "F.Cu"
- board text added: "FORCE HI (UPPER ROW)"
- board text added: "FORCE LO (LOWER ROW)"
- board text added: "In2.Cu"
- board text added: "SENSE HI (UPPER ROW)"
- board text added: "SENSE LO (LOWER ROW)"

Commit message: fab update
Other:
- board text added: "c652367"
- board text removed: "COMMIT_HASH"

Commit message: update silk
Other:
- board text added: "757897f"
- board text removed: "c652367"
Changed lines of the file:
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@@
     (effects (font (size 1.5 1.5) (thickness 0.3)))
   )
-  (gr_text "c652367" (at -84.549996 -63.01 -90) (layer "B.SilkS")
+  (gr_text "757897f" (at -84.549996 -63.01 -90) (layer "B.SilkS")
     (effects (font (size 1 1) (thickness 0.15)) (justify mirror))
   )
@@
     (effects (font (size 1 1) (thickness 0.15)))
   )
-  (gr_text "c652367" (at -84.55 -63.01 270) (layer "F.SilkS")
+  (gr_text "757897f" (at -84.55 -63.01 270) (layer "F.SilkS")
     (effects (font (size 1 1) (thickness 0.15)))
   )
