File: otter_50_by_50/otter_50_by_50.kicad_pcb (KiCad board)
At the start: 0 parts

Commit message: new otter and badger boards done
Parts:
- added H1: MountingHole_Pad, MountingHole:MountingHole_2.2mm_M2_Pad_Via, F.Cu at (0.00, 0.00)
- added J1: Conn_01x01, custom_footprints:spring_pin, F.Cu at (-55.0, -59.1)
- added J10: Conn_01x12, Connector_PinHeader_2.00mm:PinHeader_1x12_P2.00mm_Vertical, B.Cu at (-5.80, -69.0)
- added J11: Conn_01x12, Connector_PinHeader_2.00mm:PinHeader_1x12_P2.00mm_Vertical, B.Cu at (5.80, -69.0)
- added J12: Conn_01x12, Connector_PinHeader_2.00mm:PinHeader_1x12_P2.00mm_Vertical, B.Cu at (64.2, -69.0)
- added J13: Conn_01x01, custom_footprints:spring_pin, F.Cu at (33.8, -10.9)
- added J14: Conn_01x01, custom_footprints:spring_pin, F.Cu at (36.2, -10.9)
- added J15: Conn_01x01, custom_footprints:spring_pin, F.Cu at (-36.2, -10.9)
- added J16: Conn_01x01, custom_footprints:spring_pin, F.Cu at (-33.8, -10.9)
- added J17: Conn_01x12, Connector_PinHeader_2.00mm:PinHeader_1x12_P2.00mm_Vertical, B.Cu at (-64.2, -40.0)
- added J18: Conn_01x12, Connector_PinHeader_2.00mm:PinHeader_1x12_P2.00mm_Vertical, B.Cu at (-5.80, -40.0)
- added J19: Conn_01x12, Connector_PinHeader_2.00mm:PinHeader_1x12_P2.00mm_Vertical, B.Cu at (5.80, -40.0)
- added J2: Conn_01x01, custom_footprints:spring_pin, F.Cu at (-36.2, -59.1)
- added J20: Conn_01x12, Connector_PinHeader_2.00mm:PinHeader_1x12_P2.00mm_Vertical, B.Cu at (64.2, -40.0)
- added J21: Conn_01x12, Connector_PinHeader_2.00mm:PinHeader_1x12_P2.00mm_Vertical, B.Cu at (-64.2, -11.0)
- added J22: Conn_01x12, Connector_PinHeader_2.00mm:PinHeader_1x12_P2.00mm_Vertical, B.Cu at (-5.80, -11.0)
- added J23: Conn_01x12, Connector_PinHeader_2.00mm:PinHeader_1x12_P2.00mm_Vertical, B.Cu at (5.80, -11.0)
- added J24: Conn_01x12, Connector_PinHeader_2.00mm:PinHeader_1x12_P2.00mm_Vertical, B.Cu at (64.2, -11.0)
- added J25: Conn_01x12, Connector_PinHeader_2.00mm:PinHeader_1x12_P2.00mm_Vertical, B.Cu at (-64.2, 18.0)
- added J26: Conn_01x12, Connector_PinHeader_2.00mm:PinHeader_1x12_P2.00mm_Vertical, B.Cu at (-5.80, 18.0)
- added J27: Conn_01x12, Connector_PinHeader_2.00mm:PinHeader_1x12_P2.00mm_Vertical, B.Cu at (5.80, 18.0)
- added J28: Conn_01x12, Connector_PinHeader_2.00mm:PinHeader_1x12_P2.00mm_Vertical, B.Cu at (64.2, 18.0)
- added J29: Conn_01x01, custom_footprints:spring_pin, F.Cu at (-36.2, 10.9)
- added J3: Conn_01x01, custom_footprints:spring_pin, F.Cu at (-33.8, -59.1)
- added J30: Conn_01x01, custom_footprints:spring_pin, F.Cu at (-33.8, 10.9)
- added J31: Conn_01x01, custom_footprints:spring_pin, F.Cu at (33.8, 10.9)
- added J32: Conn_01x01, custom_footprints:spring_pin, F.Cu at (36.2, 10.9)
- added J33: Conn_01x12, Connector_PinHeader_2.00mm:PinHeader_1x12_P2.00mm_Vertical, B.Cu at (-64.2, 47.0)
- added J34: Conn_01x12, Connector_PinHeader_2.00mm:PinHeader_1x12_P2.00mm_Vertical, B.Cu at (-5.80, 47.0)
- added J35: Conn_01x12, Connector_PinHeader_2.00mm:PinHeader_1x12_P2.00mm_Vertical, B.Cu at (5.80, 47.0)
- added J36: Conn_01x12, Connector_PinHeader_2.00mm:PinHeader_1x12_P2.00mm_Vertical, B.Cu at (64.2, 47.0)
- added J37: Conn_01x01, custom_footprints:spring_pin, F.Cu at (-55.0, 59.1)
- added J38: Conn_01x01, custom_footprints:spring_pin, F.Cu at (-36.2, 59.1)
- added J39: Conn_01x01, custom_footprints:spring_pin, F.Cu at (-33.8, 59.1)
- added J4: Conn_01x01, custom_footprints:spring_pin, F.Cu at (-15.0, -59.1)
- added J40: Conn_01x01, custom_footprints:spring_pin, F.Cu at (-15.0, 59.1)
- added J41: Conn_01x01, custom_footprints:spring_pin, F.Cu at (15.0, 59.1)
- added J42: Conn_01x01, custom_footprints:spring_pin, F.Cu at (33.8, 59.1)
- added J43: Conn_01x01, custom_footprints:spring_pin, F.Cu at (36.2, 59.1)
- added J44: Conn_01x01, custom_footprints:spring_pin, F.Cu at (55.0, 59.1)
- added J5: Conn_01x01, custom_footprints:spring_pin, F.Cu at (15.0, -59.1)
- added J6: Conn_01x01, custom_footprints:spring_pin, F.Cu at (36.2, -59.1)
- added J7: Conn_01x01, custom_footprints:spring_pin, F.Cu at (33.8, -59.1)
- added J8: Conn_01x01, custom_footprints:spring_pin, F.Cu at (55.0, -59.1)
- added J9: Conn_01x12, Connector_PinHeader_2.00mm:PinHeader_1x12_P2.00mm_Vertical, B.Cu at (-64.2, -69.0)
- added JP1: SolderJumper_3_Open, Jumper:SolderJumper-3_P2.0mm_Open_TrianglePad1.0x1.5mm_NumberLabels, B.Cu at (8.40, -23.0)
- added JP10: SolderJumper_3_Open, Jumper:SolderJumper-3_P2.0mm_Open_TrianglePad1.0x1.5mm_NumberLabels, B.Cu at (1.20, -59.2)
- added JP11: SolderJumper_3_Open, Jumper:SolderJumper-3_P2.0mm_Open_TrianglePad1.0x1.5mm_NumberLabels, B.Cu at (10.0, -67.0)
- added JP12: SolderJumper_3_Open, Jumper:SolderJumper-3_P2.0mm_Open_TrianglePad1.0x1.5mm_NumberLabels, B.Cu at (1.20, -67.0)
- added JP13: SolderJumper_3_Open, Jumper:SolderJumper-3_P2.0mm_Open_TrianglePad1.0x1.5mm_NumberLabels, B.Cu at (8.40, 35.0)
- added JP14: SolderJumper_3_Open, Jumper:SolderJumper-3_P2.0mm_Open_TrianglePad1.0x1.5mm_NumberLabels, B.Cu at (3.20, 35.0)
- added JP15: SolderJumper_3_Open, Jumper:SolderJumper-3_P2.0mm_Open_TrianglePad1.0x1.5mm_NumberLabels, B.Cu at (10.0, 24.0)
- added JP16: SolderJumper_3_Open, Jumper:SolderJumper-3_P2.0mm_Open_TrianglePad1.0x1.5mm_NumberLabels, B.Cu at (1.20, 24.0)
- added JP17: SolderJumper_3_Open, Jumper:SolderJumper-3_P2.0mm_Open_TrianglePad1.0x1.5mm_NumberLabels, B.Cu at (8.40, 18.0)
- added JP18: SolderJumper_3_Open, Jumper:SolderJumper-3_P2.0mm_Open_TrianglePad1.0x1.5mm_NumberLabels, B.Cu at (3.20, 18.0)
- added JP19: SolderJumper_3_Open, Jumper:SolderJumper-3_P2.0mm_Open_TrianglePad1.0x1.5mm_NumberLabels, B.Cu at (8.40, 64.0)
- added JP2: SolderJumper_3_Open, Jumper:SolderJumper-3_P2.0mm_Open_TrianglePad1.0x1.5mm_NumberLabels, B.Cu at (3.20, -23.0)
- added JP20: SolderJumper_3_Open, Jumper:SolderJumper-3_P2.0mm_Open_TrianglePad1.0x1.5mm_NumberLabels, B.Cu at (3.20, 64.0)
- added JP21: SolderJumper_3_Open, Jumper:SolderJumper-3_P2.0mm_Open_TrianglePad1.0x1.5mm_NumberLabels, B.Cu at (10.0, 53.0)
- added JP22: SolderJumper_3_Open, Jumper:SolderJumper-3_P2.0mm_Open_TrianglePad1.0x1.5mm_NumberLabels, B.Cu at (1.20, 53.0)
- added JP23: SolderJumper_3_Open, Jumper:SolderJumper-3_P2.0mm_Open_TrianglePad1.0x1.5mm_NumberLabels, B.Cu at (8.40, 47.0)
- added JP24: SolderJumper_3_Open, Jumper:SolderJumper-3_P2.0mm_Open_TrianglePad1.0x1.5mm_NumberLabels, B.Cu at (3.20, 47.0)
- added JP3: SolderJumper_3_Open, Jumper:SolderJumper-3_P2.0mm_Open_TrianglePad1.0x1.5mm_NumberLabels, B.Cu at (10.0, -34.0)
- added JP4: SolderJumper_3_Open, Jumper:SolderJumper-3_P2.0mm_Open_TrianglePad1.0x1.5mm_NumberLabels, B.Cu at (1.20, -34.0)
- added JP5: SolderJumper_3_Open, Jumper:SolderJumper-3_P2.0mm_Open_TrianglePad1.0x1.5mm_NumberLabels, B.Cu at (8.40, -40.0)
- added JP6: SolderJumper_3_Open, Jumper:SolderJumper-3_P2.0mm_Open_TrianglePad1.0x1.5mm_NumberLabels, B.Cu at (3.20, -40.0)
- added JP7: SolderJumper_3_Open, Jumper:SolderJumper-3_P2.0mm_Open_TrianglePad1.0x1.5mm_NumberLabels, B.Cu at (8.40, -52.0)
- added JP8: SolderJumper_3_Open, Jumper:SolderJumper-3_P2.0mm_Open_TrianglePad1.0x1.5mm_NumberLabels, B.Cu at (3.20, -52.0)
- added JP9: SolderJumper_3_Open, Jumper:SolderJumper-3_P2.0mm_Open_TrianglePad1.0x1.5mm_NumberLabels, B.Cu at (10.4, -60.0)
- added LOGO1: Logo_Open_Hardware_Small, custom_footprints:site_small, F.Cu at (-47.5, -11.2)
- added LOGO2: Logo_Open_Hardware_Small, custom_footprints:site_small, F.Cu at (47.2, 11.2)
Routing:
- net 3D_bit3b: track 0.00 -> 93.0 mm, vias 0 -> 1
- net 3E_bit6b: track 0.00 -> 89.5 mm
- net 3A_bit3b: track 0.00 -> 88.9 mm, vias 0 -> 1
- net 3B_bit6b: track 0.00 -> 88.9 mm
- net 3E_bit6a: track 0.00 -> 86.1 mm
- net 3B_bit6a: track 0.00 -> 85.9 mm
- net 3A_bit3a: track 0.00 -> 79.7 mm, vias 0 -> 1
- net 3B_bit3b: track 0.00 -> 79.1 mm, vias 0 -> 1
- net 3D_bit3a: track 0.00 -> 78.3 mm, vias 0 -> 1
- net 3D_bit6b: track 0.00 -> 73.9 mm
- net 3D_bit6a: track 0.00 -> 70.4 mm
- net 3B_bit3a: track 0.00 -> 65.5 mm, vias 0 -> 1
- net 3A_bit6b: track 0.00 -> 62.0 mm
- net 3A_bit6a: track 0.00 -> 58.4 mm
- net 3E_bit3a: track 0.00 -> 47.9 mm, vias 0 -> 1
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- added copper zone on B.Cu, net GND
Other:
- board outline added: 130.4 x 141.4 mm
- copper layers 0 -> 2
- board text added: "MODULE 1"
- board text added: "MODULE 2"
- board text added: "MODULE 3"
- board text added: "MODULE 4"
- board text added: "commithash"
