File: otter_50_by_50/otter_50_by_50.kicad_pcb (KiCad board)
At the start: 2 copper layers, 130.4 x 141.4 mm, 71 parts, among them J1 Conn_01x01, J10 Conn_01x12, J11 Conn_01x12, J12 Conn_01x12, J13 Conn_01x01, J14 Conn_01x01, J15 Conn_01x01, J16 Conn_01x01, J17 Conn_01x12, J18 Conn_01x12, J19 Conn_01x12, J2 Conn_01x01, J20 Conn_01x12, J21 Conn_01x12, J22 Conn_01x12, J23 Conn_01x12, J24 Conn_01x12, J25 Conn_01x12, J26 Conn_01x12, J27 Conn_01x12, J28 Conn_01x12, J29 Conn_01x01, J3 Conn_01x01, J30 Conn_01x01, J31 Conn_01x01, J32 Conn_01x01, J33 Conn_01x12, J34 Conn_01x12, J35 Conn_01x12, J36 Conn_01x12, J37 Conn_01x01, J38 Conn_01x01, J39 Conn_01x01, J4 Conn_01x01, J40 Conn_01x01, J41 Conn_01x01, J42 Conn_01x01, J43 Conn_01x01, J44 Conn_01x01, J5 Conn_01x01, J6 Conn_01x01, J7 Conn_01x01, J8 Conn_01x01, J9 Conn_01x12

Commit message: fab update
Other:
- board text added: "c652367"
- board text removed: "commithash"
Changed lines of the file:
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@@
     (effects (font (size 1.5 1.5) (thickness 0.3)))
   )
-  (gr_text "commithash" (at 44.25 -58.5) (layer "F.SilkS")
+  (gr_text "c652367" (at 44.25 -58.50001) (layer "F.SilkS")
     (effects (font (size 1 1) (thickness 0.15)))
   )

Commit message: update silk
Other:
- board text added: "757897f"
- board text removed: "c652367"
Changed lines of the file:
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@@
   (gr_arc (start 56.125 -56.125) (end 57.625 -56.125) (angle -90) (layer "Edge.Cuts") (width 0.05))
   (gr_line (start -13.875 -12.375) (end -56.125 -12.375) (layer "Edge.Cuts") (width 0.05))
+  (gr_text "757897f" (at 44.5 -58.5 180) (layer "B.SilkS")
+    (effects (font (size 1 1) (thickness 0.15)) (justify mirror))
+  )
   (gr_text "MODULE 3" (at -25 11) (layer "F.SilkS")
     (effects (font (size 1.5 1.5) (thickness 0.3)))
@@
     (effects (font (size 1.5 1.5) (thickness 0.3)))
   )
-  (gr_text "c652367" (at 44.25 -58.50001) (layer "F.SilkS")
+  (gr_text "757897f" (at 44.5 -58.5) (layer "F.SilkS")
     (effects (font (size 1 1) (thickness 0.15)))
   )
