File: otter_50_by_50/otter_50_by_50.kicad_sch (KiCad schematic)
At the start: 70 parts

Commit message: new otter and badger boards done
Parts:
- removed JP?: SolderJumper_3_Open, symbol Jumper:SolderJumper_3_Open
- added H1: MountingHole_Pad, MountingHole:MountingHole_2.2mm_M2_Pad_Via, symbol Mechanical:MountingHole_Pad
- added JP22: SolderJumper_3_Open, Jumper:SolderJumper-3_P2.0mm_Open_TrianglePad1.0x1.5mm_NumberLabels, symbol Jumper:SolderJumper_3_Open
- J1, J13, J14, J15, J16, J2, J29, J3, J30, J31, J32, J37, J38, J39, J4, J40, J41, J42, J43, J44, J5, J6, J7, J8: renamed from J?; footprint (none) -> custom_footprints:spring_pin
- J10, J11, J12, J17, J18, J19, J20, J21, J22, J23, J24, J25, J26, J27, J28, J33, J34, J35, J36, J9: renamed from J?; footprint (none) -> Connector_PinHeader_2.00mm:PinHeader_1x12_P2.00mm_Vertical
- JP1, JP10, JP11, JP12, JP13, JP14, JP15, JP16, JP17, JP18, JP19, JP2, JP20, JP21, JP23, JP24, JP3, JP4, JP5, JP6, JP7, JP8, JP9: renamed from JP?; footprint (none) -> Jumper:SolderJumper-3_P2.0mm_Open_TrianglePad1.0x1.5mm_NumberLabels
- LOGO1, LOGO2: renamed from LOGO?; footprint (none) -> custom_footprints:site_small
Connections:
- net 3A_bit1a: now also JP19.1 (A), JP20.1 (A)
- net 3A_bit1b: now also JP19.3 (B), JP20.3 (B)
- net 3A_bit3a: now also JP19.2 (C), JP21.2 (C)
- net 3A_bit3b: now also JP20.2 (C), JP22.2 (C)
- net 3A_bit5a: now also JP21.1 (A), JP22.1 (A)
- net 3A_bit5b: now also JP21.3 (B), JP22.3 (B)
- net 3A_bit6a: now also JP23.2 (C)
- net 3A_bit6b: now also JP24.2 (C)
- net 3A_bit7a: now also JP23.1 (A), JP24.1 (A)
- net 3A_bit7b: now also JP23.3 (B), JP24.3 (B)
- net 3B_bit1a: now also JP13.1 (A), JP14.1 (A)
- net 3B_bit1b: now also JP13.3 (B), JP14.3 (B)
- net 3B_bit3a: now also JP13.2 (C), JP15.2 (C); no longer JP13.1 (A), JP14.1 (A), JP15.1 (A), JP16.1 (A)
- net 3B_bit3b: now also JP14.2 (C), JP16.2 (C); no longer JP13.3 (B), JP14.3 (B), JP15.3 (B), JP16.3 (B)
- net 3B_bit5a: now also JP15.1 (A), JP16.1 (A)
- net 3B_bit5b: now also JP15.3 (B), JP16.3 (B)
- net 3B_bit6a: now also J39.1 (Pin_1), JP17.2 (C); no longer J13.1 (Pin_1)
- net 3B_bit6b: now also J38.1 (Pin_1), JP18.2 (C); no longer J14.1 (Pin_1)
- net 3B_bit7a: now also JP17.1 (A), JP18.1 (A)
- net 3B_bit7b: now also JP17.3 (B), JP18.3 (B)
- net 3D_bit1a: now also JP1.1 (A), JP2.1 (A)
- net 3D_bit1b: now also JP1.3 (B), JP2.3 (B)
- net 3D_bit3a: now also JP1.2 (C), JP3.2 (C)
- net 3D_bit3b: now also JP2.2 (C), JP4.2 (C)
- net 3D_bit5a: now also JP3.1 (A), JP4.1 (A)
- net 3D_bit5b: now also JP3.3 (B), JP4.3 (B)
- net 3D_bit6a: now also JP5.2 (C)
- net 3D_bit6b: now also JP6.2 (C)
- net 3D_bit7a: now also JP5.1 (A), JP6.1 (A)
- net 3D_bit7b: now also JP5.3 (B), JP6.3 (B)
- net 3E_bit1a: now also JP7.1 (A), JP8.1 (A)
- net 3E_bit1b: now also JP7.3 (B), JP8.3 (B)
- net 3E_bit3a: now also JP7.2 (C), JP9.2 (C)
- net 3E_bit3b: now also JP10.2 (C), JP8.2 (C)
- net 3E_bit5a: now also JP10.1 (A), JP9.1 (A)
- net 3E_bit5b: now also JP10.3 (B), JP9.3 (B)
- net 3E_bit6a: now also J13.1 (Pin_1), JP11.2 (C); no longer J39.1 (Pin_1)
- net 3E_bit6b: now also J14.1 (Pin_1), JP12.2 (C); no longer J38.1 (Pin_1)
- net 3E_bit7a: now also JP11.1 (A), JP12.1 (A)
- net 3E_bit7b: now also JP11.3 (B), JP12.3 (B)
- new net GND: H1.1
Other:
- moved on the sheet: J1, J10, J11, J12, J13, J14, J15, J16, J17, J18, J19, J2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
