File: adapter/adapter.kicad_pcb (KiCad board)
At the start: 2 copper layers, 30 x 30 mm, 46 parts, among them J1 Conn_01x01, J10 Conn_01x01, J11 Conn_01x01, J12 Conn_01x01, J13 Conn_01x01, J14 Conn_01x01, J15 Conn_01x01, J16 Conn_01x01, J17 Conn_01x01, J18 Conn_01x01, J19 Conn_01x01, J2 Conn_01x01, J20 Conn_01x01, J21 Conn_01x01, J22 Conn_01x01, J23 Conn_01x01, J24 Conn_01x01, J25 Conn_01x01, J26 Conn_01x01, J27 Conn_01x01, J28 Conn_01x01, J29 Conn_01x01, J3 Conn_01x01, J30 Conn_01x01, J31 Conn_01x01, J32 Conn_01x01, J33 Conn_01x01, J34 Conn_01x01, J35 Conn_01x01, J36 Conn_01x01, J37 Conn_01x01, J38 Conn_01x01, J39 Conn_01x01, J4 Conn_01x01, J40 Conn_01x01, J41 Conn_01x01, J42 Conn_01x01, J43 Conn_01x01, J44 Conn_01x01, J5 Conn_01x01, J6 Conn_01x01, J7 Conn_01x01, J8 Conn_01x01, J9 Conn_01x01

Commit message: update silk
Other:
- board text added: "0dbcc89"
- board text removed: "98e55eb"
Changed lines of the file:
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@@
   (gr_arc (start 10 7.9) (end 10 9.9) (angle -90) (layer "Edge.Cuts") (width 0.05))
   (gr_line (start -15 15) (end 15 15) (layer "Edge.Cuts") (width 0.05))
-  (gr_text "98e55eb" (at 14 10 90) (layer "B.SilkS")
+  (gr_text "0dbcc89" (at 14 10 90) (layer "B.SilkS")
     (effects (font (size 1.5 1.5) (thickness 0.3)) (justify mirror))
   )
-  (gr_text "98e55eb" (at 14 10 90) (layer "F.SilkS")
+  (gr_text "0dbcc89" (at 14 10 90) (layer "F.SilkS")
     (effects (font (size 1.5 1.5) (thickness 0.3)))
   )

Commit message: update adapter boards for pressfit
Parts:
- J1, J10, J11, J12, J13, J14, J15, J16, J17, J18, J19, J2, J20, J21, J22, J23, J24, J3, J4, J5, J6, J7, J8, J9: footprint custom_footprints:5342 -> custom_footprints:PTT-one-pin
- moved J25 0.25 mm to (-11.4, -12.0)
- moved J26 0.25 mm to (-8.91, -12.0)
- moved J27 0.25 mm to (-6.33, -12.0)
- moved J28 0.25 mm to (-3.83, -12.0)
- moved J29 0.25 mm to (-1.25, -12.0)
- moved J30 0.25 mm to (1.25, -12.0)
- moved J31 0.25 mm to (3.83, -12.0)
- moved J32 0.25 mm to (6.33, -12.0)
- moved J33 0.25 mm to (8.91, -12.0)
- moved J34 0.25 mm to (11.4, -12.0)
- moved J35 0.25 mm to (11.4, 12.0)
- moved J36 0.25 mm to (8.91, 12.0)
- moved J37 0.25 mm to (6.33, 12.0)
- moved J38 0.25 mm to (3.83, 12.0)
- moved J39 0.25 mm to (1.25, 12.0)
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
Commit message: update silk
Parts:
- moved LOGO1 28.7 mm to (14.2, 1.00)
- moved LOGO2 28.7 mm to (14.2, 1.00)
Other:
- board text added: "1"
- board text added: "2"
- board text added: "5"
- board text added: "6"
- board text added: "b5195e4"
- board text removed: "0dbcc89"
Changed lines of the file:
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@@
   )
   (footprint "custom_footprints:logo_small" (layer "F.Cu")
-    (at -14 -4 90)
+    (at 14.25 1 90)
     (property "Sheetfile" "adapter.kicad_sch")
     (property "Sheetname" "")
@@
     (property "Sheetfile" "adapter.kicad_sch")
     (property "Sheetname" "")
-    (fp_text reference "J22" (at 0 2 180 unlocked) (layer "B.SilkS")
+    (fp_text reference "J22" (at 0 2 180 unlocked) (layer "B.SilkS") hide
       (effects (font (size 1 1) (thickness 0.15)) (justify mirror))
     )
@@
     (property "Sheetfile" "adapter.kicad_sch")
     (property "Sheetname" "")
-    (fp_text reference "J19" (at 0 2 180 unlocked) (layer "B.SilkS")
+    (fp_text reference "J19" (at 0 2 180 unlocked) (layer "B.SilkS") hide
       (effects (font (size 1 1) (thickness 0.15)) (justify mirror))
     )
@@
     (property "Sheetfile" "adapter.kicad_sch")
     (property "Sheetname" "")
-    (fp_text reference "J20" (at 0 2 180 unlocked) (layer "B.SilkS")
+    (fp_text reference "J20" (at 0 2 180 unlocked) (layer "B.SilkS") hide
       (effects (font (size 1 1) (thickness 0.15)) (justify mirror))
     )
@@
     (property "Sheetfile" "adapter.kicad_sch")
     (property "Sheetname" "")
-    (fp_text reference "J23" (at 0 2 180 unlocked) (layer "B.SilkS")
+    (fp_text reference "J23" (at 0 2 180 unlocked) (layer "B.SilkS") hide
       (effects (font (size 1 1) (thickness 0.15)) (justify mirror))
     )
@@
     (property "Sheetfile" "adapter.kicad_sch")
     (property "Sheetname" "")
-    (fp_text reference "J15" (at 0 2 180 unlocked) (layer "B.SilkS")
+    (fp_text reference "J15" (at 0 2 180 unlocked) (layer "B.SilkS") hide
       (effects (font (size 1 1) (thickness 0.15)) (justify mirror))
     )
@@
   )
   (footprint "custom_footprints:logo_small" (layer "B.Cu")
-    (at -14 -4 -90)
+    (at 14.25 1 -90)
     (property "Sheetfile" "adapter.kicad_sch")
     (property "Sheetname" "")
@@
     (property "Sheetfile" "adapter.kicad_sch")
     (property "Sheetname" "")
-    (fp_text reference "J14" (at 0 2 180 unlocked) (layer "B.SilkS")
+    (fp_text reference "J14" (at 0 2 180 unlocked) (layer "B.SilkS") hide
       (effects (font (size 1 1) (thickness 0.15)) (justify mirror))
     )
@@
     (property "Sheetfile" "adapter.kicad_sch")
     (property "Sheetname" "")
-    (fp_text reference "J13" (at 0 2 180 unlocked) (layer "B.SilkS")
+    (fp_text reference "J13" (at 0 2 180 unlocked) (layer "B.SilkS") hide
       (effects (font (size 1 1) (thickness 0.15)) (justify mirror))
     )
@@
     (property "Sheetfile" "adapter.kicad_sch")
     (property "Sheetname" "")
-    (fp_text reference "J21" (at 0 2 180 unlocked) (layer "B.SilkS")
+    (fp_text reference "J21" (at 0 2 180 unlocked) (layer "B.SilkS") hide
       (effects (font (size 1 1) (thickness 0.15)) (justify mirror))
     )
@@
     (property "Sheetfile" "adapter.kicad_sch")
     (property "Sheetname" "")
-    (fp_text reference "J17" (at 0 2 180 unlocked) (layer "B.SilkS")
+    (fp_text reference "J17" (at 0 2 180 unlocked) (layer "B.SilkS") hide
       (effects (font (size 1 1) (thickness 0.15)) (justify mirror))
     )
@@
     (property "Sheetfile" "adapter.kicad_sch")
     (property "Sheetname" "")
-    (fp_text reference "J18" (at 0 2 180 unlocked) (layer "B.SilkS")
+    (fp_text reference "J18" (at 0 2 180 unlocked) (layer "B.SilkS") hide
       (effects (font (size 1 1) (thickness 0.15)) (justify mirror))
     )
@@
     (property "Sheetfile" "adapter.kicad_sch")
     (property "Sheetname" "")
-    (fp_text reference "J24" (at 0 2 180 unlocked) (layer "B.SilkS")
+    (fp_text reference "J24" (at 0 2 180 unlocked) (layer "B.SilkS") hide
       (effects (font (size 1 1) (thickness 0.15)) (justify mirror))
     )
@@
     (property "Sheetfile" "adapter.kicad_sch")
     (property "Sheetname" "")
-    (fp_text reference "J16" (at 0 2 180 unlocked) (layer "B.SilkS")
+    (fp_text reference "J16" (at 0 2 180 unlocked) (layer "B.SilkS") hide
       (effects (font (size 1 1) (thickness 0.15)) (justify mirror))
     )
@@
   (gr_arc (start 10 7.9) (end 10 9.9) (angle -90) (layer "Edge.Cuts") (width 0.05))
   (gr_line (start -15 15) (end 15 15) (layer "Edge.Cuts") (width 0.05))
-  (gr_text "0dbcc89" (at 14 10 90) (layer "B.SilkS")
+  (gr_text "b5195e4" (at -13.5 0 90) (layer "B.SilkS")
     (effects (font (size 1.5 1.5) (thickness 0.3)) (justify mirror))
   )
-  (gr_text "0dbcc89" (at 14 10 90) (layer "F.SilkS")
+  (gr_text "b5195e4" (at -13.5 0 90) (layer "F.SilkS")
     (effects (font (size 1.5 1.5) (thickness 0.3)))
   )
+  (gr_text "6" (at 13.75 -13.75 180) (layer "F.SilkS")
+    (effects (font (size 1.5 1.5) (thickness 0.3)))
+  )
+  (gr_text "5" (at 13.5 13.5) (layer "F.SilkS")
+    (effects (font (size 1.5 1.5) (thickness 0.3)))
+  )
+  (gr_text "2" (at -13.5 -13.5 180) (layer "F.SilkS")
+    (effects (font (size 1.5 1.5) (thickness 0.3)))
+  )
+  (gr_text "1" (at -13.5 13.5) (layer "F.SilkS")
+    (effects (font (size 1.5 1.5) (thickness 0.3)))
+  )
