File: crossbar-4x1x30x10-half/crossbar-4x1x30x10-half.kicad_sch (KiCad schematic)
At the start: 30 parts, among them J1 Conn_02x06_Counter_Clockwise, J10 Conn_02x06_Counter_Clockwise, J11 Conn_02x06_Counter_Clockwise, J12 Conn_02x06_Counter_Clockwise, J13 Conn_02x06_Counter_Clockwise, J14 Conn_02x06_Counter_Clockwise, J15 Conn_02x06_Counter_Clockwise, J16 Conn_02x06_Counter_Clockwise, J17 Conn_02x06_Counter_Clockwise, J18 Conn_02x06_Counter_Clockwise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

Commit message: top pcb doneish
Parts:
- added J21, J22, J23, J24: Conn_01x06, MINE:MMS-106-02-X-SH, symbol Connector_Generic:Conn_01x06
- added LOGO1, LOGO2: Logo, MINE:logo_small, symbol Graphic:Logo_Open_Hardware_Small
Connections:
- net 1_a1: now also J23.6 (Pin_6)
- net 1_a11: now also J21.1 (Pin_1)
- net 1_a12: now also J21.2 (Pin_2)
- net 1_a2: now also J23.5 (Pin_5)
- net 1_a5: now also J23.2 (Pin_2)
- net 1_a8: now also J21.5 (Pin_5)
- net 2_a1: now also J23.4 (Pin_4)
- net 2_a11: now also J21.3 (Pin_3)
- net 2_a12: now also J21.4 (Pin_4)
- net 2_a2: now also J23.3 (Pin_3)
- net 2_a5: now also J23.1 (Pin_1)
- net 2_a8: now also J21.6 (Pin_6)
- net 3_a1: now also J22.3 (Pin_3)
- net 3_a11: now also J24.4 (Pin_4)
- net 3_a12: now also J24.3 (Pin_3)
- net 3_a2: now also J22.4 (Pin_4)
- net 3_a5: now also J22.1 (Pin_1)
- net 3_a8: now also J24.6 (Pin_6)
- net 4_a1: now also J22.5 (Pin_5)
- net 4_a11: now also J24.2 (Pin_2)
- net 4_a12: now also J24.1 (Pin_1)
- net 4_a2: now also J22.6 (Pin_6)
- net 4_a5: now also J22.2 (Pin_2)
- net 4_a8: now also J24.5 (Pin_5)
Other:
- moved on the sheet: H1, H2, H5, JP1, JP2
