File: led_mockup/led_mockup.kicad_pcb (KiCad board)
At the start: 4 copper layers, 350 x 350 mm, 638 parts, among them J1 Conn_01x04, J2 Conn_01x04

Commit message: update led mockup
Other:
- net class Default removed
- net class nomask removed
