File: spring_pin_spacer/spring_pin_spacer.kicad_pcb (KiCad board)
At the start: 2 copper layers, 184 x 48 mm, 56 parts

Commit message: update silk
Parts:
- turned LOGO2 to 0 degrees
Other:
- board text added: "0dbcc89"
- board text removed: "98e55eb"
Changed lines of the file:
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@@
   )
   (footprint "custom_footprints:logo" (layer "B.Cu")
-    (at -71 -22 180)
+    (at -71 -22)
     (property "Sheetfile" "spring_pin_spacer.kicad_sch")
     (property "Sheetname" "")
@@
   (gr_arc (start 34 9.254248) (end 32 9.254248) (angle -41.40962211) (layer "Edge.Cuts") (width 0.05))
   (gr_arc (start -6 9.254248) (end -8 9.254248) (angle -41.40962211) (layer "Edge.Cuts") (width 0.05))
-  (gr_text "98e55eb" (at -88.5 -20) (layer "B.SilkS")
+  (gr_text "0dbcc89" (at -88.25 -20.25 180) (layer "B.SilkS")
     (effects (font (size 1 1) (thickness 0.15)) (justify mirror))
   )
-  (gr_text "98e55eb" (at -88.5 -20 180) (layer "F.SilkS")
+  (gr_text "0dbcc89" (at -88.25 -20.25 180) (layer "F.SilkS")
     (effects (font (size 1 1) (thickness 0.15)))
   )

Commit message: some mods
Other:
- board size 184 x 48 mm -> 184 x 184 mm
