File: squirrel/squirrel.kicad_sch (KiCad schematic)
At the start: 45 parts, among them J1 Conn_01x01, J10 Conn_01x01, J11 Conn_01x01, J12 Conn_01x01, J13 Conn_01x01, J14 Conn_01x01, J15 Conn_01x01, J16 Conn_01x01, J17 Conn_01x01, J18 Conn_01x01, J19 Conn_01x01, J2 Conn_01x01, J20 Conn_01x01, J21 Conn_01x01, J22 Conn_01x01, J23 Conn_01x01, J24 Conn_01x01, J25 Conn_01x01, J26 Conn_01x01, J27 Conn_01x01, J28 Conn_01x01, J29 Conn_01x01, J3 Conn_01x01, J30 Conn_01x01, J31 Conn_01x01, J32 Conn_01x01, J33 Conn_01x01, J34 Conn_01x01, J35 Conn_01x01, J36 Conn_01x01, J37 Conn_01x01, J38 Conn_01x01, J39 Conn_01x01, J4 Conn_01x01, J40 Conn_01x01, J41 Conn_02x20_Odd_Even, J5 Conn_01x01, J6 Conn_01x01, J7 Conn_01x01, J8 Conn_01x01, J9 Conn_01x01

Commit message: wip on squ
Parts:
- added H10, H11, H12, H13, H14, H15, H16, H17, H18, H19, H5, H6, H7, H8, H9: MountingHole, MountingHole:MountingHole_3.2mm_M3, symbol Mechanical:MountingHole
- J1, J10, J11, J12, J13, J14, J15, J16, J17, J18, J19, J2, J20, J21, J22, J23, J24, J25, J26, J27, J28, J29, J3, J30, J31, J32, J33, J34, J35, J36, J37, J38, J39, J4, J40, J5, J6, J7, J8, J9: footprint Connector_PinHeader_2.54mm:PinHeader_1x01_P2.54mm_Vertical -> custom_footprints:0921
Connections:
- net F1: now also J41.40 (Pin_40); no longer J41.1 (Pin_1)
- net F10: now also J41.22 (Pin_22); no longer J41.19 (Pin_19)
- net F11: now also J41.20 (Pin_20); no longer J41.21 (Pin_21)
- net F12: now also J41.18 (Pin_18); no longer J41.23 (Pin_23)
- net F13: now also J41.16 (Pin_16); no longer J41.25 (Pin_25)
- net F14: now also J41.14 (Pin_14); no longer J41.27 (Pin_27)
- net F15: now also J41.12 (Pin_12); no longer J41.29 (Pin_29)
- net F16: now also J41.10 (Pin_10); no longer J41.31 (Pin_31)
- net F17: now also J41.8 (Pin_8); no longer J41.33 (Pin_33)
- net F18: now also J41.6 (Pin_6); no longer J41.35 (Pin_35)
- net F19: now also J41.4 (Pin_4); no longer J41.37 (Pin_37)
- net F2: now also J41.38 (Pin_38); no longer J41.3 (Pin_3)
- net F20: now also J41.2 (Pin_2); no longer J41.39 (Pin_39)
- net F3: now also J41.36 (Pin_36); no longer J41.5 (Pin_5)
- net F4: now also J41.34 (Pin_34); no longer J41.7 (Pin_7)
- net F5: now also J41.32 (Pin_32); no longer J41.9 (Pin_9)
- net F6: now also J41.30 (Pin_30); no longer J41.11 (Pin_11)
- net F7: now also J41.28 (Pin_28); no longer J41.13 (Pin_13)
- net F8: now also J41.26 (Pin_26); no longer J41.15 (Pin_15)
- net F9: now also J41.24 (Pin_24); no longer J41.17 (Pin_17)
- net S1: now also J41.39 (Pin_39); no longer J41.2 (Pin_2)
- net S10: now also J41.21 (Pin_21); no longer J41.20 (Pin_20)
- net S11: now also J41.19 (Pin_19); no longer J41.22 (Pin_22)
- net S12: now also J41.17 (Pin_17); no longer J41.24 (Pin_24)
- net S13: now also J41.15 (Pin_15); no longer J41.26 (Pin_26)
- net S14: now also J41.13 (Pin_13); no longer J41.28 (Pin_28)
- net S15: now also J41.11 (Pin_11); no longer J41.30 (Pin_30)
- net S16: now also J41.9 (Pin_9); no longer J41.32 (Pin_32)
- net S17: now also J41.7 (Pin_7); no longer J41.34 (Pin_34)
- net S18: now also J41.5 (Pin_5); no longer J41.36 (Pin_36)
- net S19: now also J41.3 (Pin_3); no longer J41.38 (Pin_38)
- net S2: now also J41.37 (Pin_37); no longer J41.4 (Pin_4)
- net S20: now also J41.1 (Pin_1); no longer J41.40 (Pin_40)
- net S3: now also J41.35 (Pin_35); no longer J41.6 (Pin_6)
- net S4: now also J41.33 (Pin_33); no longer J41.8 (Pin_8)
- net S5: now also J41.31 (Pin_31); no longer J41.10 (Pin_10)
- net S6: now also J41.29 (Pin_29); no longer J41.12 (Pin_12)
- net S7: now also J41.27 (Pin_27); no longer J41.14 (Pin_14)
- net S8: now also J41.25 (Pin_25); no longer J41.16 (Pin_16)
- net S9: now also J41.23 (Pin_23); no longer J41.18 (Pin_18)
Other:
- moved on the sheet: H1, H2, H3, H4

Commit message: wip on sq pcb
Parts:
- added H20, H21, H22, H23, H24, H25: MountingHole, custom_footprints:MountingHole_3.2mm_M3_wscrew, symbol Mechanical:MountingHole
- added J42, J43: Conn_02x20_Odd_Even, custom_footprints:TST-120-01-G-D, symbol Connector_Generic:Conn_02x20_Odd_Even
- H10, H11, H12, H13, H14, H15, H16, H17, H18, H19, H5, H6, H7, H8, H9: footprint MountingHole:MountingHole_3.2mm_M3 -> custom_footprints:MountingHole_3.2mm_M3_wscrew
- J41: footprint (none) -> custom_footprints:TST-120-01-G-D
Connections:
- net F1: now also J41.2 (Pin_2); no longer J41.40 (Pin_40)
- net F10: now also J41.20 (Pin_20); no longer J41.22 (Pin_22)
- net F11: now also J41.22 (Pin_22); no longer J41.20 (Pin_20)
- net F12: now also J41.24 (Pin_24); no longer J41.18 (Pin_18)
- net F13: now also J41.26 (Pin_26); no longer J41.16 (Pin_16)
- net F14: now also J41.28 (Pin_28); no longer J41.14 (Pin_14)
- net F15: now also J41.30 (Pin_30); no longer J41.12 (Pin_12)
- net F16: now also J41.32 (Pin_32); no longer J41.10 (Pin_10)
- net F17: now also J41.34 (Pin_34); no longer J41.8 (Pin_8)
- net F18: now also J41.36 (Pin_36); no longer J41.6 (Pin_6)
- net F19: now also J41.38 (Pin_38); no longer J41.4 (Pin_4)
- net F2: now also J41.4 (Pin_4); no longer J41.38 (Pin_38)
- net F20: now also J41.40 (Pin_40); no longer J41.2 (Pin_2)
- net F3: now also J41.6 (Pin_6); no longer J41.36 (Pin_36)
- net F4: now also J41.8 (Pin_8); no longer J41.34 (Pin_34)
- net F5: now also J41.10 (Pin_10); no longer J41.32 (Pin_32)
- net F6: now also J41.12 (Pin_12); no longer J41.30 (Pin_30)
- net F7: now also J41.14 (Pin_14); no longer J41.28 (Pin_28)
- net F8: now also J41.16 (Pin_16); no longer J41.26 (Pin_26)
- net F9: now also J41.18 (Pin_18); no longer J41.24 (Pin_24)
- net S1: now also J41.1 (Pin_1); no longer J41.39 (Pin_39)
- net S10: now also J41.19 (Pin_19); no longer J41.21 (Pin_21)
- net S11: now also J41.21 (Pin_21); no longer J41.19 (Pin_19)
- net S12: now also J41.23 (Pin_23); no longer J41.17 (Pin_17)
- net S13: now also J41.25 (Pin_25); no longer J41.15 (Pin_15)
- net S14: now also J41.27 (Pin_27); no longer J41.13 (Pin_13)
- net S15: now also J41.29 (Pin_29); no longer J41.11 (Pin_11)
- net S16: now also J41.31 (Pin_31); no longer J41.9 (Pin_9)
- net S17: now also J41.33 (Pin_33); no longer J41.7 (Pin_7)
- net S18: now also J41.35 (Pin_35); no longer J41.5 (Pin_5)
- net S19: now also J41.37 (Pin_37); no longer J41.3 (Pin_3)
- net S2: now also J41.3 (Pin_3); no longer J41.37 (Pin_37)
- net S20: now also J41.39 (Pin_39); no longer J41.1 (Pin_1)
- net S3: now also J41.5 (Pin_5); no longer J41.35 (Pin_35)
- net S4: now also J41.7 (Pin_7); no longer J41.33 (Pin_33)
- net S5: now also J41.9 (Pin_9); no longer J41.31 (Pin_31)
- net S6: now also J41.11 (Pin_11); no longer J41.29 (Pin_29)
- net S7: now also J41.13 (Pin_13); no longer J41.27 (Pin_27)
- net S8: now also J41.15 (Pin_15); no longer J41.25 (Pin_25)
- net S9: now also J41.17 (Pin_17); no longer J41.23 (Pin_23)

Commit message: wip on squ
Connections:
- net PT_F20: now reaches J43.1 (Pin_1)
- net PT_F20: now also J42.40 (Pin_40)
- net PT_S16: now reaches J43.10 (Pin_10)
- net PT_S16: now also J42.31 (Pin_31)
- net PT_F15: now reaches J43.11 (Pin_11)
- net PT_F15: now also J42.30 (Pin_30)
- net PT_S15: now reaches J43.12 (Pin_12)
- net PT_S15: now also J42.29 (Pin_29)
- net PT_F14: now reaches J43.13 (Pin_13)
- net PT_F14: now also J42.28 (Pin_28)
- net PT_S14: now reaches J43.14 (Pin_14)
- net PT_S14: now also J42.27 (Pin_27)
- net PT_F13: now reaches J43.15 (Pin_15)
- net PT_F13: now also J42.26 (Pin_26)
- net PT_S13: now reaches J43.16 (Pin_16)
- net PT_S13: now also J42.25 (Pin_25)
- net PT_F12: now reaches J43.17 (Pin_17)
- net PT_F12: now also J42.24 (Pin_24)
- net PT_S12: now reaches J43.18 (Pin_18)
- net PT_S12: now also J42.23 (Pin_23)
- net PT_F11: now reaches J43.19 (Pin_19)
- net PT_F11: now also J42.22 (Pin_22)
- net PT_S20: now reaches J43.2 (Pin_2)
- net PT_S20: now also J42.39 (Pin_39)
- net PT_S11: now reaches J43.20 (Pin_20)
- net PT_S11: now also J42.21 (Pin_21)
- net PT_F10: now reaches J43.21 (Pin_21)
- net PT_F10: now also J42.20 (Pin_20)
- net PT_S10: now reaches J43.22 (Pin_22)
- net PT_S10: now also J42.19 (Pin_19)
- net PT_F9: now reaches J43.23 (Pin_23)
- net PT_F9: now also J42.18 (Pin_18)
- net PT_S9: now reaches J43.24 (Pin_24)
- net PT_S9: now also J42.17 (Pin_17)
- net PT_F8: now reaches J43.25 (Pin_25)
- net PT_F8: now also J42.16 (Pin_16)
- net PT_S8: now reaches J43.26 (Pin_26)
- net PT_S8: now also J42.15 (Pin_15)
- net PT_F7: now reaches J43.27 (Pin_27)
- net PT_F7: now also J42.14 (Pin_14)
- net PT_S7: now reaches J43.28 (Pin_28)
- net PT_S7: now also J42.13 (Pin_13)
- net PT_F6: now reaches J43.29 (Pin_29)
- net PT_F6: now also J42.12 (Pin_12)
- net PT_F19: now reaches J43.3 (Pin_3)
- net PT_F19: now also J42.38 (Pin_38)
- net PT_S6: now reaches J43.30 (Pin_30)
- net PT_S6: now also J42.11 (Pin_11)
- net PT_F5: now reaches J43.31 (Pin_31)
- net PT_F5: now also J42.10 (Pin_10)
- net PT_S5: now reaches J43.32 (Pin_32)
- net PT_S5: now also J42.9 (Pin_9)
- net PT_F4: now reaches J43.33 (Pin_33)
- net PT_F4: now also J42.8 (Pin_8)
- net PT_S4: now reaches J43.34 (Pin_34)
- net PT_S4: now also J42.7 (Pin_7)
- net PT_F3: now reaches J43.35 (Pin_35)
- net PT_F3: now also J42.6 (Pin_6)
- net PT_S3: now reaches J43.36 (Pin_36)
- net PT_S3: now also J42.5 (Pin_5)
- net PT_F2: now reaches J43.37 (Pin_37)
- net PT_F2: now also J42.4 (Pin_4)
- net PT_S2: now reaches J43.38 (Pin_38)
- net PT_S2: now also J42.3 (Pin_3)
- net PT_F1: now reaches J43.39 (Pin_39)
- net PT_F1: now also J42.2 (Pin_2)
- net PT_S19: now reaches J43.4 (Pin_4)
- net PT_S19: now also J42.37 (Pin_37)
- net PT_S1: now reaches J43.40 (Pin_40)
- net PT_S1: now also J42.1 (Pin_1)
- net PT_F18: now reaches J43.5 (Pin_5)
- net PT_F18: now also J42.36 (Pin_36)
- net PT_S18: now reaches J43.6 (Pin_6)
- net PT_S18: now also J42.35 (Pin_35)
- net PT_F17: now reaches J43.7 (Pin_7)
- net PT_F17: now also J42.34 (Pin_34)
- net PT_S17: now reaches J43.8 (Pin_8)
- net PT_S17: now also J42.33 (Pin_33)
- net PT_F16: now reaches J43.9 (Pin_9)
- net PT_F16: now also J42.32 (Pin_32)
Other:
- moved on the sheet: H1, H10, H11, H12, H13, H14, H15, H16, H17, H18, H19, H2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

Commit message: wip on sq pcb
Parts:
- removed H22, H23, H24, H25: MountingHole, custom_footprints:MountingHole_3.2mm_M3_wscrew, symbol Mechanical:MountingHole
- removed J42: Conn_02x20_Odd_Even, custom_footprints:TST-120-01-G-D, symbol Connector_Generic:Conn_02x20_Odd_Even
- added H22, H23, H24, H25: MountingHole_Pad, custom_footprints:MountingHole_3.2mm_M3_ISO7380_Pad_TopBottom_screw, symbol Mechanical:MountingHole_Pad
- added J44: Conn_02x25_Odd_Even, Connector_PinHeader_2.54mm:PinHeader_2x25_P2.54mm_Vertical, symbol Connector_Generic:Conn_02x25_Odd_Even
Connections:
- net F1: now also J41.40 (Pin_40); no longer J41.2 (Pin_2)
- net F10: now also J41.22 (Pin_22); no longer J41.20 (Pin_20)
- net F11: now also J41.20 (Pin_20); no longer J41.22 (Pin_22)
- net F12: now also J41.18 (Pin_18); no longer J41.24 (Pin_24)
- net F13: now also J41.16 (Pin_16); no longer J41.26 (Pin_26)
- net F14: now also J41.14 (Pin_14); no longer J41.28 (Pin_28)
- net F15: now also J41.12 (Pin_12); no longer J41.30 (Pin_30)
- net F16: now also J41.10 (Pin_10); no longer J41.32 (Pin_32)
- net F17: now also J41.8 (Pin_8); no longer J41.34 (Pin_34)
- net F18: now also J41.6 (Pin_6); no longer J41.36 (Pin_36)
- net F19: now also J41.4 (Pin_4); no longer J41.38 (Pin_38)
- net F2: now also J41.38 (Pin_38); no longer J41.4 (Pin_4)
- net F20: now also J41.2 (Pin_2); no longer J41.40 (Pin_40)
- net F3: now also J41.36 (Pin_36); no longer J41.6 (Pin_6)
- net F4: now also J41.34 (Pin_34); no longer J41.8 (Pin_8)
- net F5: now also J41.32 (Pin_32); no longer J41.10 (Pin_10)
- net F6: now also J41.30 (Pin_30); no longer J41.12 (Pin_12)
- net F7: now also J41.28 (Pin_28); no longer J41.14 (Pin_14)
- net F8: now also J41.26 (Pin_26); no longer J41.16 (Pin_16)
- net F9: now also J41.24 (Pin_24); no longer J41.18 (Pin_18)
- net PT_F1: now also J44.2 (Pin_2)
- net PT_F10: now also J44.20 (Pin_20)
- net PT_F11: now also J44.22 (Pin_22)
- net PT_F12: now also J44.24 (Pin_24)
- net PT_F13: now also J44.26 (Pin_26)
- net PT_F14: now also J44.28 (Pin_28)
- net PT_F15: now also J44.30 (Pin_30)
- net PT_F16: now also J44.32 (Pin_32)
- net PT_F17: now also J44.34 (Pin_34)
- net PT_F18: now also J44.36 (Pin_36)
- net PT_F19: now also J44.38 (Pin_38)
- net PT_F2: now also J44.4 (Pin_4)
- net PT_F20: now also J44.40 (Pin_40)
- net PT_F3: now also J44.6 (Pin_6)
- net PT_F4: now also J44.8 (Pin_8)
- net PT_F5: now also J44.10 (Pin_10)
- net PT_F6: now also J44.12 (Pin_12)
- net PT_F7: now also J44.14 (Pin_14)
- net PT_F8: now also J44.16 (Pin_16)
- net PT_F9: now also J44.18 (Pin_18)
- net PT_S1: now also J44.1 (Pin_1)
- net PT_S10: now also J44.19 (Pin_19)
- net PT_S11: now also J44.21 (Pin_21)
- net PT_S12: now also J44.23 (Pin_23)
- net PT_S13: now also J44.25 (Pin_25)
- net PT_S14: now also J44.27 (Pin_27)
- net PT_S15: now also J44.29 (Pin_29)
- net PT_S16: now also J44.31 (Pin_31)
- net PT_S17: now also J44.33 (Pin_33)
- net PT_S18: now also J44.35 (Pin_35)
- net PT_S19: now also J44.37 (Pin_37)
- net PT_S2: now also J44.3 (Pin_3)
- net PT_S20: now also J44.39 (Pin_39)
- net PT_S3: now also J44.5 (Pin_5)
- net PT_S4: now also J44.7 (Pin_7)
- net PT_S5: now also J44.9 (Pin_9)
- net PT_S6: now also J44.11 (Pin_11)
- net PT_S7: now also J44.13 (Pin_13)
- net PT_S8: now also J44.15 (Pin_15)
- net PT_S9: now also J44.17 (Pin_17)
- net S1: now also J41.39 (Pin_39); no longer J41.1 (Pin_1)
- net S10: now also J41.21 (Pin_21); no longer J41.19 (Pin_19)
- net S11: now also J41.19 (Pin_19); no longer J41.21 (Pin_21)
- net S12: now also J41.17 (Pin_17); no longer J41.23 (Pin_23)
- net S13: now also J41.15 (Pin_15); no longer J41.25 (Pin_25)
- net S14: now also J41.13 (Pin_13); no longer J41.27 (Pin_27)
- net S15: now also J41.11 (Pin_11); no longer J41.29 (Pin_29)
- net S16: now also J41.9 (Pin_9); no longer J41.31 (Pin_31)
- net S17: now also J41.7 (Pin_7); no longer J41.33 (Pin_33)
- net S18: now also J41.5 (Pin_5); no longer J41.35 (Pin_35)
- net S19: now also J41.3 (Pin_3); no longer J41.37 (Pin_37)
- net S2: now also J41.37 (Pin_37); no longer J41.3 (Pin_3)
- net S20: now also J41.1 (Pin_1); no longer J41.39 (Pin_39)
- net S3: now also J41.35 (Pin_35); no longer J41.5 (Pin_5)
- net S4: now also J41.33 (Pin_33); no longer J41.7 (Pin_7)
- net S5: now also J41.31 (Pin_31); no longer J41.9 (Pin_9)
- net S6: now also J41.29 (Pin_29); no longer J41.11 (Pin_11)
- net S7: now also J41.27 (Pin_27); no longer J41.13 (Pin_13)
- net S8: now also J41.25 (Pin_25); no longer J41.15 (Pin_15)
- net S9: now also J41.23 (Pin_23); no longer J41.17 (Pin_17)
- new net GND: H22.1, H23.1, H24.1, H25.1, J44.49 (Pin_49), J44.50 (Pin_50)
- no-connect marks 0 -> 8
Other:
- moved on the sheet: J41

Commit message: wip on sq pcb
Parts:
- added J42: Conn_01x02, Connector_Wire:SolderWire-0.1sqmm_1x02_P3.6mm_D0.4mm_OD1mm, symbol Connector_Generic:Conn_01x02
- J44: footprint Connector_PinHeader_2.54mm:PinHeader_2x25_P2.54mm_Vertical -> custom_footprints:TST-125-01-G-D
Connections:
- net GND: now also J44.45 (Pin_45), J44.46 (Pin_46), J44.47 (Pin_47), J44.48 (Pin_48)
- net RTD1: now reaches J44.41 (Pin_41)
- net RTD1: now also J44.43 (Pin_43), J42.1 (Pin_1)
- net RTD2: now reaches J44.42 (Pin_42)
- net RTD2: now also J44.44 (Pin_44), J42.2 (Pin_2)
- no-connect marks 8 -> 0
Changed lines of the file:
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@@
 (kicad_sch (version 20211123) (generator eeschema)
   (paper "A4")
-  (no_connect (at 33.02 93.98))
-  (no_connect (at 33.02 96.52))
-  (no_connect (at 33.02 99.06))
-  (no_connect (at 33.02 101.6))
-  (no_connect (at 45.72 101.6))
-  (no_connect (at 45.72 99.06))
-  (no_connect (at 45.72 96.52))
-  (no_connect (at 45.72 93.98))
+  (junction (at 31.75 101.6) (diameter 0) (color 0 0 0 0)
+  )
+  (junction (at 46.99 101.6) (diameter 0) (color 0 0 0 0)
+  )
+  (junction (at 31.75 104.14) (diameter 0) (color 0 0 0 0)
+  )
+  (junction (at 46.99 104.14) (diameter 0) (color 0 0 0 0)
+  )
   (polyline (pts (xy 192.405 108.585) (xy 192.405 118.745))
     (stroke (width 0) (type default) (color 0 0 0 0))
@@
     (stroke (width 0) (type default) (color 0 0 0 0))
   )
+  (wire (pts (xy 31.75 99.06) (xy 33.02 99.06))
+    (stroke (width 0) (type default) (color 0 0 0 0))
+  )
   (polyline (pts (xy 206.375 118.745) (xy 216.535 118.745))
     (stroke (width 0) (type default) (color 0 0 0 0))
@@
     (stroke (width 0) (type default) (color 0 0 0 0))
   )
+  (wire (pts (xy 46.99 104.14) (xy 46.99 101.6))
+    (stroke (width 0) (type default) (color 0 0 0 0))
+  )
   (polyline (pts (xy 202.565 137.795) (xy 202.565 127.635))
     (stroke (width 0) (type default) (color 0 0 0 0))
@@
     (stroke (width 0) (type default) (color 0 0 0 0))
   )
+  (wire (pts (xy 31.75 104.14) (xy 31.75 101.6))
+    (stroke (width 0) (type default) (color 0 0 0 0))
+  )
   (polyline (pts (xy 192.405 67.945) (xy 192.405 78.105))
     (stroke (width 0) (type default) (color 0 0 0 0))
@@
     (stroke (width 0) (type default) (color 0 0 0 0))
   )
+  (wire (pts (xy 31.75 101.6) (xy 31.75 99.06))
+    (stroke (width 0) (type default) (color 0 0 0 0))
+  )
   (polyline (pts (xy 202.565 78.105) (xy 202.565 67.945))
     (stroke (width 0) (type default) (color 0 0 0 0))
@@
     (stroke (width 0) (type default) (color 0 0 0 0))
   )
+  (wire (pts (xy 46.99 101.6) (xy 45.72 101.6))
+    (stroke (width 0) (type default) (color 0 0 0 0))
+  )
   (polyline (pts (xy 188.595 98.425) (xy 188.595 88.265))
     (stroke (width 0) (type default) (color 0 0 0 0))
@@
     (stroke (width 0) (type default) (color 0 0 0 0))
   )
+  (wire (pts (xy 31.75 101.6) (xy 33.02 101.6))
+    (stroke (width 0) (type default) (color 0 0 0 0))
+  )
   (polyline (pts (xy 192.405 78.105) (xy 202.565 78.105))
     (stroke (width 0) (type default) (color 0 0 0 0))
@@
     (stroke (width 0) (type default) (color 0 0 0 0))
   )
+  (wire (pts (xy 46.99 101.6) (xy 46.99 99.06))
+    (stroke (width 0) (type default) (color 0 0 0 0))
+  )
   (polyline (pts (xy 216.535 57.785) (xy 216.535 47.625))
     (stroke (width 0) (type default) (color 0 0 0 0))
   )
+  (wire (pts (xy 46.99 99.06) (xy 45.72 99.06))
+    (stroke (width 0) (type default) (color 0 0 0 0))
+  )
   (polyline (pts (xy 188.595 78.105) (xy 188.595 67.945))
     (stroke (width 0) (type default) (color 0 0 0 0))
@@
     (effects (font (size 1.27 1.27)) (justify left bottom))
   )
+  (label "RTD2" (at 45.72 96.52 0)
+    (effects (font (size 1.27 1.27)) (justify left bottom))
+  )
   (label "F7" (at 196.215 81.915 270)
     (effects (font (size 1.27 1.27)) (justify right bottom))
@@
     (effects (font (size 1.27 1.27)) (justify right bottom))
   )
+  (label "RTD2" (at 48.26 140.97 180)
+    (effects (font (size 1.27 1.27)) (justify right bottom))
+  )
   (label "F6" (at 210.185 81.915 270)
     (effects (font (size 1.27 1.27)) (justify right bottom))
@@
     (effects (font (size 1.27 1.27)) (justify right bottom))
   )
+  (label "RTD1" (at 48.26 138.43 180)
+    (effects (font (size 1.27 1.27)) (justify right bottom))
+  )
   (label "PT_F7" (at 45.72 58.42 0)
     (effects (font (size 1.27 1.27)) (justify left bottom))
@@
     (effects (font (size 1.27 1.27)) (justify right bottom))
   )
+  (label "RTD1" (at 33.02 96.52 180)
+    (effects (font (size 1.27 1.27)) (justify right bottom))
+  )
   (label "F8" (at 182.245 81.915 270)
     (effects (font (size 1.27 1.27)) (justify right bottom))
@@
     (effects (font (size 1.27 1.27)) (justify right bottom))
   )
+  (label "RTD2" (at 45.72 93.98 0)
+    (effects (font (size 1.27 1.27)) (justify left bottom))
+  )
   (label "PT_S12" (at 64.135 71.755 180)
     (effects (font (size 1.27 1.27)) (justify right bottom))
@@
   (label "PT_F16" (at 76.835 81.915 0)
     (effects (font (size 1.27 1.27)) (justify left bottom))
+  )
+  (label "RTD1" (at 33.02 93.98 180)
+    (effects (font (size 1.27 1.27)) (justify right bottom))
   )
   (symbol (lib_id "Connector_Generic:Conn_01x01") (at 182.245 56.515 90) (unit 1)
@@
     (property "Reference" "J44" (id 0) (at 39.37 36.83 0))
     (property "Value" "Conn_02x25_Odd_Even" (id 1) (at 39.37 39.37 0))
-    (property "Footprint" "Connector_PinHeader_2.54mm:PinHeader_2x25_P2.54mm_Vertical" (id 2) (at 38.1 73.66 0)
+    (property "Footprint" "custom_footprints:TST-125-01-G-D" (id 2) (at 38.1 73.66 0)
       (effects (font (size 1.27 1.27)) hide)
     )
@@
     (pin "1")
   )
+  (symbol (lib_id "Connector_Generic:Conn_01x02") (at 53.34 138.43 0) (unit 1)
+    (in_bom yes) (on_board yes) (fields_autoplaced)
+    (property "Reference" "J42" (id 0) (at 55.88 138.4299 0)
+      (effects (font (size 1.27 1.27)) (justify left))
+    )
+    (property "Value" "Conn_01x02" (id 1) (at 55.88 140.9699 0)
+      (effects (font (size 1.27 1.27)) (justify left))
+    )
+    (property "Footprint" "Connector_Wire:SolderWire-0.1sqmm_1x02_P3.6mm_D0.4mm_OD1mm" (id 2) (at 53.34 138.43 0)
+      (effects (font (size 1.27 1.27)) hide)
+    )
+    (property "Datasheet" "~" (id 3) (at 53.34 138.43 0)
+      (effects (font (size 1.27 1.27)) hide)
+    )
+    (pin "1")
+    (pin "2")
+  )
   (symbol (lib_id "Connector_Generic:Conn_01x01") (at 182.245 97.155 90) (unit 1)
     (in_bom yes) (on_board yes)
@@
       (reference "J41") (unit 1) (value "Conn_02x20_Odd_Even") (footprint "custom_footprints:TST-120-01-G-D")
     )
+    (path "/a7607c2a-6f7c-4bc0-821d-d10e70612f07"
+      (reference "J42") (unit 1) (value "Conn_01x02") (footprint "Connector_Wire:SolderWire-0.1sqmm_1x02_P3.6mm_D0.4mm_OD1mm")
+    )
     (path "/545ca384-b26e-43be-8c78-25a5055751b8"
       (reference "J43") (unit 1) (value "Conn_02x20_Odd_Even") (footprint "custom_footprints:TST-120-01-G-D")
     )
     (path "/167a03a6-ba64-4d94-a75b-ab3eeb832de3"
-      (reference "J44") (unit 1) (value "Conn_02x25_Odd_Even") (footprint "Connector_PinHeader_2.54mm:PinHeader_2x25_P2.54mm_Vertical")
-    )
-  )
+      (reference "J44") (unit 1) (value "Conn_02x25_Odd_Even") (footprint "custom_footprints:TST-125-01-G-D")
+    )
+  )
