File: sqpt/sqpt.kicad_pcb (KiCad board)
At the start: 2 copper layers, 30.5 x 84.1 mm, 21 parts, among them J1 Conn_02x25_Odd_Even, J2 Conn_02x05_Odd_Even, J3 Conn_02x20_Odd_Even

Commit message: sqpcbs layed out
Parts:
- moved JP13 1.12 mm to (7.90, 8.03)
- moved JP12 1.09 mm to (7.90, 5.53)
- moved JP11 1.06 mm to (7.90, 3.03)
- moved JP8 0.74 mm to (7.90, -8.72)
- moved JP9 0.74 mm to (7.90, -6.22)
- moved JP10 0.73 mm to (7.90, -3.72)
- moved JP14 0.48 mm to (3.65, 0.00)
- turned JP2 to -90 degrees
Connections:
- J1 pad 41: /RTD1 -> /RTD_A_S
- J1 pad 42: /RTD2 -> /RTD_A_F
- J1 pad 43: /RTD1 -> /RTD_B_S
- J1 pad 44: /RTD2 -> /RTD_B_F
Routing:
- net Earth_Protective: track 0.00 -> 274.3 mm, vias 0 -> 8
- net GND1: track 0.00 -> 66.9 mm, vias 0 -> 3
- net GND2: track 0.00 -> 62.0 mm, vias 0 -> 3
- net /RTD_A_S: track 0.00 -> 29.0 mm
- net /RTD_B_S: track 0.00 -> 25.4 mm
- net /RTD_A_F: track 0.00 -> 25.4 mm
- net /PT_S14: track 0.00 -> 23.4 mm
- net /PT_S16: track 0.00 -> 23.3 mm
- net /PT_S15: track 0.00 -> 23.2 mm
- net /PT_F10: track 0.00 -> 23.1 mm
- net /PT_F11: track 0.00 -> 23.0 mm
- net /PT_F12: track 0.00 -> 23.0 mm
- net /PT_S2: track 0.00 -> 22.8 mm
- net /PT_S20: track 0.00 -> 22.8 mm
- net /PT_S8: track 0.00 -> 22.8 mm
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- added copper zone on F.Cu, net GND
- added copper zone on B.Cu, net GND3
Other:
- copper layers 2 -> 4

Commit message: silk
Parts:
- added LOGO1: Logo_Open_Hardware_Small, custom_footprints:site_small, B.Cu at (5.65, -29.1)
- added LOGO2: Logo_Open_Hardware_Small, custom_footprints:site_small, F.Cu at (5.65, -29.1)
Other:
- board text added: "1823471"

Commit message: update silk
Other:
- board text added: "f74efd5"
- board text removed: "1823471"
Changed lines of the file:
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@@
   (gr_line (start 19.325 42.06) (end -7.217 42.06) (layer "Edge.Cuts") (width 0.1))
   (gr_arc (start 21.325 40.06) (mid 20.739214 41.474214) (end 19.325 42.06) (layer "Edge.Cuts") (width 0.1))
-  (gr_text "1823471" (at 7.75084 -22.52 90) (layer "B.SilkS")
+  (gr_text "f74efd5" (at 7.75084 -22.52 90) (layer "B.SilkS")
     (effects (font (size 1 1) (thickness 0.15)) (justify mirror))
   )
+  (gr_text "f74efd5" (at 8.15084 -36.22 90) (layer "F.SilkS")
+    (effects (font (size 1 1) (thickness 0.15)))
+  )
   (segment (start -4.70916 -34.94) (end -4.70916 -38.56) (width 1) (layer "B.Cu") (net 1))

Commit message: update silk
Other:
- board text added: "050ec02"
- board text removed: "f74efd5"
Changed lines of the file:
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@@
   (gr_line (start 19.325 42.06) (end -7.217 42.06) (layer "Edge.Cuts") (width 0.1))
   (gr_arc (start 21.325 40.06) (mid 20.739214 41.474214) (end 19.325 42.06) (layer "Edge.Cuts") (width 0.1))
-  (gr_text "f74efd5" (at 7.75084 -22.52 90) (layer "B.SilkS")
+  (gr_text "050ec02" (at 7.75084 -22.52 90) (layer "B.SilkS")
     (effects (font (size 1 1) (thickness 0.15)) (justify mirror))
   )
-  (gr_text "f74efd5" (at 8.15084 -36.22 90) (layer "F.SilkS")
+  (gr_text "050ec02" (at 8.15084 -36.22 90) (layer "F.SilkS")
     (effects (font (size 1 1) (thickness 0.15)))
   )
