File: switches/switches/switches.kicad_sch (KiCad schematic)
At the start: 53 parts, among them J1 Conn_02x06_Odd_Even, J10 Conn_01x01_Socket, J11 Conn_01x01_Socket, J12 Conn_01x01_Socket, J2 Conn_02x06_Odd_Even, J3 Conn_02x06_Odd_Even, J4 Conn_02x06_Odd_Even, J5 Conn_Coaxial, J6 Conn_Coaxial, J7 Conn_Coaxial, J8 Conn_Coaxial, J9 Conn_01x01_Socket, SW1 SW_Push_DPDT, SW10 SW_Push_DPDT, SW11 SW_Push_DPDT, SW12 SW_Push_DPDT, SW13 SW_Push_DPDT, SW14 SW_Push_DPDT, SW15 SW_Push_DPDT, SW16 SW_Push_DPDT, SW17 SW_Push_DPDT, SW18 SW_Push_DPDT, SW19 SW_Push_DPDT, SW2 SW_Push_DPDT, SW20 SW_Push_DPDT, SW3 SW_Push_DPDT, SW4 SW_Push_DPDT, SW5 SW_Push_DPDT, SW6 SW_Push_DPDT, SW7 SW_Push_DPDT, SW8 SW_Push_DPDT, SW9 SW_Push_DPDT

Commit message: spruce up the switches
Parts:
- SW1: renamed from SW2; Alternate Part # (none) -> L202011MS02Q; Part# (none) -> JS202011CQN
- SW10, SW11, SW20, SW7, SW8, SW9: Alternate Part # (none) -> L202011MS02Q; Part# (none) -> JS202011CQN
- SW12: renamed from SW13; Alternate Part # (none) -> L202011MS02Q; Part# (none) -> JS202011CQN
- SW13: renamed from SW15; Alternate Part # (none) -> L202011MS02Q; Part# (none) -> JS202011CQN
- SW14: renamed from SW17; Alternate Part # (none) -> L202011MS02Q; Part# (none) -> JS202011CQN
- SW15: renamed from SW19; Alternate Part # (none) -> L202011MS02Q; Part# (none) -> JS202011CQN
- SW16: renamed from SW12; Alternate Part # (none) -> L202011MS02Q; Part# (none) -> JS202011CQN
- SW17: renamed from SW14; Alternate Part # (none) -> L202011MS02Q; Part# (none) -> JS202011CQN
- SW18: renamed from SW16; Alternate Part # (none) -> L202011MS02Q; Part# (none) -> JS202011CQN
- SW19: renamed from SW18; Alternate Part # (none) -> L202011MS02Q; Part# (none) -> JS202011CQN
- SW2: renamed from SW3; Alternate Part # (none) -> L202011MS02Q; Part# (none) -> JS202011CQN
- SW3: renamed from SW4; Alternate Part # (none) -> L202011MS02Q; Part# (none) -> JS202011CQN
- SW4: renamed from SW5; Alternate Part # (none) -> L202011MS02Q; Part# (none) -> JS202011CQN
- SW5: renamed from SW6; Alternate Part # (none) -> L202011MS02Q; Part# (none) -> JS202011CQN
- SW6: renamed from SW1; Alternate Part # (none) -> L202011MS02Q; Part# (none) -> JS202011CQN
- renumbered J11 to J10, J8 to J11, J4 to J3, J3 to J4, J9 to J6, J6 to J7, J10 to J8, J7 to J9, JP13 to JP10, JP10 to JP11, JP14 to JP12, JP11 to JP13, JP15 to JP14, JP12 to JP15, JP5 to JP2, JP2 to JP3, JP6 to JP4, JP3 to JP5, JP7 to JP6, JP4 to JP7
Other:
- moved on the sheet: H1, H2, H3, H4, J10, J11, J12, J5, J6, J7, J8, J9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

Commit message: wip on switches
Parts:
- J10, J12, J6, J8: footprint Connector:Banana_Cliff_FCR7350x_S16N-PC_Horizontal -> custom:Banana_Cliff_FCR7350x_S16N-PC_Horizontal
Changed lines of the file:
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@@
       (effects (font (size 1.27 1.27)) (justify left))
     )
-    (property "Footprint" "Connector:Banana_Cliff_FCR7350x_S16N-PC_Horizontal" (at 261.62 124.46 0)
+    (property "Footprint" "custom:Banana_Cliff_FCR7350x_S16N-PC_Horizontal" (at 261.62 124.46 0)
       (effects (font (size 1.27 1.27)) hide)
     )
@@
       (effects (font (size 1.27 1.27)) (justify left))
     )
-    (property "Footprint" "Connector:Banana_Cliff_FCR7350x_S16N-PC_Horizontal" (at 261.62 90.17 0)
+    (property "Footprint" "custom:Banana_Cliff_FCR7350x_S16N-PC_Horizontal" (at 261.62 90.17 0)
       (effects (font (size 1.27 1.27)) hide)
     )
@@
       (effects (font (size 1.27 1.27)) (justify left))
     )
-    (property "Footprint" "Connector:Banana_Cliff_FCR7350x_S16N-PC_Horizontal" (at 261.62 111.76 0)
+    (property "Footprint" "custom:Banana_Cliff_FCR7350x_S16N-PC_Horizontal" (at 261.62 111.76 0)
       (effects (font (size 1.27 1.27)) hide)
     )
@@
       (effects (font (size 1.27 1.27)) (justify left))
     )
-    (property "Footprint" "Connector:Banana_Cliff_FCR7350x_S16N-PC_Horizontal" (at 261.62 100.33 0)
-      (effects (font (size 1.27 1.27)) hide)
-    )
+    (property "Footprint" "custom:Banana_Cliff_FCR7350x_S16N-PC_Horizontal" (at 261.62 100.33 0)
+      (effects (font (size 1.27 1.27)) hide)
+    )

Commit message: switches pcb complete
Parts:
- added SYM1, SYM2: Logo_Open_Hardware_Small, custom:site_small, symbol Graphic:Logo_Open_Hardware_Small
Changed lines of the file:
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@@
+    )
+  )
+  (symbol (lib_id "Graphic:Logo_Open_Hardware_Small") (at 213.36 175.26 0) (unit 1)
+    (in_bom no) (on_board yes) (dnp no) (fields_autoplaced)
+    (property "Reference" "SYM1" (at 213.36 168.275 0)
+      (effects (font (size 1.27 1.27)) hide)
+    )
+    (property "Value" "Logo_Open_Hardware_Small" (at 213.36 180.975 0)
+      (effects (font (size 1.27 1.27)) hide)
+    )
+    (property "Footprint" "custom:site_small" (at 213.36 175.26 0)
+      (effects (font (size 1.27 1.27)) hide)
+    )
+    (property "Datasheet" "~" (at 213.36 175.26 0)
+      (effects (font (size 1.27 1.27)) hide)
+    )
+    (property "Sim.Enable" "1" (at 213.36 175.26 0)
+      (effects (font (size 1.27 1.27)) hide)
+    )
+    (instances
+      (project "switches"
+        (path "/c79f6033-b458-4cb3-95d8-16a2aef64c3c"
+          (reference "SYM1") (unit 1)
+        )
+      )
     )
   )
@@
         )
       )
+    )
+  )
+  (symbol (lib_id "Graphic:Logo_Open_Hardware_Small") (at 261.62 175.26 0) (unit 1)
+    (in_bom no) (on_board yes) (dnp no) (fields_autoplaced)
+    (property "Reference" "SYM2" (at 261.62 168.275 0)
+      (effects (font (size 1.27 1.27)) hide)
+    )
+    (property "Value" "Logo_Open_Hardware_Small" (at 261.62 180.975 0)
+      (effects (font (size 1.27 1.27)) hide)
+    )
+    (property "Footprint" "custom:site_small" (at 261.62 175.26 0)
+      (effects (font (size 1.27 1.27)) hide)
+    )
+    (property "Datasheet" "~" (at 261.62 175.26 0)
+      (effects (font (size 1.27 1.27)) hide)
+    )
+    (property "Sim.Enable" "1" (at 261.62 175.26 0)
+      (effects (font (size 1.27 1.27)) hide)
+    )
+    (instances
+      (project "switches"
+        (path "/c79f6033-b458-4cb3-95d8-16a2aef64c3c"
+          (reference "SYM2") (unit 1)
+        )
+      )
