File: switches/switches/switches.kicad_pcb (KiCad board)
At the start: 2 copper layers, 203.2 x 114.3 mm, 53 parts, among them J1 Conn_02x06_Odd_Even, J10 Conn_01x01_Socket, J11 Conn_01x01_Socket, J12 Conn_01x01_Socket, J2 Conn_02x06_Odd_Even, J3 Conn_02x06_Odd_Even, J4 Conn_02x06_Odd_Even, J5 Conn_Coaxial, J6 Conn_Coaxial, J7 Conn_Coaxial, J8 Conn_Coaxial, J9 Conn_01x01_Socket, SW1 SW_Push_DPDT, SW10 SW_Push_DPDT, SW11 SW_Push_DPDT, SW12 SW_Push_DPDT, SW13 SW_Push_DPDT, SW14 SW_Push_DPDT, SW15 SW_Push_DPDT, SW16 SW_Push_DPDT, SW17 SW_Push_DPDT, SW18 SW_Push_DPDT, SW19 SW_Push_DPDT, SW2 SW_Push_DPDT, SW20 SW_Push_DPDT, SW3 SW_Push_DPDT, SW4 SW_Push_DPDT, SW5 SW_Push_DPDT, SW6 SW_Push_DPDT, SW7 SW_Push_DPDT, SW8 SW_Push_DPDT, SW9 SW_Push_DPDT

Commit message: spruce up the switches
Parts:
- JP1, JP16, JP8, JP9: moved to B.Cu
- JP10: renamed from JP13; moved to B.Cu
- JP11: renamed from JP10; moved to B.Cu
- JP12: renamed from JP14; moved to B.Cu
- JP13: renamed from JP11; moved to B.Cu
- JP14: renamed from JP15; moved to B.Cu
- JP15: renamed from JP12; moved to B.Cu
- JP2: renamed from JP5; moved to B.Cu
- JP3: renamed from JP2; moved to B.Cu
- JP4: renamed from JP6; moved to B.Cu
- JP5: renamed from JP3; moved to B.Cu
- JP6: renamed from JP7; moved to B.Cu
- JP7: renamed from JP4; moved to B.Cu
- moved SW15 128.3 mm to (234.2, 51.7), turned to 90 degrees
- moved TP1 126.8 mm to (57.3, 17.0), turned to 90 degrees
- moved SW13 123.3 mm to (198.2, 51.7), turned to 90 degrees
- moved SW20 122.1 mm to (234.2, 71.7), turned to 90 degrees
- moved SW14 106.5 mm to (216.2, 51.7), turned to 90 degrees
- moved JP1 104.0 mm to (64.2, 43.0), turned to 90 degrees
- moved SW12 101.9 mm to (180.2, 51.7), turned to 90 degrees
- moved JP5 101.4 mm to (64.2, 63.0), turned to 90 degrees
- moved SW19 100.7 mm to (216.2, 71.7), turned to 90 degrees
- moved SW5 92.4 mm to (144.2, 51.7), turned to 90 degrees
- moved SW17 92.2 mm to (180.2, 71.7), turned to 90 degrees
- moved JP3 85.5 mm to (82.2, 51.0), turned to 90 degrees
- moved JP7 83.0 mm to (82.2, 71.0), turned to 90 degrees
- moved SW11 80.7 mm to (162.2, 51.7), turned to 90 degrees
- moved SW4 79.5 mm to (126.2, 51.7), turned to 90 degrees
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- renumbered J11 to J10, J8 to J11, J4 to J3, J3 to J4, J9 to J6, J6 to J7, J10 to J8, J7 to J9, SW2 to SW1, SW13 to SW12, SW15 to SW13, SW17 to SW14, SW19 to SW15, SW12 to SW16, SW14 to SW17, SW16 to SW18, SW18 to SW19, SW3 to SW2, SW4 to SW3, SW5 to SW4, SW6 to SW5, SW1 to SW6
Routing:
- net Earth_Clean: track 0.00 -> 416.7 mm
- net /B_V_EV_T: track 0.00 -> 144.8 mm
- net /A_V_EV_T: track 0.00 -> 143.8 mm
- net /B_I_EV_T: track 0.00 -> 136.7 mm
- net /A_I_EV_T: track 0.00 -> 135.3 mm
- net /B_I_2: track 0.00 -> 116.0 mm
- net /A_I_2: track 0.00 -> 115.6 mm
- net /A_V_2: track 0.00 -> 113.2 mm
- net /B_V_2: track 0.00 -> 112.3 mm
- net /A_V_OD_T: track 0.00 -> 101.8 mm
- net /A_I_4: track 0.00 -> 100.5 mm
- net /B_I_4: track 0.00 -> 99.9 mm
- net /A_V_4: track 0.00 -> 97.7 mm
- net /A_I_OD_T: track 0.00 -> 97.2 mm
- net /B_V_4: track 0.00 -> 95.2 mm
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- added copper zone on F.Cu, net /FORCE_HI
- added copper zone on B.Cu, net /FORCE_LO
- added copper zone on In1.Cu, net /SENSE_HI
- added copper zone on In2.Cu, net /SENSE_LO
Other:
- board size 203.2 x 114.3 mm -> 203.2 x 81.3 mm
- copper layers 2 -> 4
- board text added: "1"
- board text added: "2"
- board text added: "3"
- board text added: "4"
- board text added: "5"
- board text added: "6"
- board text added: "A1"
- board text added: "A2"
- board text added: "A3"
- board text added: "A4"
- board text added: "A5"
- board text added: "A6"
- board text added: "AC1"
- board text added: "AC2"
- board text added: "AC3"
- board text added: "AC4"
- board text added: "B1"
- board text added: "B2"
- board text added: "B3"
- board text added: "B4"
- board text added: "B5"
- board text added: "B6"
- board text added: "BC1"
- board text added: "BC2"
- board text added: "BC3"
- board text added: "BC4"
- board text added: "EVEN"
- board text added: "FORCE HI"
- board text added: "FORCE LO"
- board text added: "ODD"
- board text added: "OFF"
- board text added: "ON"
- board text added: "SENSE HI"
- board text added: "SENSE LO"
- board text added: "SLOT A"
- board text added: "SLOT B"

Commit message: wip on switches
Parts:
- J10, J12, J6, J8: footprint Connector:Banana_Cliff_FCR7350x_S16N-PC_Horizontal -> custom:Banana_Cliff_FCR7350x_S16N-PC_Horizontal
- JP9: moved to F.Cu
- moved JP9 13.3 mm to (167.5, 42.0), turned to 180 degrees
- moved JP4 9.90 mm to (147.2, 44.0), turned to -90 degrees
- moved JP14 7.99 mm to (232.2, 68.3)
- moved JP1 7.81 mm to (70.2, 48.0)
- moved JP10 7.81 mm to (232.2, 48.0)
- moved JP13 7.81 mm to (160.2, 68.0)
- moved JP5 7.81 mm to (70.2, 68.0)
- moved JP6 7.81 mm to (142.2, 68.0)
- moved JP2 7.78 mm to (142.0, 48.3)
- moved JP11 5.83 mm to (167.2, 48.0)
- moved JP12 5.83 mm to (239.2, 48.0)
- moved JP15 5.83 mm to (167.2, 68.0)
- moved JP16 5.83 mm to (239.2, 68.0)
- moved JP3 5.83 mm to (77.2, 48.0)
- moved JP7 5.83 mm to (77.2, 68.0)
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Routing:
- net /B_V_OD_T: track 62.2 -> 177.2 mm
- net /B_V_1: track 41.8 -> 135.3 mm
- net /B_V_3: track 36.4 -> 109.8 mm
- net /A_V_OD_T: track 101.8 -> 160.3 mm
- net /A_V_1: track 70.6 -> 128.6 mm
- net /A_V_EV_T: track 143.8 -> 197.4 mm
- net /A_V_2: track 113.2 -> 164.2 mm
- net /A_V_3: track 56.1 -> 103.1 mm
- net /B_V_5: track 40.5 -> 84.3 mm
- net /A_V_4: track 97.7 -> 138.7 mm
- net /B_V_EV_T: track 144.8 -> 185.0 mm
- net /B_V_2: track 112.3 -> 152.3 mm
- net /A_V_6: track 81.2 -> 113.1 mm
- net /B_V_4: track 95.2 -> 126.6 mm
- net /A_V_5: track 47.3 -> 77.6 mm
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
Commit message: switches pcb complete
Parts:
- added SYM1: Logo_Open_Hardware_Small, custom:site_small, F.Cu at (198.2, 37.0)
- added SYM2: Logo_Open_Hardware_Small, custom:site_small, B.Cu at (198.2, 37.0)
- JP9: moved to B.Cu
- moved JP9 13.4 mm to (164.2, 55.0), turned to 90 degrees
Routing:
- net /A_V_OD_T: track 160.3 -> 97.5 mm
- net /SENSE_LO: track 21.9 -> 23.5 mm
- net /A_V_EV_T: track 197.4 -> 198.5 mm
- net /A_V_4: track 138.7 -> 139.8 mm
- net /A_V_2: track 164.2 -> 165.3 mm
- net /A_V_6: track 113.1 -> 114.3 mm
- net /B_V_OD_T: track 177.2 -> 176.3 mm
- net /A_V_EV_B: track 85.3 -> 84.8 mm
Other:
- board text added: "6918b29"

Commit message: update silk
Other:
- board text added: "775fbec"
- board text removed: "6918b29"
Changed lines of the file:
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@@
   (gr_arc (start 52.179998 6.839998) (mid 53.667896 3.247896) (end 57.259998 1.759998)
     (stroke (width 0.1) (type default)) (layer "Edge.Cuts"))
-  (gr_text "6918b29" (at 214.23 37.985) (layer "B.SilkS")
+  (gr_text "775fbec" (at 214.23 37.985) (layer "B.SilkS")
     (effects (font (size 1.5 1.5) (thickness 0.3) bold) (justify bottom mirror))
   )
@@
     (effects (font (size 3 3) (thickness 0.6) bold))
   )
-  (gr_text "6918b29" (at 214.23 37.985) (layer "F.SilkS")
+  (gr_text "775fbec" (at 214.23 37.985) (layer "F.SilkS")
     (effects (font (size 1.5 1.5) (thickness 0.3) bold) (justify bottom))
   )
