File: switches/switches.kicad_pcb (KiCad board)
At the start: 4 copper layers, 203.2 x 81.3 mm, 55 parts, among them J1 Conn_02x06_Odd_Even, J10 Conn_01x01_Socket, J11 Conn_Coaxial, J12 Conn_01x01_Socket, J2 Conn_02x06_Odd_Even, J3 Conn_02x06_Odd_Even, J4 Conn_02x06_Odd_Even, J5 Conn_Coaxial, J6 Conn_01x01_Socket, J7 Conn_Coaxial, J8 Conn_01x01_Socket, J9 Conn_Coaxial, SW1 SW_Push_DPDT, SW10 SW_Push_DPDT, SW11 SW_Push_DPDT, SW12 SW_Push_DPDT, SW13 SW_Push_DPDT, SW14 SW_Push_DPDT, SW15 SW_Push_DPDT, SW16 SW_Push_DPDT, SW17 SW_Push_DPDT, SW18 SW_Push_DPDT, SW19 SW_Push_DPDT, SW2 SW_Push_DPDT, SW20 SW_Push_DPDT, SW3 SW_Push_DPDT, SW4 SW_Push_DPDT, SW5 SW_Push_DPDT, SW6 SW_Push_DPDT, SW7 SW_Push_DPDT, SW8 SW_Push_DPDT, SW9 SW_Push_DPDT

Commit message: update silk
Other:
- board text added: "b8007ef"
- board text removed: "775fbec"
Changed lines of the file:
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@@
       (outputformat 1)
       (mirror false)
-      (drillshape 1)
+      (drillshape 0)
       (scaleselection 1)
-      (outputdirectory "")
+      (outputdirectory "output")
     )
   )
@@
     (fp_line (start 13.28 17.8) (end 4.38 17.8)
       (stroke (width 0.1) (type solid)) (layer "F.Fab"))
-    (pad "1" thru_hole roundrect (at 0 0 90) (size 1.7 1.7) (drill 1) (layers "*.Cu" "*.Mask") (roundrect_rratio 0.147059)
+    (pad "1" thru_hole roundrect (at 0 0 90) (size 1.7 1.7) (drill 1) (layers "*.Cu" "*.Mask") (roundrect_rratio 0.1470588235)
       (net 25 "/B_I_EV_T") (pinfunction "Pin_1") (pintype "passive"))
     (pad "2" thru_hole circle (at 2.54 0 90) (size 1.7 1.7) (drill 1) (layers "*.Cu" "*.Mask")
@@
     (pad "1" thru_hole circle (at 0 0 270) (size 3.5 3.5) (drill 2.2) (layers "*.Cu" "*.Mask")
       (net 52 "/SENSE_LO") (pinfunction "Pin_1") (pintype "passive"))
-    (model "${KIPRJMOD}/../../shared_libs/3d/FCR7350.stp"
+    (model "${KIPRJMOD}/../shared_libs/3d/FCR7350.stp"
       (offset (xyz -13.5 0 6.3))
       (scale (xyz 1 1 1))
@@
     (pad "1" thru_hole circle (at 0 0 270) (size 3.5 3.5) (drill 2.2) (layers "*.Cu" "*.Mask")
       (net 49 "/FORCE_HI") (pinfunction "Pin_1") (pintype "passive"))
-    (model "${KIPRJMOD}/../../shared_libs/3d/FCR7350.stp"
+    (model "${KIPRJMOD}/../shared_libs/3d/FCR7350.stp"
       (offset (xyz -13.5 0 6.3))
       (scale (xyz 1 1 1))
@@
     (fp_line (start 13.28 17.8) (end 4.38 17.8)
       (stroke (width 0.1) (type solid)) (layer "F.Fab"))
-    (pad "1" thru_hole roundrect (at 0 0 90) (size 1.7 1.7) (drill 1) (layers "*.Cu" "*.Mask") (roundrect_rratio 0.147059)
+    (pad "1" thru_hole roundrect (at 0 0 90) (size 1.7 1.7) (drill 1) (layers "*.Cu" "*.Mask") (roundrect_rratio 0.1470588235)
       (net 1 "/A_I_OD_T") (pinfunction "Pin_1") (pintype "passive"))
     (pad "2" thru_hole circle (at 2.54 0 90) (size 1.7 1.7) (drill 1) (layers "*.Cu" "*.Mask")
@@
     (fp_line (start 13.28 17.8) (end 4.38 17.8)
       (stroke (width 0.1) (type solid)) (layer "F.Fab"))
-    (pad "1" thru_hole roundrect (at 0 0 90) (size 1.7 1.7) (drill 1) (layers "*.Cu" "*.Mask") (roundrect_rratio 0.147059)
+    (pad "1" thru_hole roundrect (at 0 0 90) (size 1.7 1.7) (drill 1) (layers "*.Cu" "*.Mask") (roundrect_rratio 0.1470588235)
       (net 37 "/B_I_OD_T") (pinfunction "Pin_1") (pintype "passive"))
     (pad "2" thru_hole circle (at 2.54 0 90) (size 1.7 1.7) (drill 1) (layers "*.Cu" "*.Mask")
@@
     (pad "1" thru_hole circle (at 0 0 270) (size 3.5 3.5) (drill 2.2) (layers "*.Cu" "*.Mask")
       (net 53 "/FORCE_LO") (pinfunction "Pin_1") (pintype "passive"))
-    (model "${KIPRJMOD}/../../shared_libs/3d/FCR7350.stp"
+    (model "${KIPRJMOD}/../shared_libs/3d/FCR7350.stp"
       (offset (xyz -13.5 0 6.3))
       (scale (xyz 1 1 1))
@@
     (pad "1" thru_hole circle (at 0 0 270) (size 3.5 3.5) (drill 2.2) (layers "*.Cu" "*.Mask")
       (net 51 "/SENSE_HI") (pinfunction "Pin_1") (pintype "passive"))
-    (model "${KIPRJMOD}/../../shared_libs/3d/FCR7350.stp"
+    (model "${KIPRJMOD}/../shared_libs/3d/FCR7350.stp"
       (offset (xyz -13.5 0 6.3))
       (scale (xyz 1 1 1))
@@
     (fp_line (start 13.28 17.8) (end 4.38 17.8)
       (stroke (width 0.1) (type solid)) (layer "F.Fab"))
-    (pad "1" thru_hole roundrect (at 0 0 90) (size 1.7 1.7) (drill 1) (layers "*.Cu" "*.Mask") (roundrect_rratio 0.147059)
+    (pad "1" thru_hole roundrect (at 0 0 90) (size 1.7 1.7) (drill 1) (layers "*.Cu" "*.Mask") (roundrect_rratio 0.1470588235)
       (net 13 "/A_I_EV_T") (pinfunction "Pin_1") (pintype "passive"))
     (pad "2" thru_hole circle (at 2.54 0 90) (size 1.7 1.7) (drill 1) (layers "*.Cu" "*.Mask")
@@
   (gr_arc (start 52.179998 6.839998) (mid 53.667896 3.247896) (end 57.259998 1.759998)
     (stroke (width 0.1) (type default)) (layer "Edge.Cuts"))
-  (gr_text "775fbec" (at 214.23 37.985) (layer "B.SilkS")
+  (gr_text "b8007ef" (at 214.23 37.985) (layer "B.SilkS")
     (effects (font (size 1.5 1.5) (thickness 0.3) bold) (justify bottom mirror))
   )
@@
     (effects (font (size 3 3) (thickness 0.6) bold))
   )
-  (gr_text "775fbec" (at 214.23 37.985) (layer "F.SilkS")
+  (gr_text "b8007ef" (at 214.23 37.985) (layer "F.SilkS")
     (effects (font (size 1.5 1.5) (thickness 0.3) bold) (justify bottom))
   )
