File: hoye_holder/hoye_holder.kicad_pcb (KiCad board)
At the start: 2 copper layers, 30 x 30 mm, 24 parts, among them J1 Conn_02x08_Odd_Even, J10 Conn_01x01, J11 Conn_01x01, J12 Conn_01x01, J13 Conn_01x01, J14 Conn_01x01, J15 Conn_01x01, J16 Conn_01x01, J17 Conn_01x01, J18 Conn_01x01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

Commit message: update silk
Other:
- board text added: "b8007ef"
- board text removed: "03d2124"
Changed lines of the file:
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@@
     (effects (font (size 1 1) (thickness 0.15)) (justify mirror))
   )
-  (gr_text "03d2124" (at 154.7 94.14 180) (layer "B.SilkS")
+  (gr_text "b8007ef" (at 154.7 94.14 180) (layer "B.SilkS")
     (effects (font (size 0.5 0.5) (thickness 0.0625)) (justify mirror))
   )
@@
     (effects (font (size 1 1) (thickness 0.15)))
   )
-  (gr_text "03d2124" (at 154.7 94.14) (layer "F.SilkS")
+  (gr_text "b8007ef" (at 154.7 94.14) (layer "F.SilkS")
     (effects (font (size 0.5 0.5) (thickness 0.0625)))
   )

Commit message: plotted
Changed lines of the file:
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@@
       (outputformat 1)
       (mirror false)
-      (drillshape 1)
+      (drillshape 0)
       (scaleselection 1)
-      (outputdirectory "")
+      (outputdirectory "output")
     )
   )
@@
     (fp_line (start 5.72 5.1) (end 5.72 -22.88)
       (stroke (width 0.1) (type solid)) (layer "B.Fab"))
-    (pad "1" thru_hole roundrect (at 0 0 270) (size 1.7 1.7) (drill 1) (layers "*.Cu" "*.Mask") (roundrect_rratio 0.147059)
+    (pad "1" thru_hole roundrect (at 0 0 270) (size 1.7 1.7) (drill 1) (layers "*.Cu" "*.Mask") (roundrect_rratio 0.1470588235)
       (net 23 "unconnected-(J2-Pin_1-Pad1)") (pinfunction "Pin_1") (pintype "passive+no_connect"))
     (pad "2" thru_hole circle (at 2.54 0 270) (size 1.7 1.7) (drill 1) (layers "*.Cu" "*.Mask")
@@
     (fp_line (start 5.72 5.1) (end 5.72 -22.88)
       (stroke (width 0.1) (type solid)) (layer "B.Fab"))
-    (pad "1" thru_hole roundrect (at 0 0 270) (size 1.7 1.7) (drill 1) (layers "*.Cu" "*.Mask") (roundrect_rratio 0.147059)
+    (pad "1" thru_hole roundrect (at 0 0 270) (size 1.7 1.7) (drill 1) (layers "*.Cu" "*.Mask") (roundrect_rratio 0.1470588235)
       (net 21 "unconnected-(J1-Pin_1-Pad1)") (pinfunction "Pin_1") (pintype "passive+no_connect"))
     (pad "2" thru_hole circle (at 2.54 0 270) (size 1.7 1.7) (drill 1) (layers "*.Cu" "*.Mask")
