File: yen_holder/yen_holder.kicad_pcb (KiCad board)
At the start: 2 copper layers, 30 x 30 mm, 24 parts, among them J1 Conn_02x08_Odd_Even, J10 Conn_01x01, J11 Conn_01x01, J12 Conn_01x01, J13 Conn_01x01, J14 Conn_01x01, J15 Conn_01x01, J16 Conn_01x01, J17 Conn_01x01, J18 Conn_01x01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

Commit message: new holder pcbs
Other:
- board text removed: "H"
Changed lines of the file:
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@@
     )
     (pad_to_mask_clearance 0)
-    (grid_origin 127 94.14)
+    (grid_origin 135.65 90.33)
     (pcbplotparams
       (layerselection 0x00010fc_ffffffff)
@@
   (net 31 "unconnected-(J1-Pin_16-Pad16)")
   (footprint "custom:S25-022+P25-4023_OFF" (layer "F.Cu")
-    (at 135.67 82.14)
+    (at 135.65 82.14)
     (descr "S25-022+P25-4023 OFFSET")
     (tags "harwin spring pins offset")
@@
   )
   (footprint "custom:S25-022+P25-4023_OFF" (layer "F.Cu")
-    (at 133.09 82.14)
+    (at 133.11 82.14)
     (descr "S25-022+P25-4023 OFFSET")
     (tags "harwin spring pins offset")
@@
   )
   (footprint "custom:S25-022+P25-4023_OFF" (layer "F.Cu")
-    (at 130.59 82.14)
+    (at 130.57 82.14)
     (descr "S25-022+P25-4023 OFFSET")
     (tags "harwin spring pins offset")
@@
   )
   (footprint "custom:S25-022+P25-4023_OFF" (layer "F.Cu")
-    (at 140.75 106.14)
+    (at 140.73 106.14)
     (descr "S25-022+P25-4023 OFFSET")
     (tags "harwin spring pins offset")
@@
   )
   (footprint "custom:S25-022+P25-4023_OFF" (layer "F.Cu")
-    (at 138.17 82.14)
+    (at 138.19 82.14)
     (descr "S25-022+P25-4023 OFFSET")
     (tags "harwin spring pins offset")
@@
   )
   (footprint "custom:S25-022+P25-4023_OFF" (layer "F.Cu")
-    (at 150.91 106.14)
+    (at 150.89 106.14)
     (descr "S25-022+P25-4023 OFFSET")
     (tags "harwin spring pins offset")
@@
   )
   (footprint "custom:S25-022+P25-4023_OFF" (layer "F.Cu")
-    (at 145.83 106.14)
+    (at 145.81 106.14)
     (descr "S25-022+P25-4023 OFFSET")
     (tags "harwin spring pins offset")
@@
   )
   (footprint "custom:S25-022+P25-4023_OFF" (layer "F.Cu")
-    (at 148.33 106.14)
+    (at 148.35 106.14)
     (descr "S25-022+P25-4023 OFFSET")
     (tags "harwin spring pins offset")
@@
   )
   (footprint "custom:S25-022+P25-4023_OFF" (layer "F.Cu")
-    (at 145.83 82.14)
+    (at 145.81 82.14)
     (descr "S25-022+P25-4023 OFFSET")
     (tags "harwin spring pins offset")
@@
   )
   (footprint "custom:S25-022+P25-4023_OFF" (layer "F.Cu")
-    (at 135.67 106.14)
+    (at 135.65 106.14)
     (descr "S25-022+P25-4023 OFFSET")
     (tags "harwin spring pins offset")
@@
   )
   (footprint "custom:S25-022+P25-4023_OFF" (layer "F.Cu")
-    (at 130.59 106.14)
+    (at 130.57 106.14)
     (descr "S25-022+P25-4023 OFFSET")
     (tags "harwin spring pins offset")
@@
   )
   (footprint "custom:S25-022+P25-4023_OFF" (layer "F.Cu")
-    (at 153.41 82.14)
+    (at 153.43 82.14)
     (descr "S25-022+P25-4023 OFFSET")
     (tags "harwin spring pins offset")
@@
   )
   (footprint "custom:S25-022+P25-4023_OFF" (layer "F.Cu")
-    (at 143.25 82.14)
+    (at 143.27 82.14)
     (descr "S25-022+P25-4023 OFFSET")
     (tags "harwin spring pins offset")
@@
   )
   (footprint "custom:S25-022+P25-4023_OFF" (layer "F.Cu")
-    (at 140.75 82.14)
+    (at 140.73 82.14)
     (descr "S25-022+P25-4023 OFFSET")
     (tags "harwin spring pins offset")
@@
   )
   (footprint "custom:S25-022+P25-4023_OFF" (layer "F.Cu")
-    (at 138.17 106.14)
+    (at 138.19 106.14)
     (descr "S25-022+P25-4023 OFFSET")
     (tags "harwin spring pins offset")
@@
   )
   (footprint "custom:S25-022+P25-4023_OFF" (layer "F.Cu")
-    (at 150.91 82.14)
+    (at 150.89 82.14)
     (descr "S25-022+P25-4023 OFFSET")
     (tags "harwin spring pins offset")
@@
   )
   (footprint "custom:S25-022+P25-4023_OFF" (layer "F.Cu")
-    (at 153.41 106.14)
+    (at 153.43 106.14)
     (descr "S25-022+P25-4023 OFFSET")
     (tags "harwin spring pins offset")
@@
   )
   (footprint "custom:S25-022+P25-4023_OFF" (layer "F.Cu")
-    (at 133.09 106.14)
+    (at 133.11 106.14)
     (descr "S25-022+P25-4023 OFFSET")
     (tags "harwin spring pins offset")
@@
   )
   (footprint "custom:S25-022+P25-4023_OFF" (layer "F.Cu")
-    (at 143.25 106.14)
+    (at 143.27 106.14)
     (descr "S25-022+P25-4023 OFFSET")
     (tags "harwin spring pins offset")
@@
   )
   (footprint "custom:S25-022+P25-4023_OFF" (layer "F.Cu")
-    (at 148.33 82.14)
+    (at 148.35 82.14)
     (descr "S25-022+P25-4023 OFFSET")
     (tags "harwin spring pins offset")
@@
     (effects (font (size 1 1) (thickness 0.15)) (justify mirror))
   )
-  (gr_text "H" (at 128 94.14 90) (layer "B.SilkS")
-    (effects (font (size 1 1) (thickness 0.15)) (justify mirror))
-  )
   (gr_text "5" (at 147.08 108.11) (layer "B.SilkS")
     (effects (font (size 1 1) (thickness 0.15)) (justify mirror))
   )
-  (gr_text "H" (at 128 94.14 -90) (layer "F.SilkS")
-    (effects (font (size 1 1) (thickness 0.15)))
-  )
   (gr_text "03d2124" (at 154.7 94.14) (layer "F.SilkS")

Commit message: update silk
Other:
- board text added: "b8007ef"
- board text removed: "03d2124"
Changed lines of the file:
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@@
     (effects (font (size 1 1) (thickness 0.15)) (justify mirror))
   )
-  (gr_text "03d2124" (at 154.7 94.14 180) (layer "B.SilkS")
+  (gr_text "b8007ef" (at 154.7 94.14 180) (layer "B.SilkS")
     (effects (font (size 0.5 0.5) (thickness 0.0625)) (justify mirror))
   )
@@
     (effects (font (size 1 1) (thickness 0.15)) (justify mirror))
   )
-  (gr_text "03d2124" (at 154.7 94.14) (layer "F.SilkS")
+  (gr_text "b8007ef" (at 154.7 94.14) (layer "F.SilkS")
     (effects (font (size 0.5 0.5) (thickness 0.0625)))
   )

Commit message: plotted
Changed lines of the file:
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@@
       (outputformat 1)
       (mirror false)
-      (drillshape 1)
+      (drillshape 0)
       (scaleselection 1)
-      (outputdirectory "")
+      (outputdirectory "output")
     )
   )
@@
     (fp_line (start 5.72 5.1) (end 5.72 -22.88)
       (stroke (width 0.1) (type solid)) (layer "B.Fab"))
-    (pad "1" thru_hole roundrect (at 0 0 270) (size 1.7 1.7) (drill 1) (layers "*.Cu" "*.Mask") (roundrect_rratio 0.147059)
+    (pad "1" thru_hole roundrect (at 0 0 270) (size 1.7 1.7) (drill 1) (layers "*.Cu" "*.Mask") (roundrect_rratio 0.1470588235)
       (net 23 "unconnected-(J2-Pin_1-Pad1)") (pinfunction "Pin_1") (pintype "passive+no_connect"))
     (pad "2" thru_hole circle (at 2.54 0 270) (size 1.7 1.7) (drill 1) (layers "*.Cu" "*.Mask")
@@
     (fp_line (start 5.72 5.1) (end 5.72 -22.88)
       (stroke (width 0.1) (type solid)) (layer "B.Fab"))
-    (pad "1" thru_hole roundrect (at 0 0 270) (size 1.7 1.7) (drill 1) (layers "*.Cu" "*.Mask") (roundrect_rratio 0.147059)
+    (pad "1" thru_hole roundrect (at 0 0 270) (size 1.7 1.7) (drill 1) (layers "*.Cu" "*.Mask") (roundrect_rratio 0.1470588235)
       (net 21 "unconnected-(J1-Pin_1-Pad1)") (pinfunction "Pin_1") (pintype "passive+no_connect"))
     (pad "2" thru_hole circle (at 2.54 0 270) (size 1.7 1.7) (drill 1) (layers "*.Cu" "*.Mask")

Commit message: change some logos
Parts:
- SYM1, SYM2: footprint custom:site_small -> custom:logo_small
