File: lightboard/lightboard.kicad_pcb (KiCad board)
At the start: 2 copper layers, 90 x 90 mm, 38 parts, among them J1 Conn_01x02, J2 Conn_01x01, J3 Conn_01x01, J4 Conn_01x02, J5 Conn_01x01, J6 Conn_01x01, Q1 FTZ651, U1 AL5817

Commit message: contact checker fixups
Parts:
- H1, H2, H3, H4: footprint MountingHole:MountingHole_4.3mm_M4_ISO7380_Pad -> MountingHole:MountingHole_4mm_Pad
- J1, J4: footprint Connector_Coaxial:BNC_TEConnectivity_1478204_Vertical -> Connector_Coaxial:BNC_TEConnectivity_1478035_Horizontal
- moved J1 38.6 mm to (36.0, 0.00), turned to -90 degrees
- moved J4 38.6 mm to (-36.0, 0.00), turned to 90 degrees
- moved J6 19.0 mm to (19.0, -40.0)
- moved J2 15.0 mm to (0.00, -40.0)
- moved H1 8.49 mm to (-36.0, -36.0)
- moved H2 8.49 mm to (-36.0, 36.0)
- moved H3 8.49 mm to (36.0, 36.0)
- moved H4 8.49 mm to (36.0, -36.0)
- moved J3 4.00 mm to (-19.0, -40.0)
- moved J5 1.00 mm to (-41.0, -28.0)
Routing:
- net /Vin: track 79.0 -> 43.0 mm, vias 1 -> 0
- net Net-(D3-A): track 69.8 -> 42.0 mm
- net Net-(D5-K): track 41.0 -> 62.2 mm
- net VCC: track 0.00 -> 2.50 mm
- net Net-(J5-Pin_1): track 35.0 -> 34.0 mm
