File: lightboard/lightboard.kicad_sch (KiCad schematic)
At the start: 38 parts, among them J1 Conn_01x02, J2 Conn_01x01, J3 Conn_01x01, J4 Conn_01x02, J5 Conn_01x01, J6 Conn_01x01, Q1 FTZ651, U1 AL5817

Commit message: contact checker fixups
Parts:
- H1, H2, H3, H4: footprint MountingHole:MountingHole_4.3mm_M4_ISO7380_Pad -> MountingHole:MountingHole_4mm_Pad
- J1, J4: footprint Connector_Coaxial:BNC_TEConnectivity_1478204_Vertical -> Connector_Coaxial:BNC_TEConnectivity_1478035_Horizontal
Changed lines of the file:
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@@
       (effects (font (size 1.27 1.27)) hide)
     )
-    (property "Footprint" "Connector_Coaxial:BNC_TEConnectivity_1478204_Vertical" (at 88.265 100.33 0)
+    (property "Footprint" "Connector_Coaxial:BNC_TEConnectivity_1478035_Horizontal" (at 88.265 100.33 0)
       (effects (font (size 1.27 1.27)) hide)
     )
@@
       (effects (font (size 1.27 1.27)) (justify left))
     )
-    (property "Footprint" "MountingHole:MountingHole_4.3mm_M4_ISO7380_Pad" (at 64.77 135.255 0)
+    (property "Footprint" "MountingHole:MountingHole_4mm_Pad" (at 64.77 135.255 0)
       (effects (font (size 1.27 1.27)) hide)
     )
@@
       (effects (font (size 1.27 1.27)) (justify left))
     )
-    (property "Footprint" "MountingHole:MountingHole_4.3mm_M4_ISO7380_Pad" (at 64.135 60.325 0)
+    (property "Footprint" "MountingHole:MountingHole_4mm_Pad" (at 64.135 60.325 0)
       (effects (font (size 1.27 1.27)) hide)
     )
@@
       (effects (font (size 1.27 1.27)) (justify left))
     )
-    (property "Footprint" "MountingHole:MountingHole_4.3mm_M4_ISO7380_Pad" (at 223.52 61.595 0)
+    (property "Footprint" "MountingHole:MountingHole_4mm_Pad" (at 223.52 61.595 0)
       (effects (font (size 1.27 1.27)) hide)
     )
@@
       (effects (font (size 1.27 1.27)) (justify left))
     )
-    (property "Footprint" "MountingHole:MountingHole_4.3mm_M4_ISO7380_Pad" (at 219.71 139.7 0)
+    (property "Footprint" "MountingHole:MountingHole_4mm_Pad" (at 219.71 139.7 0)
       (effects (font (size 1.27 1.27)) hide)
     )
@@
       (effects (font (size 1.27 1.27)) hide)
     )
-    (property "Footprint" "Connector_Coaxial:BNC_TEConnectivity_1478204_Vertical" (at 177.165 85.09 0)
-      (effects (font (size 1.27 1.27)) hide)
-    )
+    (property "Footprint" "Connector_Coaxial:BNC_TEConnectivity_1478035_Horizontal" (at 177.165 85.09 0)
+      (effects (font (size 1.27 1.27)) hide)
+    )
