File: rabbit_holder/rabbit_holder.kicad_pcb (KiCad board)
At the start: 2 copper layers, 105.8 x 84.8 mm, 67 parts, among them J1 Conn_02x32_Odd_Even, J10 Conn_01x01, J11 Conn_01x01, J12 Conn_01x01, J13 Conn_01x01, J15 Conn_01x01, J16 Conn_01x01, J17 Conn_01x01, J18 Conn_01x01, J19 Conn_01x01, J2 Conn_01x01, J20 Conn_01x01, J21 Conn_01x01, J22 Conn_01x01, J24 Conn_01x01, J25 Conn_01x01, J26 Conn_01x01, J27 Conn_01x01, J28 Conn_01x01, J29 Conn_01x01, J3 Conn_01x01, J30 Conn_01x01, J31 Conn_01x01, J32 Conn_01x01, J33 Conn_01x01, J34 Conn_01x01, J35 Conn_01x01, J37 Conn_01x01, J38 Conn_01x01, J39 Conn_01x01, J4 Conn_01x01, J40 Conn_01x01, J41 Conn_01x01, J42 Conn_01x01, J43 Conn_01x01, J44 Conn_01x01, J45 Conn_01x01, J46 Conn_01x01, J47 Conn_01x01, J48 Conn_01x01, J5 Conn_01x01, J50 Conn_01x01, J51 Conn_01x01, J52 Conn_01x01, J53 Conn_01x01, J54 Conn_01x01, J55 Conn_01x01, J56 Conn_01x01, J57 Conn_01x01, J59 Conn_01x01, J6 Conn_01x01, J60 Conn_01x01, J61 Conn_01x01, J62 Conn_01x01, J63 Conn_01x01, J64 Conn_01x01, J65 Conn_01x01, J66 Conn_01x01, J67 Conn_01x01, J68 Conn_01x01, J69 Conn_01x01, J7 Conn_01x01, J70 Conn_01x01, J8 Conn_01x01, J9 Conn_01x01

Commit message: update silk
Other:
- board text added: "df832fb"
- board text removed: "b8007ef"
Changed lines of the file:
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@@
   (gr_rect (start -19.27 18.73) (end -16.73 20.0025)
     (stroke (width 0.15) (type default)) (fill none) (layer "B.SilkS"))
-  (gr_rect (start -13.73 11.2725) (end -16.27 10)
+  (gr_rect (start -16.27 10) (end -13.73 11.2725)
     (stroke (width 0.15) (type default)) (fill none) (layer "B.SilkS"))
   (gr_rect (start 16.73 10) (end 19.27 11.2725)
@@
   (gr_rect (start -20 -16.27) (end -18.7275 -13.73)
     (stroke (width 0.15) (type default)) (fill none) (layer "B.SilkS"))
-  (gr_rect (start -11.2725 16.27) (end -10 13.73)
-    (stroke (width 0.15) (type default)) (fill none) (layer "B.SilkS"))
-  (gr_rect (start -10.73 11.2725) (end -13.27 10)
+  (gr_rect (start -11.2725 13.73) (end -10 16.27)
+    (stroke (width 0.15) (type default)) (fill none) (layer "B.SilkS"))
+  (gr_rect (start -13.27 10) (end -10.73 11.2725)
     (stroke (width 0.15) (type default)) (fill none) (layer "B.SilkS"))
   (gr_rect (start 13.73 18.7275) (end 16.27 20)
@@
   (gr_rect (start 13.73 -20) (end 16.27 -18.7275)
     (stroke (width 0.15) (type default)) (fill none) (layer "B.SilkS"))
-  (gr_rect (start -16.73 11.2725) (end -19.27 10)
+  (gr_rect (start -19.27 10) (end -16.73 11.2725)
     (stroke (width 0.15) (type default)) (fill none) (layer "B.SilkS"))
   (gr_line (start -42.5 -42.4) (end -42.5 42.4)
@@
   (gr_rect (start 13.73 10) (end 16.27 11.2725)
     (stroke (width 0.15) (type default)) (fill none) (layer "B.SilkS"))
-  (gr_rect (start -18.7275 13.73) (end -20 16.27)
+  (gr_rect (start -20 13.73) (end -18.7275 16.27)
     (stroke (width 0.15) (type default)) (fill none) (layer "B.SilkS"))
   (gr_rect (start -16.27 -20) (end -13.73 -18.7275)
@@
     (effects (font (size 1 1) (thickness 0.15)) (justify mirror))
   )
-  (gr_text "b8007ef" (at 0.905 -13.63 270) (layer "B.SilkS")
+  (gr_text "df832fb" (at 0.905 -13.63 270) (layer "B.SilkS")
     (effects (font (size 1 1) (thickness 0.125)) (justify mirror))
   )
@@
     (effects (font (size 1 1) (thickness 0.15)) (justify mirror))
   )
-  (gr_text "b8007ef" (at -61.095 35.87 270) (layer "F.SilkS")
+  (gr_text "df832fb" (at -61.095 35.87 270) (layer "F.SilkS")
     (effects (font (size 1 1) (thickness 0.125)) (justify left))
   )

Commit message: make two sided
Other:
- board text added: "arkmetrica.com"
Changed lines of the file:
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@@
     (fp_line (start 5.72 5.1) (end 5.72 -83.84)
       (stroke (width 0.1) (type solid)) (layer "B.Fab"))
-    (pad "1" thru_hole roundrect (at 0 0) (size 1.7 1.7) (drill 1) (layers "*.Cu" "*.Mask") (roundrect_rratio 0.147059)
+    (pad "1" thru_hole roundrect (at 0 0) (size 1.7 1.7) (drill 1) (layers "*.Cu" "*.Mask") (roundrect_rratio 0.1470588235)
       (net 63 "/3VT") (pinfunction "Pin_1") (pintype "passive"))
     (pad "2" thru_hole circle (at 2.54 0) (size 1.7 1.7) (drill 1) (layers "*.Cu" "*.Mask")
@@
   (gr_arc (start 37 40.4) (mid 36.414214 41.814214) (end 35 42.4)
     (stroke (width 0.1) (type solid)) (layer "Edge.Cuts"))
+  (gr_text "arkmetrica.com" (at -34.88 0) (layer "F.Cu")
+    (effects (font (size 1.5 1.5) (thickness 0.3) bold) (justify left bottom))
+  )
+  (gr_text "arkmetrica.com" (at 33.7 -20.32 90) (layer "F.Cu")
+    (effects (font (size 1.5 1.5) (thickness 0.3) bold) (justify left bottom))
+  )
+  (gr_text "arkmetrica.com" (at 33.7 38.1 90) (layer "F.Cu")
+    (effects (font (size 1.5 1.5) (thickness 0.3) bold) (justify left bottom))
+  )
   (gr_text "6" (at 18 -19.3625 180) (layer "B.SilkS")
     (effects (font (size 1 1) (thickness 0.15)) (justify mirror))

Commit message: change 1234 to abcd
Other:
- board text added: "7e2ad0d"
- board text added: "A"
- board text added: "B"
- board text added: "C"
- board text added: "D"
- board text removed: "df832fb"
Changed lines of the file:
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@@
     (effects (font (size 1 1) (thickness 0.15)) (justify mirror))
   )
-  (gr_text "3" (at 15 15) (layer "B.SilkS")
+  (gr_text "C" (at 15 15) (layer "B.SilkS")
     (effects (font (size 3 3) (thickness 0.3)) (justify mirror))
   )
@@
     (effects (font (size 1 1) (thickness 0.15)) (justify mirror))
   )
-  (gr_text "df832fb" (at 0.905 -13.63 270) (layer "B.SilkS")
+  (gr_text "7e2ad0d" (at 0.905 -13.63 270) (layer "B.SilkS")
     (effects (font (size 1 1) (thickness 0.125)) (justify mirror))
   )
@@
     (effects (font (size 1 1) (thickness 0.15)) (justify mirror))
   )
-  (gr_text "2" (at -15 -15) (layer "B.SilkS")
+  (gr_text "B" (at -15 -15) (layer "B.SilkS")
     (effects (font (size 3 3) (thickness 0.3)) (justify mirror))
   )
@@
     (effects (font (size 1 1) (thickness 0.15)) (justify mirror))
   )
-  (gr_text "1" (at -15 15) (layer "B.SilkS")
+  (gr_text "A" (at -15 15) (layer "B.SilkS")
     (effects (font (size 3 3) (thickness 0.3)) (justify mirror))
   )
@@
     (effects (font (size 1 1) (thickness 0.15)) (justify mirror))
   )
-  (gr_text "4" (at 15 -15) (layer "B.SilkS")
+  (gr_text "D" (at 15 -15) (layer "B.SilkS")
     (effects (font (size 3 3) (thickness 0.3)) (justify mirror))
   )
@@
     (effects (font (size 1 1) (thickness 0.15)) (justify mirror))
   )
-  (gr_text "df832fb" (at -61.095 35.87 270) (layer "F.SilkS")
+  (gr_text "7e2ad0d" (at -61.095 35.87 270) (layer "F.SilkS")
     (effects (font (size 1 1) (thickness 0.125)) (justify left))
   )

Commit message: update silk
Other:
- board text added: "4acdf1e"
- board text removed: "7e2ad0d"
Changed lines of the file:
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@@
     (effects (font (size 1 1) (thickness 0.15)) (justify mirror))
   )
-  (gr_text "7e2ad0d" (at 0.905 -13.63 270) (layer "B.SilkS")
+  (gr_text "4acdf1e" (at 0.905 -13.63 270) (layer "B.SilkS")
     (effects (font (size 1 1) (thickness 0.125)) (justify mirror))
   )
@@
     (effects (font (size 1 1) (thickness 0.15)) (justify mirror))
   )
-  (gr_text "7e2ad0d" (at -61.095 35.87 270) (layer "F.SilkS")
+  (gr_text "4acdf1e" (at -61.095 35.87 270) (layer "F.SilkS")
     (effects (font (size 1 1) (thickness 0.125)) (justify left))
   )
