File: snaith_holder/snaith_holder.kicad_pcb (KiCad board)
At the start: 2 copper layers, 30 x 30 mm, 32 parts, among them J1 Conn_02x08_Odd_Even, J10 Conn_01x01, J11 Conn_01x01, J12 Conn_01x01, J13 Conn_01x01, J14 Conn_01x01, J15 Conn_01x01, J16 Conn_01x01, J17 Conn_01x01, J18 Conn_01x01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

Commit message: update silk
Other:
- board text added: "febfbda"
- board text removed: "c5b4c2a"
Changed lines of the file:
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@@
     (effects (font (size 1 1) (thickness 0.15)) (justify mirror))
   )
-  (gr_text "c5b4c2a" (at 154.7 94.14 180) (layer "B.SilkS")
+  (gr_text "febfbda" (at 154.7 94.14 180) (layer "B.SilkS")
     (effects (font (size 0.5 0.5) (thickness 0.0625)) (justify mirror))
   )
@@
     (effects (font (size 1.5 1.5) (thickness 0.3) bold))
   )
-  (gr_text "c5b4c2a" (at 129 86.14 90) (layer "F.SilkS")
+  (gr_text "febfbda" (at 129 86.14 90) (layer "F.SilkS")
     (effects (font (size 0.5 0.5) (thickness 0.0625)))
   )
