File: direct_lightboard/direct_lightboard.kicad_pcb (KiCad board)
At the start: 2 copper layers, 90 x 90 mm, 22 parts, among them J1 Conn_01x01, J2 Conn_01x01, J3 Conn_01x01, J4 Conn_01x01, Q1 Q_NPN_BCEC, U1 LM7321MA

Commit message: update silk
Other:
- board text added: "fadbe0e"
- board text removed: "0b3434e"
Changed lines of the file:
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@@
 		(tags "resistor handsolder")
 		(property "Reference" "R1"
-			(at 0 -2.62 270)
+			(at 0 -2.62 -90)
 			(layer "F.SilkS")
 			(effects
@@
 		)
 		(property "Value" "1R"
-			(at 0 2.62 270)
+			(at 0 2.62 -90)
 			(layer "F.Fab")
 			(effects
@@
 		)
 		(fp_text user "${REFERENCE}"
-			(at 0 0 270)
+			(at 0 0 -90)
 			(layer "F.Fab")
 			(effects
@@
 		(tags "VSSOP-8 3.0 x 3.0")
 		(property "Reference" "U1"
-			(at -1 -2.5 360)
+			(at -1 -2.5 0)
 			(layer "F.SilkS")
 			(effects
@@
 		)
 		(property "Value" "LM7321MA	"
-			(at 0.02 2.73 360)
+			(at 0.02 2.73 0)
 			(layer "F.Fab")
 			(effects
@@
 		)
 		(fp_text user "${REFERENCE}"
-			(at 0 0 360)
+			(at 0 0 0)
 			(layer "F.Fab")
 			(effects
@@
 		(tags "capacitor handsolder")
 		(property "Reference" "C2"
-			(at -3 -0.5 270)
+			(at -3 -0.5 -90)
 			(layer "F.SilkS")
 			(effects
@@
 		)
 		(property "Value" "1n"
-			(at 0 1.68 270)
+			(at 0 1.68 -90)
 			(layer "F.Fab")
 			(effects
@@
 		)
 		(fp_text user "${REFERENCE}"
-			(at 0 0 270)
+			(at 0 0 -90)
 			(layer "F.Fab")
 			(effects
@@
 		(tags "LED Cree XB")
 		(property "Reference" "D1"
-			(at 0 2.5 270)
+			(at 0 2.5 -90)
 			(layer "F.SilkS")
 			(effects
@@
 		)
 		(property "Value" "LED_Pad"
-			(at 0 2.25 270)
+			(at 0 2.25 -90)
 			(layer "F.Fab")
 			(effects
@@
 		)
 		(fp_text user "${REFERENCE}"
-			(at 0 0 270)
+			(at 0 0 -90)
 			(layer "F.Fab")
 			(effects
@@
 		(layer "Edge.Cuts")
 	)
-	(gr_text "0b3434e"
+	(gr_text "fadbe0e"
 		(at 159 137 0)
 		(layer "F.SilkS")

Commit message: fix connector spacing
Parts:
- SYM1: footprint custom_footprints:logo -> custom_footprints:site_small
- moved J1 1.50 mm to (149.5, 60.1)
- moved J3 1.50 mm to (137.5, 60.1)
- moved J2 0.50 mm to (141.5, 60.1)
- moved J4 0.50 mm to (145.5, 60.1)
Routing:
- net Net-(J4-Pin_1): track 15.8 -> 14.6 mm
- net VCC: track 45.1 -> 44.4 mm
- net Net-(D4-K): track 54.4 -> 53.8 mm

Commit message: update silk
Other:
- board text added: "5373dc5"
- board text removed: "fadbe0e"
Changed lines of the file:
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@@
 		(layer "Edge.Cuts")
 	)
-	(gr_text "fadbe0e"
+	(gr_text "5373dc5"
 		(at 148.5 137.5 0)
 		(layer "F.SilkS")

Commit message: wip on lb
Parts:
- J1, J2, J3, J4: footprint Connector_TE-Connectivity:TE_2834006-1_1x01_P4.0mm_Horizontal -> custom_footprints:TE_2834006-1_1x01_P4.0mm_Horizontal
Changed lines of the file:
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@@
 		)
 	)
-	(footprint "Connector_TE-Connectivity:TE_2834006-1_1x01_P4.0mm_Horizontal"
+	(footprint "custom_footprints:TE_2834006-1_1x01_P4.0mm_Horizontal"
 		(layer "F.Cu")
 		(at 137.5 60.125 180)
@@
 			)
 		)
-		(property "Footprint" "Connector_TE-Connectivity:TE_2834006-1_1x01_P4.0mm_Horizontal"
+		(property "Footprint" "custom_footprints:TE_2834006-1_1x01_P4.0mm_Horizontal"
 			(at 0 0 180)
 			(unlocked yes)
@@
 		)
 		(fp_line
+			(start 1.5 4.5)
+			(end 1.5 0.5)
+			(stroke
+				(width 0.1)
+				(type default)
+			)
+			(layer "F.SilkS")
+		)
+		(fp_line
 			(start -1.3 -6.75)
 			(end -2.4 -6.75)
@@
 			(layer "F.SilkS")
 		)
+		(fp_rect
+			(start -3.11 4.21)
+			(end -2.1 5.282)
+			(stroke
+				(width 0.1)
+				(type solid)
+			)
+			(fill solid)
+			(layer "F.SilkS")
+		)
+		(fp_rect
+			(start -3.11 -5.64)
+			(end -2.1 -4.569)
+			(stroke
+				(width 0.1)
+				(type solid)
+			)
+			(fill solid)
+			(layer "F.SilkS")
+		)
+		(fp_poly
+			(pts
+				(xy 1 1) (xy 1.5 0.5) (xy 2 1)
+			)
+			(stroke
+				(width 0.1)
+				(type solid)
+			)
+			(fill solid)
+			(layer "F.SilkS")
+		)
 		(fp_line
 			(start 2.5 6.85)
@@
 			(layer "F.Fab")
 		)
-		(fp_rect
-			(start -3.11 4.21)
-			(end -2 5.282)
-			(stroke
-				(width 0.1)
-				(type solid)
-			)
-			(fill none)
-			(layer "F.Fab")
-		)
-		(fp_rect
-			(start -3.11 -5.64)
-			(end -2 -4.569)
-			(stroke
-				(width 0.1)
-				(type solid)
-			)
-			(fill none)
-			(layer "F.Fab")
-		)
 		(fp_circle
 			(center 0 -2.45)
@@
 			(pintype "passive")
 		)
-		(model "${KICAD8_3DMODEL_DIR}/Connector_TE-Connectivity.3dshapes/TE_2834006-1_1x01_P4.0mm_Horizontal.wrl"
+		(model "${KIPRJMOD}/../shared_libs/3d/c-2834006-1-c-3d.stp"
 			(offset
-				(xyz 0 0 0)
+				(xyz 0 -6 1.875)
 			)
 			(scale
@@
 			)
 			(rotate
-				(xyz 0 0 0)
+				(xyz -90 0 0)
 			)
 		)
@@
 		)
 	)
-	(footprint "Connector_TE-Connectivity:TE_2834006-1_1x01_P4.0mm_Horizontal"
+	(footprint "custom_footprints:TE_2834006-1_1x01_P4.0mm_Horizontal"
 		(layer "F.Cu")
 		(at 145.5 60.125 180)
@@
 			)
 		)
-		(property "Footprint" "Connector_TE-Connectivity:TE_2834006-1_1x01_P4.0mm_Horizontal"
+		(property "Footprint" "custom_footprints:TE_2834006-1_1x01_P4.0mm_Horizontal"
 			(at 0 0 180)
 			(unlocked yes)
@@
 		)
 		(fp_line
+			(start 1.5 4.5)
+			(end 1.5 0.5)
+			(stroke
+				(width 0.1)
+				(type default)
+			)
+			(layer "F.SilkS")
+		)
+		(fp_line
 			(start -1.3 -6.75)
 			(end -2.4 -6.75)
@@
 			(layer "F.SilkS")
 		)
+		(fp_rect
+			(start -3.11 4.21)
+			(end -2.1 5.282)
+			(stroke
+				(width 0.1)
+				(type solid)
+			)
+			(fill solid)
+			(layer "F.SilkS")
+		)
+		(fp_rect
+			(start -3.11 -5.64)
+			(end -2.1 -4.569)
+			(stroke
+				(width 0.1)
+				(type solid)
+			)
+			(fill solid)
+			(layer "F.SilkS")
+		)
+		(fp_poly
+			(pts
+				(xy 1 1) (xy 1.5 0.5) (xy 2 1)
+			)
+			(stroke
+				(width 0.1)
+				(type solid)
+			)
+			(fill solid)
+			(layer "F.SilkS")
+		)
 		(fp_line
 			(start 2.5 6.85)
@@
 			(layer "F.Fab")
 		)
-		(fp_rect
-			(start -3.11 4.21)
-			(end -2 5.282)
-			(stroke
-				(width 0.1)
-				(type solid)
-			)
-			(fill none)
-			(layer "F.Fab")
-		)
-		(fp_rect
-			(start -3.11 -5.64)
-			(end -2 -4.569)
-			(stroke
-				(width 0.1)
-				(type solid)
-			)
-			(fill none)
-			(layer "F.Fab")
-		)
 		(fp_circle
 			(center 0 -2.45)
@@
 			(pintype "passive")
 		)
-		(model "${KICAD8_3DMODEL_DIR}/Connector_TE-Connectivity.3dshapes/TE_2834006-1_1x01_P4.0mm_Horizontal.wrl"
+		(model "${KIPRJMOD}/../shared_libs/3d/c-2834006-1-c-3d.stp"
 			(offset
-				(xyz 0 0 0)
+				(xyz 0 -6 1.875)
 			)
 			(scale
@@
 			)
 			(rotate
-				(xyz 0 0 0)
+				(xyz -90 0 0)
 			)
 		)
@@
 		)
 	)
-	(footprint "Connector_TE-Connectivity:TE_2834006-1_1x01_P4.0mm_Horizontal"
+	(footprint "custom_footprints:TE_2834006-1_1x01_P4.0mm_Horizontal"
 		(layer "F.Cu")
 		(at 141.5 60.125 180)
@@
 			)
 		)
-		(property "Footprint" "Connector_TE-Connectivity:TE_2834006-1_1x01_P4.0mm_Horizontal"
+		(property "Footprint" "custom_footprints:TE_2834006-1_1x01_P4.0mm_Horizontal"
 			(at 0 0 180)
 			(unlocked yes)
@@
 		)
 		(fp_line
+			(start 1.5 4.5)
+			(end 1.5 0.5)
+			(stroke
+				(width 0.1)
+				(type default)
+			)
+			(layer "F.SilkS")
+		)
+		(fp_line
 			(start -1.3 -6.75)
 			(end -2.4 -6.75)
@@
 			(layer "F.SilkS")
 		)
+		(fp_rect
+			(start -3.11 4.21)
+			(end -2.1 5.282)
+			(stroke
+				(width 0.1)
+				(type solid)
+			)
+			(fill solid)
+			(layer "F.SilkS")
+		)
+		(fp_rect
+			(start -3.11 -5.64)
+			(end -2.1 -4.569)
+			(stroke
+				(width 0.1)
+				(type solid)
+			)
+			(fill solid)
+			(layer "F.SilkS")
+		)
+		(fp_poly
+			(pts
+				(xy 1 1) (xy 1.5 0.5) (xy 2 1)
+			)
+			(stroke
+				(width 0.1)
+				(type solid)
+			)
+			(fill solid)
+			(layer "F.SilkS")
+		)
 		(fp_line
 			(start 2.5 6.85)
@@
 			(layer "F.Fab")
 		)
-		(fp_rect
-			(start -3.11 4.21)
-			(end -2 5.282)
-			(stroke
-				(width 0.1)
-				(type solid)
-			)
-			(fill none)
-			(layer "F.Fab")
-		)
-		(fp_rect
-			(start -3.11 -5.64)
-			(end -2 -4.569)
-			(stroke
-				(width 0.1)
-				(type solid)
-			)
-			(fill none)
-			(layer "F.Fab")
-		)
 		(fp_circle
 			(center 0 -2.45)
@@
 			(pintype "passive")
 		)
-		(model "${KICAD8_3DMODEL_DIR}/Connector_TE-Connectivity.3dshapes/TE_2834006-1_1x01_P4.0mm_Horizontal.wrl"
+		(model "${KIPRJMOD}/../shared_libs/3d/c-2834006-1-c-3d.stp"
 			(offset
-				(xyz 0 0 0)
+				(xyz 0 -6 1.875)
 			)
 			(scale
@@
 			)
 			(rotate
-				(xyz 0 0 0)
+				(xyz -90 0 0)
 			)
 		)
@@
 		)
 	)
-	(footprint "Connector_TE-Connectivity:TE_2834006-1_1x01_P4.0mm_Horizontal"
+	(footprint "custom_footprints:TE_2834006-1_1x01_P4.0mm_Horizontal"
 		(layer "F.Cu")
 		(at 149.5 60.125 180)
@@
 			)
 		)
-		(property "Footprint" "Connector_TE-Connectivity:TE_2834006-1_1x01_P4.0mm_Horizontal"
+		(property "Footprint" "custom_footprints:TE_2834006-1_1x01_P4.0mm_Horizontal"
 			(at 0 0 180)
 			(unlocked yes)
@@
 		)
 		(fp_line
+			(start 1.5 4.5)
+			(end 1.5 0.5)
+			(stroke
+				(width 0.1)
+				(type default)
+			)
+			(layer "F.SilkS")
+		)
+		(fp_line
 			(start -1.3 -6.75)
 			(end -2.4 -6.75)
@@
 			(layer "F.SilkS")
 		)
+		(fp_rect
+			(start -3.11 4.21)
+			(end -2.1 5.282)
+			(stroke
+				(width 0.1)
+				(type solid)
+			)
+			(fill solid)
+			(layer "F.SilkS")
+		)
+		(fp_rect
+			(start -3.11 -5.64)
+			(end -2.1 -4.569)
+			(stroke
+				(width 0.1)
+				(type solid)
+			)
+			(fill solid)
+			(layer "F.SilkS")
+		)
+		(fp_poly
+			(pts
+				(xy 1 1) (xy 1.5 0.5) (xy 2 1)
+			)
+			(stroke
+				(width 0.1)
+				(type solid)
+			)
+			(fill solid)
+			(layer "F.SilkS")
+		)
 		(fp_line
 			(start 2.5 6.85)
@@
 			(layer "F.Fab")
 		)
-		(fp_rect
-			(start -3.11 4.21)
-			(end -2 5.282)
-			(stroke
-				(width 0.1)
-				(type solid)
-			)
-			(fill none)
-			(layer "F.Fab")
-		)
-		(fp_rect
-			(start -3.11 -5.64)
-			(end -2 -4.569)
-			(stroke
-				(width 0.1)
-				(type solid)
-			)
-			(fill none)
-			(layer "F.Fab")
-		)
 		(fp_circle
 			(center 0 -2.45)
@@
 			(pintype "passive")
 		)
-		(model "${KICAD8_3DMODEL_DIR}/Connector_TE-Connectivity.3dshapes/TE_2834006-1_1x01_P4.0mm_Horizontal.wrl"
+		(model "${KIPRJMOD}/../shared_libs/3d/c-2834006-1-c-3d.stp"
 			(offset
-				(xyz 0 0 0)
+				(xyz 0 -6 1.875)
 			)
 			(scale
@@
 			)
 			(rotate
-				(xyz 0 0 0)
+				(xyz -90 0 0)
 			)
 		)
