File: direct_lightboard/direct_lightboard.kicad_sch (KiCad schematic)
At the start: 22 parts, among them J1 Conn_01x01, J2 Conn_01x01, J3 Conn_01x01, J4 Conn_01x01, Q1 Q_NPN_BCEC, U1 LM7321MA

Commit message: fix connector spacing
Parts:
- SYM1: footprint custom_footprints:logo -> custom_footprints:site_small
Changed lines of the file:
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@@
 		(at 184.15 173.99 0)
 		(unit 1)
-		(exclude_from_sim no)
+		(exclude_from_sim yes)
 		(in_bom no)
 		(on_board yes)
@@
 			)
 		)
-		(property "Footprint" "custom_footprints:logo"
+		(property "Footprint" "custom_footprints:site_small"
 			(at 184.15 173.99 0)
 			(effects
@@
 			(at 184.15 173.99 0)
 			(effects
-				(font
-					(size 1.27 1.27)
-				)
-				(hide yes)
-			)
-		)
-		(property "Sim.Enable" "0"
-			(at 184.15 173.99 0)
-			(effects

Commit message: wip on lb
Parts:
- J1, J2, J3, J4: footprint Connector_TE-Connectivity:TE_2834006-1_1x01_P4.0mm_Horizontal -> custom_footprints:TE_2834006-1_1x01_P4.0mm_Horizontal
Changed lines of the file:
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@@
 			)
 		)
-		(property "Footprint" "Connector_TE-Connectivity:TE_2834006-1_1x01_P4.0mm_Horizontal"
+		(property "Footprint" "custom_footprints:TE_2834006-1_1x01_P4.0mm_Horizontal"
 			(at 96.52 100.33 0)
 			(effects
@@
 			)
 		)
-		(property "Footprint" "Connector_TE-Connectivity:TE_2834006-1_1x01_P4.0mm_Horizontal"
+		(property "Footprint" "custom_footprints:TE_2834006-1_1x01_P4.0mm_Horizontal"
 			(at 186.69 87.63 0)
 			(effects
@@
 			)
 		)
-		(property "Footprint" "Connector_TE-Connectivity:TE_2834006-1_1x01_P4.0mm_Horizontal"
+		(property "Footprint" "custom_footprints:TE_2834006-1_1x01_P4.0mm_Horizontal"
 			(at 187.96 36.83 0)
 			(effects
@@
 			)
 		)
-		(property "Footprint" "Connector_TE-Connectivity:TE_2834006-1_1x01_P4.0mm_Horizontal"
+		(property "Footprint" "custom_footprints:TE_2834006-1_1x01_P4.0mm_Horizontal"
 			(at 181.61 146.05 0)
 			(effects
