File: distrobd/distrobd.kicad_pcb (KiCad board)
At the start: 4 copper layers, 276 x 216 mm, 91 parts, among them J1 Conn_01x01, J10 Conn_01x01, J11 Conn_01x01, J12 Conn_02x03_Odd_Even, J13 Conn_02x03_Odd_Even, J14 Conn_02x03_Odd_Even, J15 Conn_02x03_Odd_Even, J16 Conn_01x01, J17 Conn_01x01, J18 Conn_02x03_Odd_Even, J19 Conn_02x03_Odd_Even, J2 Conn_01x01, J20 Conn_01x01, J21 Conn_01x01, J22 Conn_02x03_Odd_Even, J23 Conn_02x03_Odd_Even, J24 Conn_01x01, J25 Conn_01x01, J26 Conn_02x03_Odd_Even, J27 Conn_02x03_Odd_Even, J28 Conn_01x01, J29 Conn_01x01, J3 Conn_01x14, J30 Conn_02x03_Odd_Even, J31 Conn_02x03_Odd_Even, J32 Conn_01x01, J33 Conn_01x01, J34 Conn_02x03_Odd_Even, J35 Conn_02x03_Odd_Even, J36 Conn_01x01, J37 Conn_01x01, J38 Conn_02x03_Odd_Even, J39 Conn_02x03_Odd_Even, J4 Conn_01x14, J40 Conn_01x01, J41 Conn_01x01, J42 Conn_02x03_Odd_Even, J43 Conn_02x03_Odd_Even, J44 Conn_01x01, J45 Conn_01x01, J46 Conn_01x01, J47 Conn_01x01, J48 Conn_01x01, J49 Conn_01x01, J5 Conn_01x01, J50 Conn_01x01, J51 Conn_01x01, J6 Conn_01x01, J7 Conn_01x06, J8 Conn_01x06, J9 Conn_01x08

Commit message: update silk
Other:
- board text added: "3523217"
Changed lines of the file:
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@@
+		)
+	)
+	(gr_text "3523217"
+		(at 122 -107 180)
+		(layer "F.SilkS")
+		(effects
+			(font
+				(size 1 1)
+				(thickness 0.1)
+			)
+			(justify left bottom)
 		)
 	)

Commit message: minor touchups
Parts:
- added J52: Conn_01x04, Connector_Harwin:Harwin_M20-89004xx_1x04_P2.54mm_Horizontal, F.Cu at (-126.3, -26.6)
- added JP3: SolderJumper_2_Bridged, Jumper:SolderJumper-2_P1.3mm_Bridged_RoundedPad1.0x1.5mm, F.Cu at (-127.0, -34.4)
- added JP4: SolderJumper_2_Bridged, Jumper:SolderJumper-2_P1.3mm_Bridged_RoundedPad1.0x1.5mm, F.Cu at (-133.0, -34.4)
- added R1: 4k7, Resistor_SMD:R_1206_3216Metric_Pad1.30x1.75mm_HandSolder, F.Cu at (-123.2, -6.35)
- added R2: 4k7, Resistor_SMD:R_1206_3216Metric_Pad1.30x1.75mm_HandSolder, F.Cu at (-125.7, -6.35)
- added R3: 4k7, Resistor_SMD:R_1206_3216Metric_Pad1.30x1.75mm_HandSolder, F.Cu at (-128.3, -6.35)
- added R4: 4k7, Resistor_SMD:R_1206_3216Metric_Pad1.30x1.75mm_HandSolder, F.Cu at (-130.8, -6.35)
- moved SYM1 1.27 mm to (126.0, -104.0)
Connections:
- J4 pad 6: unconnected-(J4-Pin_6-Pad6) -> /SDA3
- J4 pad 7: unconnected-(J4-Pin_7-Pad7) -> /SCL3
- J8 pad 1: unconnected-(J8-Pin_1-Pad1) -> Net-(J52-Pin_2)
- J8 pad 2: unconnected-(J8-Pin_2-Pad2) -> /DUINO_GND
- J8 pad 3: unconnected-(J8-Pin_3-Pad3) -> Net-(J8-Pin_3)
- J8 pad 4: unconnected-(J8-Pin_4-Pad4) -> Net-(J8-Pin_4)
Routing:
- net /SCL3: track 0.00 -> 59.9 mm, vias 0 -> 2
- net /SDA3: track 0.00 -> 47.8 mm, vias 0 -> 2
- net Net-(J8-Pin_4): track 0.00 -> 38.0 mm, vias 0 -> 3
- net Net-(J8-Pin_3): track 0.00 -> 35.9 mm, vias 0 -> 2
- net Net-(J52-Pin_2): track 0.00 -> 33.7 mm, vias 0 -> 2
- net /V_CGND: track 169.4 -> 182.6 mm
- net /+5V: track 93.0 -> 104.2 mm, vias 2 -> 4
- net /VC: track 636.1 -> 646.5 mm, vias 19 -> 14
- net /VA: track 626.1 -> 630.7 mm, vias 19 -> 14
- net /VB: track 627.1 -> 631.6 mm, vias 19 -> 14
- net Net-(J25-Pin_1): track 159.4 -> 163.4 mm
- net /DUINO_GND: track 99.4 -> 101.0 mm, vias 2 -> 3
- net /VD: vias 19 -> 14
Other:
- board size 276 x 216 mm -> 274 x 216 mm
- board text added: "INTERLOCK"

Commit message: fillet corners
Other:
- outline, holes or cut-outs redrawn
- board text added: "ba9f584"
- board text removed: "3523217"
Changed lines of the file:
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@@
 		(allow_soldermask_bridges_in_footprints no)
 		(tenting front back)
-		(grid_origin -127.175 -26.57)
 		(pcbplotparams
 			(layerselection 0x00000000_00000000_55555555_5755f5ff)
@@
 	)
 	(gr_line
-		(start -137 -108)
-		(end -137 108)
+		(start -137 -106)
+		(end -137 106)
 		(stroke
 			(width 0.05)
@@
 		(layer "Edge.Cuts")
 	)
+	(gr_arc
+		(start 137 106)
+		(mid 136.414214 107.414214)
+		(end 135 108)
+		(stroke
+			(width 0.05)
+			(type default)
+		)
+		(layer "Edge.Cuts")
+	)
 	(gr_line
 		(start -96.5 -97.5)
@@
 	)
 	(gr_line
-		(start -137 108)
-		(end 137 108)
+		(start -135 108)
+		(end 135 108)
 		(stroke
 			(width 0.05)
@@
 		(layer "Edge.Cuts")
 	)
+	(gr_arc
+		(start 135 -108)
+		(mid 136.414214 -107.414214)
+		(end 137 -106)
+		(stroke
+			(width 0.05)
+			(type default)
+		)
+		(layer "Edge.Cuts")
+	)
 	(gr_line
 		(start 127.646447 -99.767767)
@@
 	)
 	(gr_line
-		(start 137 -108)
-		(end 137 108)
+		(start 137 -106)
+		(end 137 106)
 		(stroke
 			(width 0.05)
@@
 		(layer "Edge.Cuts")
 	)
+	(gr_arc
+		(start -135 108)
+		(mid -136.414214 107.414214)
+		(end -137 106)
+		(stroke
+			(width 0.05)
+			(type default)
+		)
+		(layer "Edge.Cuts")
+	)
 	(gr_line
 		(start 47.5 -97.5)
@@
 	)
 	(gr_line
-		(start 137 -108)
-		(end -137 -108)
+		(start 135 -108)
+		(end -135 -108)
 		(stroke
 			(width 0.05)
@@
 	)
 	(gr_arc
+		(start -137 -106)
+		(mid -136.414214 -107.414214)
+		(end -135 -108)
+		(stroke
+			(width 0.05)
+			(type default)
+		)
+		(layer "Edge.Cuts")
+	)
+	(gr_arc
 		(start -47.5 -97.5)
 		(mid -46.792893 -97.207107)
@@
 		)
 	)
-	(gr_text "3523217"
+	(gr_text "ba9f584"
 		(at 122 -107 180)
 		(layer "F.SilkS")

Commit message: update silk
Other:
- board text added: "ab0086a"
- board text removed: "ba9f584"
Changed lines of the file:
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@@
 		)
 	)
-	(gr_text "ba9f584"
+	(gr_text "ab0086a"
 		(at 122 -107 180)
 		(layer "F.SilkS")

Commit message: switch opamps to dual flavors, build in on-board TEC current control
Parts:
- added C1: C, Capacitor_SMD:C_0805_2012Metric_Pad1.18x1.45mm_HandSolder, F.Cu at (-128.0, 50.5)
- added Q1: Q_NPN_CBE, Package_TO_SOT_SMD:TO-252-2, F.Cu at (-120.0, 51.0)
- added R5: 1R, Resistor_SMD:R_2512_6332Metric_Pad1.40x3.35mm_HandSolder, F.Cu at (-122.3, 40.0)
- added R6: 4k7, Resistor_SMD:R_1206_3216Metric_Pad1.30x1.75mm_HandSolder, F.Cu at (-128.8, 37.7)
- added U1: OPA2994xD, Package_SO:SOIC-8_3.9x4.9mm_P1.27mm, F.Cu at (-129.9, 44.0)
- moved J5 13.0 mm to (-123.4, 62.0)
- moved J6 13.0 mm to (-123.4, 58.0)
- moved J2 4.00 mm to (-123.4, 66.0)
- moved J46 4.00 mm to (-123.4, 78.0)
- moved J47 4.00 mm to (-123.4, 74.0)
- moved J48 4.00 mm to (-123.4, 70.0)
Routing:
- net /DAC: track 0.00 -> 130.7 mm, vias 0 -> 3
- net /V_PGND: track 117.1 -> 145.7 mm
- net Net-(Q1-B): track 0.00 -> 14.8 mm, vias 0 -> 2
- net Net-(Q1-E): track 0.00 -> 11.9 mm, vias 0 -> 2
- net /DUINO_GND: track 101.0 -> 111.1 mm, vias 3 -> 4
- net /VGND: track 0.00 -> 7.17 mm, vias 61 -> 68
- net /V_PSS: track 290.7 -> 296.5 mm
- net /VSS: track 0.00 -> 5.23 mm
- net unconnected-(U1-Pad7): track 0.00 -> 3.60 mm

Commit message: update silk
Other:
- board text added: "ee118a9"
- board text removed: "ab0086a"
Changed lines of the file:
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@@
 		)
 	)
-	(gr_text "ab0086a"
+	(gr_text "ee118a9"
 		(at 122 -107 180)
 		(layer "F.SilkS")

Commit message: update silk
Other:
- board text added: "6737c55"
- board text removed: "ee118a9"
Changed lines of the file:
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@@
 		)
 	)
-	(gr_text "ee118a9"
+	(gr_text "6737c55"
 		(at 122 -107 180)
 		(layer "F.SilkS")

Commit message: update silk
Other:
- board text added: "5547698"
- board text removed: "6737c55"
Changed lines of the file:
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@@
 		)
 	)
-	(gr_text "6737c55"
+	(gr_text "5547698"
 		(at 122 -107 180)
 		(layer "F.SilkS")
