File: fourch_direct_lightboard/fourch_direct_lightboard.kicad_pcb (KiCad board)
At the start: 2 copper layers, 72 x 72 mm, 65 parts, among them J1 Conn_01x01_Pin, J10 Conn_01x01_Pin, J11 Conn_01x01_Pin, J12 Conn_01x01_Pin, J2 Conn_01x01_Pin, J3 Conn_01x01_Pin, J4 Conn_01x01_Pin, J5 Conn_01x01_Pin, J6 Conn_01x01_Pin, J7 Conn_01x01_Pin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

Commit message: switch opamps to dual flavors, build in on-board TEC current control
Parts:
- Q1, Q2, Q3, Q4: value Q_NPN_CBE -> NSS1C301ET4G
Changed lines of the file:
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@@
 		(sheetname "/")
 		(sheetfile "fourch_direct_lightboard.kicad_sch")
-		(attr exclude_from_pos_files)
+		(attr exclude_from_pos_files dnp)
 		(fp_circle
 			(center 0 0)
@@
 		(sheetname "/")
 		(sheetfile "fourch_direct_lightboard.kicad_sch")
-		(attr smd)
+		(attr smd dnp)
 		(fp_line
 			(start -0.227064 0.735)
@@
 		(sheetname "/")
 		(sheetfile "fourch_direct_lightboard.kicad_sch")
-		(attr smd)
+		(attr smd dnp)
 		(fp_line
 			(start -0.227064 0.735)
@@
 		(sheetname "/")
 		(sheetfile "fourch_direct_lightboard.kicad_sch")
-		(attr exclude_from_pos_files)
+		(attr exclude_from_pos_files dnp)
 		(fp_circle
 			(center 0 0)
@@
 		(sheetname "/")
 		(sheetfile "fourch_direct_lightboard.kicad_sch")
-		(attr exclude_from_pos_files)
+		(attr exclude_from_pos_files dnp)
 		(fp_circle
 			(center 0 0)
@@
 		(sheetname "/")
 		(sheetfile "fourch_direct_lightboard.kicad_sch")
-		(attr exclude_from_pos_files)
+		(attr exclude_from_pos_files dnp)
 		(fp_circle
 			(center 0 0)
@@
 		(sheetname "/")
 		(sheetfile "fourch_direct_lightboard.kicad_sch")
-		(attr exclude_from_pos_files)
+		(attr exclude_from_pos_files dnp)
 		(fp_circle
 			(center 0 0)
@@
 		(sheetname "/")
 		(sheetfile "fourch_direct_lightboard.kicad_sch")
-		(attr exclude_from_pos_files)
+		(attr exclude_from_pos_files dnp)
 		(fp_circle
 			(center 0 0)
@@
 		(sheetname "/")
 		(sheetfile "fourch_direct_lightboard.kicad_sch")
-		(attr exclude_from_pos_files)
+		(attr exclude_from_pos_files dnp)
 		(fp_circle
 			(center 0 0)
@@
 		(sheetname "/")
 		(sheetfile "fourch_direct_lightboard.kicad_sch")
-		(attr exclude_from_pos_files)
+		(attr exclude_from_pos_files dnp)
 		(fp_circle
 			(center 0 0)
@@
 		(sheetname "/")
 		(sheetfile "fourch_direct_lightboard.kicad_sch")
-		(attr exclude_from_pos_files)
+		(attr exclude_from_pos_files dnp)
 		(fp_circle
 			(center 0 0)
@@
 		(sheetname "/")
 		(sheetfile "fourch_direct_lightboard.kicad_sch")
-		(attr smd)
+		(attr smd dnp)
 		(fp_line
 			(start -0.227064 0.735)
@@
 		(sheetname "/")
 		(sheetfile "fourch_direct_lightboard.kicad_sch")
-		(attr smd)
+		(attr smd dnp)
 		(fp_line
 			(start -0.227064 -0.735)
@@
 			)
 		)
-		(property "Value" "Q_NPN_CBE"
+		(property "Value" "NSS1C301ET4G"
 			(at 0 4.5 0)
 			(layer "F.Fab")
@@
 			)
 		)
-		(property "Value" "Q_NPN_CBE"
+		(property "Value" "NSS1C301ET4G"
 			(at 0 4.5 0)
 			(layer "F.Fab")
@@
 		(sheetname "/")
 		(sheetfile "fourch_direct_lightboard.kicad_sch")
-		(attr exclude_from_pos_files)
+		(attr exclude_from_pos_files dnp)
 		(fp_circle
 			(center 0 0)
@@
 			)
 		)
-		(property "Value" "Q_NPN_CBE"
+		(property "Value" "NSS1C301ET4G"
 			(at 0 4.5 0)
 			(layer "F.Fab")
@@
 		(sheetname "/")
 		(sheetfile "fourch_direct_lightboard.kicad_sch")
-		(attr exclude_from_pos_files)
+		(attr exclude_from_pos_files dnp)
 		(fp_circle
 			(center 0 0)
@@
 		(sheetname "/")
 		(sheetfile "fourch_direct_lightboard.kicad_sch")
-		(attr smd)
+		(attr smd dnp)
 		(fp_line
 			(start -0.227064 -0.735)
@@
 		(sheetname "/")
 		(sheetfile "fourch_direct_lightboard.kicad_sch")
-		(attr smd)
+		(attr smd dnp)
 		(fp_line
 			(start -0.227064 -0.735)
@@
 		(sheetname "/")
 		(sheetfile "fourch_direct_lightboard.kicad_sch")
-		(attr smd)
+		(attr smd dnp)
 		(fp_line
 			(start -0.227064 0.735)
@@
 		(sheetname "/")
 		(sheetfile "fourch_direct_lightboard.kicad_sch")
-		(attr smd)
+		(attr smd dnp)
 		(fp_line
 			(start -0.227064 0.735)
@@
 		(sheetname "/")
 		(sheetfile "fourch_direct_lightboard.kicad_sch")
-		(attr exclude_from_pos_files)
+		(attr exclude_from_pos_files dnp)
 		(fp_circle
 			(center 0 0)
@@
 			)
 		)
-		(property "Value" "Q_NPN_CBE"
+		(property "Value" "NSS1C301ET4G"
 			(at 0 4.5 0)
 			(layer "F.Fab")

Commit message: update silk
Other:
- board text added: "ee118a9"
- board text removed: "ab0086a"
Changed lines of the file:
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@@
 		(layer "User.1")
 	)
-	(gr_text "ab0086a"
+	(gr_text "ee118a9"
 		(at 8 -4.5 0)
 		(layer "F.SilkS")

Commit message: update silk
Other:
- board text added: "6737c55"
- board text removed: "ee118a9"
Changed lines of the file:
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@@
 		(layer "User.1")
 	)
-	(gr_text "ee118a9"
+	(gr_text "6737c55"
 		(at 8 -4.5 0)
 		(layer "F.SilkS")

Commit message: update silk
Other:
- board text added: "5547698"
- board text removed: "6737c55"
Changed lines of the file:
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@@
 		(layer "User.1")
 	)
-	(gr_text "6737c55"
+	(gr_text "5547698"
 		(at 8 -4.5 0)
 		(layer "F.SilkS")

Commit message: update silk
Other:
- board text added: "8792bd6"
- board text removed: "5547698"
Changed lines of the file:
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@@
 		(layer "User.1")
 	)
-	(gr_text "5547698"
+	(gr_text "8792bd6"
 		(at 8 -4.5 0)
 		(layer "F.SilkS")

Commit message: rev up light
Parts:
- moved TH6 1.61 mm to (2.50, -17.1)
- moved TH5 1.18 mm to (-17.8, -3.17)
- moved TH1 1.15 mm to (6.35, -12.0)
- moved TH2 1.15 mm to (-12.0, -6.35)
- moved TH7 0.95 mm to (-2.56, 6.35)
- moved TH3 0.77 mm to (6.99, 11.4)
- moved TH4 0.64 mm to (-12.0, 17.1)
- moved TH8 0.34 mm to (-2.54, 18.4)

Commit message: update silk
Other:
- board text added: "325c7a5"
- board text removed: "8792bd6"
Changed lines of the file:
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@@
 		(layer "User.1")
 	)
-	(gr_text "8792bd6"
+	(gr_text "325c7a5"
 		(at 8 -4.5 0)
 		(layer "F.SilkS")
