File: arkplat3/arkplat3.kicad_pcb (KiCad board)
At the start: 2 copper layers, 160 x 100 mm, 45 parts, among them J1 Conn_02x10_Odd_Even, J10 AG5800OUT, J2 J-LINK NEEDLE, J3 Conn_02x04_Odd_Even, J4 Conn_02x04_Odd_Even, J5 Conn_02x14_Odd_Even, J6 Conn_02x14_Odd_Even, J7 RJ45_JK00177, J8 RJ45_Shielded, J9 AG5800IN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

Commit message: update silk
Other:
- board text added: "0da12f3"
- board text removed: "abcdefg"
Changed lines of the file:
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@@
 		(grid_origin 74 63)
 		(pcbplotparams
-			(layerselection 0x00000000_00000000_55555555_575555ff)
+			(layerselection 0x00000000_00000000_55555555_5755f5ff)
 			(plot_on_all_layers_selection 0x00000000_00000000_00000000_00000000)
 			(disableapertmacros no)
@@
 		(layer "Edge.Cuts")
 	)
-	(gr_text "abcdefg"
+	(gr_text "0da12f3"
 		(at 59 129 270)
 		(layer "F.SilkS")
@@
 		(single_sided no)
 		(target_length 67)
-		(target_length_max 67.1)
+		(target_length_max 67.099999)
 		(target_length_min 66.9)
 		(target_skew 0)
@@
 		(single_sided no)
 		(target_length 67)
-		(target_length_max 67.1)
+		(target_length_max 67.099999)
 		(target_length_min 66.9)
 		(target_skew 0)
@@
 		(single_sided no)
 		(target_length 65.3241)
-		(target_length_max 65.4241)
+		(target_length_max 65.424099)
 		(target_length_min 65.2241)
 		(target_skew 0)
